Commit message: fix link

File: sobit_pro_description/urdf/sensor/azure_kinect.urdf.xacro (robot description, xacro)
@@ -5,8 +5,8 @@
     <joint name="${prefix}_joint" type="fixed">
       <parent link="${parent}" />
-      <child link="${prefix}_link" />
+      <child link="${prefix}_base" />
       <origin xyz="0 0 0" rpy="0 0 0" />
     </joint>
-    <link name="${prefix}_link">
+    <link name="${prefix}_base">
       <visual>
         <origin xyz="0 0 -0.06" rpy="1.570796327 0 0" />

Commit message: Various corrections

File: sobit_pro_description/urdf/sensor/azure_kinect.urdf.xacro (robot description, xacro)
@@ -6,9 +6,9 @@
       <parent link="${parent}" />
       <child link="${prefix}_base" />
-      <origin xyz="0 0 0" rpy="0 0 0" />
+      <origin xyz="0 0 0" rpy="0 0 -1.570796327" />
     </joint>
     <link name="${prefix}_base">
       <visual>
-        <origin xyz="0 0 -0.06" rpy="1.570796327 0 0" />
+        <origin xyz="0 0 -0.06" rpy="1.570796327 0 1.570796327" />
         <geometry>
           <mesh filename="package://sobit_pro_description/meshes/sensor/azure_kinect.dae"/>
