Commit message: sobit_pro: split arm/head control wiring and sensor topic updates

File: sobit_pro_description/urdf/sensor/xtion.urdf.xacro (robot description, xacro)
@@ -29,6 +29,5 @@
       <!-- <origin xyz="0 ${asus_xtion_pro_cam_rel_rgb_py} 0" rpy="0.0 0.0 0.0"/> -->
       <origin xyz="${-asus_xtion_pro_cam_rel_rgb_py} 0 -0.019" rpy="0.0 0.0 0.0"/>
-      <!-- <parent link="${parent}"/> -->
-      <parent link="${prefix}_rgb_optical_frame"/>
+      <parent link="${parent}"/>
       <child link="${prefix}_link"/>
     </joint>

Commit message: [FIX]: Update xtion mounting transform for stable TF linkage

File: sobit_pro_description/urdf/sensor/xtion.urdf.xacro (robot description, xacro)
@@ -28,5 +28,5 @@
     <joint name="${prefix}_head_camera_joint" type="fixed">
       <!-- <origin xyz="0 ${asus_xtion_pro_cam_rel_rgb_py} 0" rpy="0.0 0.0 0.0"/> -->
-      <origin xyz="${-asus_xtion_pro_cam_rel_rgb_py} 0 -0.019" rpy="0.0 0.0 0.0"/>
+      <origin xyz="0.01 -0.0005 0.015" rpy="${-M_PI/2.0} 0.0 ${-M_PI/2.0}"/>
       <parent link="${parent}"/>
       <child link="${prefix}_link"/>
