Commit message: update/new_properties

File: sobit_pro_description/urdf/common.xacro (robot description, xacro)
@@ -2,5 +2,5 @@
 <robot xmlns:xacro="http://www.ros.org/wiki.xacro">
   <xacro:property name="M_PI" value="3.14159265359" />
-  <macro name="position_joint_transmission" params="joint reduction">
+  <xacro:macro name="position_joint_transmission" params="joint reduction">
     <transmission name="${joint}_transmission">
       <type>transmission_interface/SimpleTransmission</type>
@@ -13,4 +13,4 @@
       </actuator>
     </transmission>
-  </macro>
+  </xacro:macro>
 </robot>

File: sobit_pro_description/urdf/materials.urdf.xacro (robot description, xacro)
@@ -16,3 +16,9 @@
     <color rgba="0.0 0.0 1.0 1.0" />
   </material>
+  <material name="aluminum">
+    <color rgba="0.5 0.5 0.5 1"/>
+  </material>
+  <material name="plastic">
+    <color rgba="0.1 0.1 0.1 1"/>
+  </material>
 </robot>
