Commit message: [ADD] Multi robot support dxl parameters

File: sobit_pro_description/urdf/controllers.urdf.xacro (robot description, xacro)
@@ -9,5 +9,5 @@
         <xacro:unless value="${$(arg enable_gz)}">
           <plugin>dynamixel_hardware/DynamixelHardware</plugin>
-          <param name="usb_port">/dev/ttyUSB0</param>
+          <param name="port_name">/dev/ttyUSB0</param>
           <param name="baud_rate">1000000</param>
           <!-- <param name="protocol_version">2.0</param> -->
@@ -15,8 +15,10 @@
         </xacro:unless>
       </hardware>
-      <!-- Arm joints -->
+       <!-- Position Drive - Arm -->
       <joint name="arm_shoulder_1_tilt_joint">
         <xacro:unless value="${$(arg enable_gz)}">
           <param name="id">11</param>
+          <param name="control_mode">0</param>
+          <param name="interface">rs</param>
         </xacro:unless>
         <command_interface name="position">
@@ -34,4 +36,6 @@
         <xacro:unless value="${$(arg enable_gz)}">
           <param name="id">12</param>
+          <param name="control_mode">0</param>
+          <param name="interface">rs</param>
         </xacro:unless>
         <command_interface name="position">
@@ -49,4 +53,6 @@
         <xacro:unless value="${$(arg enable_gz)}">
           <param name="id">13</param>
+          <param name="control_mode">0</param>
+          <param name="interface">rs</param>
         </xacro:unless>
         <command_interface name="position">
@@ -64,4 +70,6 @@
         <xacro:unless value="${$(arg enable_gz)}">
           <param name="id">14</param>
+          <param name="control_mode">0</param>
+          <param name="interface">rs</param>
         </xacro:unless>
         <command_interface name="position">
@@ -79,4 +87,6 @@
         <xacro:unless value="${$(arg enable_gz)}">
           <param name="id">15</param>
+          <param name="control_mode">0</param>
+          <param name="interface">rs</param>
         </xacro:unless>
         <command_interface name="position">
@@ -94,4 +104,6 @@
         <xacro:unless value="${$(arg enable_gz)}">
           <param name="id">16</param>
+          <param name="control_mode">0</param>
+          <param name="interface">rs</param>
         </xacro:unless>
         <command_interface name="position">
@@ -109,4 +121,6 @@
         <xacro:unless value="${$(arg enable_gz)}">
           <param name="id">17</param>
+          <param name="control_mode">0</param>
+          <param name="interface">rs</param>
         </xacro:unless>
         <command_interface name="position">
@@ -121,7 +135,12 @@
         <state_interface name="effort"/>
       </joint>
+      <!-- Position Drive: Hand -->
       <joint name="hand_joint">
         <xacro:unless value="${$(arg enable_gz)}">
           <param name="id">18</param>
+          <param name="control_mode">6</param>
+          <param name="Goal_Current">50</param>  <!-- TODO: Check correct goal value -->
+          <param name="interface">rs</param>
+          <param name="gear_ratio">-59.504383354</param>  <!-- TODO: Check correct gear_ratio value -->
         </xacro:unless>
         <command_interface name="position">
@@ -136,7 +155,10 @@
         <state_interface name="effort"/>
       </joint>
+      <!-- Position Drive: Head -->
       <joint name="head_pan_joint">
         <xacro:unless value="${$(arg enable_gz)}">
           <param name="id">21</param>
+          <param name="control_mode">0</param>
+          <param name="interface">rs</param>
         </xacro:unless>
         <command_interface name="position">
@@ -154,20 +176,24 @@
         <xacro:unless value="${$(arg enable_gz)}">
           <param name="id">22</param>
-        </xacro:unless>
-        <command_interface name="position">
-          <param name="min">-1.570796327</param>
-          <param name="max">1.570796327</param>
-        </command_interface>
-        <!-- <command_interface name="velocity"/> -->
-        <state_interface name="position">
-          <param name="initial_value">0.0</param>
-        </state_interface>
-        <state_interface name="velocity"/>
-        <state_interface name="effort"/>
-      </joint>
-      <!-- Wheel joints -->
+          <param name="control_mode">0</param>
+          <param name="interface">rs</param>
+        </xacro:unless>
+        <command_interface name="position">
+          <param name="min">-1.570796327</param>
+          <param name="max">1.570796327</param>
+        </command_interface>
+        <!-- <command_interface name="velocity"/> -->
+        <state_interface name="position">
+          <param name="initial_value">0.0</param>
+        </state_interface>
+        <state_interface name="velocity"/>
+        <state_interface name="effort"/>
+      </joint>
+      <!-- Position Drive: Wheels -->
       <joint name="wheel_f_r_steer_joint">
         <xacro:unless value="${$(arg enable_gz)}">
           <param name="id">5</param>
+          <param name="control_mode">0</param>
+          <param name="interface">rs</param>
         </xacro:unless>
         <command_interface name="position">
@@ -185,4 +211,6 @@
         <xacro:unless value="${$(arg enable_gz)}">
           <param name="id">6</param>
+          <param name="control_mode">0</param>
+          <param name="interface">rs</param>
         </xacro:unless>
         <command_interface name="position">
@@ -200,4 +228,6 @@
         <xacro:unless value="${$(arg enable_gz)}">
           <param name="id">7</param>
+          <param name="control_mode">0</param>
+          <param name="interface">rs</param>
         </xacro:unless>
         <command_interface name="position">
@@ -215,4 +245,6 @@
         <xacro:unless value="${$(arg enable_gz)}">
           <param name="id">8</param>
+          <param name="control_mode">0</param>
+          <param name="interface">rs</param>
         </xacro:unless>
         <command_interface name="position">
@@ -230,4 +262,6 @@
         <xacro:unless value="${$(arg enable_gz)}">
           <param name="id">1</param>
+          <param name="control_mode">1</param>
+          <param name="interface">rs</param>
         </xacro:unless>
         <command_interface name="velocity"/>
@@ -238,4 +272,6 @@
         <xacro:unless value="${$(arg enable_gz)}">
           <param name="id">2</param>
+          <param name="control_mode">1</param>
+          <param name="interface">rs</param>
         </xacro:unless>
         <command_interface name="velocity"/>
@@ -246,4 +282,6 @@
         <xacro:unless value="${$(arg enable_gz)}">
           <param name="id">3</param>
+          <param name="control_mode">1</param>
+          <param name="interface">rs</param>
         </xacro:unless>
         <command_interface name="velocity"/>
@@ -254,4 +292,6 @@
         <xacro:unless value="${$(arg enable_gz)}">
           <param name="id">4</param>
+          <param name="control_mode">1</param>
+          <param name="interface">rs</param>
         </xacro:unless>
         <command_interface name="velocity"/>

Commit message: [ADD] New mimic parameters for SOBIT PRO hand

File: sobit_pro_description/urdf/controllers.urdf.xacro (robot description, xacro)
@@ -155,4 +155,51 @@
         <state_interface name="effort"/>
       </joint>
+      <xacro:if value="${$(arg enable_gz)}">
+        <joint name="hand_inner_l_joint">
+          <param name="mimic">hand_joint</param>
+          <param name="multiplier">-1</param>
+          <command_interface name="position"/>
+          <!-- <command_interface name="velocity"/> -->
+          <state_interface name="position"/>
+          <state_interface name="velocity"/>
+          <state_interface name="effort"/>
+        </joint>
+          <!-- Outer Left -->
+        <joint name="hand_outer_l_joint">
+          <param name="mimic">hand_joint</param>
+          <param name="multiplier">-1</param> <!-- flip if needed -->
+          <command_interface name="position"/>
+          <state_interface name="position"/>
+          <state_interface name="velocity"/>
+          <state_interface name="effort"/>
+        </joint>
+        <!-- Outer Right -->
+        <joint name="hand_outer_r_joint">
+          <param name="mimic">hand_joint</param>
+          <param name="multiplier">1</param> <!-- same direction as hand_joint -->
+          <command_interface name="position"/>
+          <state_interface name="position"/>
+          <state_interface name="velocity"/>
+          <state_interface name="effort"/>
+      </joint>
+                <!-- Outer Left -->
+        <joint name="hand_finger_l_joint">
+          <param name="mimic">hand_joint</param>
+          <param name="multiplier">-0.5</param> <!-- flip if needed -->
+          <command_interface name="position"/>
+          <state_interface name="position"/>
+          <state_interface name="velocity"/>
+          <state_interface name="effort"/>
+        </joint>
+        <!-- Outer Right -->
+        <joint name="hand_finger_r_joint">
+          <param name="mimic">hand_joint</param>
+          <param name="multiplier">0.5</param> <!-- same direction as hand_joint -->
+          <command_interface name="position"/>
+          <state_interface name="position"/>
+          <state_interface name="velocity"/>
+          <state_interface name="effort"/>
+      </joint>
+      </xacro:if>
       <!-- Position Drive: Head -->
       <joint name="head_pan_joint">

File: sobit_pro_description/urdf/hand/hand.urdf.xacro (robot description, xacro)
@@ -3,5 +3,10 @@
        xmlns:xacro="http://ros.org/wiki/xacro" >
   <xacro:include filename="$(find sobit_pro_description)/urdf/hand/hand.transmission.xacro" />
-  <xacro:macro name="hand" params="prefix_hand prefix_finger parent">
+  <xacro:macro name="hand" params="prefix_hand prefix_finger parent
+                                   enable_inner_l:=true
+                                 enable_outer_l:=true
+                                 enable_outer_r:=true
+                                 enable_fingers:=true">
+    <!-- Joint: Hand base-->
     <joint name="${prefix_hand}_base_joint" type="fixed">
       <parent link="${parent}" />
@@ -31,10 +36,13 @@
       </inertial>
     </link>
-    <joint name="${prefix_hand}_inner_l_joint" type="continuous">
+<xacro:if value="${enable_inner_l}">
+    <joint name="${prefix_hand}_inner_l_joint" type="revolute">
       <parent link="${prefix_hand}_base_link" />
       <child link="${prefix_hand}_inner_l_link" />
       <origin xyz="0.0631932 0.0151495 0.0372231" rpy="0.0 0.0 0.0" />
       <axis xyz="0.0 0.0 1.0" />
-      <mimic joint="${prefix_hand}_joint" multiplier="-1.0" offset="0" />
+      <limit lower="0" upper="${M_PI/2.0}" effort="1.0" velocity="2.0"/>
+      <mimic joint="${prefix_hand}_joint" multiplier="1" offset="0" />
+      <!-- <dynamics damping="50.0" friction="5.0"/> -->
     </joint>
     <link name="${prefix_hand}_inner_l_link">
@@ -60,4 +68,5 @@
       </inertial>
     </link>
+    </xacro:if>
     <joint name="${prefix_hand}_joint" type="revolute">
       <parent link="${prefix_hand}_base_link" />
@@ -65,5 +74,5 @@
       <origin xyz="0.0631932 -0.0151495 0.0372231" rpy="0.0 0.0 0.0" />
       <axis xyz="0.0 0.0 1.0" />
-      <limit lower="${-M_PI/2.0}" upper="0" effort="4.1" velocity="4.796165" />
+      <limit lower="${-M_PI/2.0}" upper="0" effort="1.0" velocity="2.0" />
     </joint>
     <link name="${prefix_hand}_link">
@@ -89,4 +98,5 @@
       </inertial>
     </link>
+<xacro:if value="${enable_outer_l}">
     <joint name="${prefix_hand}_outer_l_joint" type="continuous">
       <parent link="${prefix_hand}_base_link" />
@@ -94,5 +104,6 @@
       <origin xyz="0.043193 0.04015 0.0282231" rpy="0.0 0.0 0.0" />
       <axis xyz="0.0 0.0 1.0" />
-      <mimic joint="${prefix_hand}_inner_l_joint" multiplier="1.0" offset="0" />
+      <!-- <mimic joint="{prefix_hand}_joint" multiplier="1.0" offset="0" /> -->
+      <limit lower="0" upper="${M_PI/2.0}" effort="1.0" velocity="2.0"/>
     </joint>
     <link name="${prefix_hand}_outer_l_link">
@@ -118,9 +129,12 @@
       </inertial>
     </link>
-    <joint name="${prefix_hand}_outer_r_joint" type="continuous">
+  </xacro:if>
+<xacro:if value="${enable_outer_r}">
+    <joint name="${prefix_hand}_outer_r_joint" type="revolute">
       <parent link="${prefix_hand}_base_link" />
       <child link="${prefix_hand}_outer_r_link" />
       <origin xyz="0.043193 -0.04015 0.0282231" rpy="0.0 0.0 0.0" />
       <axis xyz="0.0 0.0 1.0" />
+      <limit lower="${-M_PI/2.0}" upper="0" effort="1.0" velocity="2.0"/>
       <mimic joint="${prefix_hand}_joint" multiplier="1.0" offset="0" />
     </joint>
@@ -147,5 +161,7 @@
       </inertial>
     </link>
-    <joint name="${prefix_hand}_${prefix_finger}_l_joint" type="continuous">
+  </xacro:if>
+<xacro:if value="${enable_fingers}">
+    <joint name="${prefix_hand}_${prefix_finger}_l_joint" type="revolute">
       <parent link="${prefix_hand}_inner_l_link" />
       <child link="${prefix_hand}_${prefix_finger}_l_link" />
@@ -153,4 +169,6 @@
       <axis xyz="0.0 0.0 1.0" />
       <mimic joint="${prefix_hand}_joint" multiplier="1.0" offset="0" />
+      <limit lower="${-M_PI/2.0}" upper="0" effort="4.1" velocity="4" />
+      <!-- <dynamics damping="0.05" friction="0.0"/> -->
     </joint>
     <link name="${prefix_hand}_${prefix_finger}_l_link">
@@ -176,5 +194,5 @@
       </inertial>
     </link>
-    <joint name="${prefix_hand}_${prefix_finger}_r_joint" type="continuous">
+    <joint name="${prefix_hand}_${prefix_finger}_r_joint" type="revolute">
       <parent link="${prefix_hand}_link" />
       <child link="${prefix_hand}_${prefix_finger}_r_link" />
@@ -182,4 +200,6 @@
       <axis xyz="0.0 0.0 1.0" />
       <mimic joint="${prefix_hand}_joint" multiplier="-1.0" offset="0" />
+      <limit lower="0" upper="${M_PI/2.0}" effort="4.1" velocity="1" />
+      <!-- <dynamics damping="50.0" friction="5.0"/> -->
     </joint>
     <link name="${prefix_hand}_${prefix_finger}_r_link">
@@ -205,4 +225,5 @@
       </inertial>
     </link>
+   </xacro:if>
     <xacro:hand_transmission prefix_hand="${prefix_hand}" prefix_finger="${prefix_finger}" />
   </xacro:macro>

Commit message: [FIX] ign to gz

File: sobit_pro_description/urdf/controllers.urdf.xacro (robot description, xacro)
@@ -5,5 +5,4 @@
       <hardware>
         <xacro:if value="${$(arg enable_gz)}">
-          <!-- <plugin>ign_ros2_control/IgnitionSystem</plugin> -->
           <plugin>gz_ros2_control/GazeboSimSystem</plugin>
         </xacro:if>
@@ -157,18 +156,18 @@
           <state_interface name="effort"/>
         </joint>
-        <xacro:if value="${$(arg enable_gz)}">
+        <!-- <xacro:if value="${$(arg enable_gz)}"> TODO
           <joint name="hand_inner_l_joint">
             <param name="mimic">hand_joint</param>
             <param name="multiplier">-1</param>
             <command_interface name="position"/>
-            <!-- <command_interface name="velocity"/> -->
+            <command_interface name="velocity"/>
             <state_interface name="position"/>
             <state_interface name="velocity"/>
             <state_interface name="effort"/>
           </joint>
-            <!-- Outer Left -->
+            Outer Left
           <joint name="hand_outer_l_joint">
             <param name="mimic">hand_joint</param>
-            <param name="multiplier">-1</param> <!-- flip if needed -->
+            <param name="multiplier">-1</param> flip if needed
             <command_interface name="position"/>
             <state_interface name="position"/>
@@ -176,17 +175,17 @@
             <state_interface name="effort"/>
           </joint>
-          <!-- Outer Right -->
+          Outer Right
           <joint name="hand_outer_r_joint">
             <param name="mimic">hand_joint</param>
-            <param name="multiplier">1</param> <!-- same direction as hand_joint -->
-            <command_interface name="position"/>
-            <state_interface name="position"/>
-            <state_interface name="velocity"/>
-            <state_interface name="effort"/>
-        </joint>
-                  <!-- Outer Left -->
+            <param name="multiplier">1</param> same direction as hand_joint
+            <command_interface name="position"/>
+            <state_interface name="position"/>
+            <state_interface name="velocity"/>
+            <state_interface name="effort"/>
+        </joint>
+                  Outer Left
           <joint name="hand_finger_l_joint">
             <param name="mimic">hand_joint</param>
-            <param name="multiplier">-0.5</param> <!-- flip if needed -->
+            <param name="multiplier">-0.5</param> flip if needed
             <command_interface name="position"/>
             <state_interface name="position"/>
@@ -194,14 +193,14 @@
             <state_interface name="effort"/>
           </joint>
-          <!-- Outer Right -->
+          Outer Right
           <joint name="hand_finger_r_joint">
             <param name="mimic">hand_joint</param>
-            <param name="multiplier">0.5</param> <!-- same direction as hand_joint -->
-            <command_interface name="position"/>
-            <state_interface name="position"/>
-            <state_interface name="velocity"/>
-            <state_interface name="effort"/>
-        </joint>
-        </xacro:if>
+            <param name="multiplier">0.5</param> same direction as hand_joint
+            <command_interface name="position"/>
+            <state_interface name="position"/>
+            <state_interface name="velocity"/>
+            <state_interface name="effort"/>
+        </joint>
+        </xacro:if> -->
       </xacro:if>
       <!-- Position Drive: Head -->
@@ -357,5 +356,4 @@
     <xacro:if value="${$(arg enable_gz)}">
       <gazebo>
-        <!-- <plugin filename="ign_ros2_control-system" name="ign_ros2_control::IgnitionROS2ControlPlugin"> -->
         <plugin filename="gz_ros2_control-system" name="gz_ros2_control::GazeboSimROS2ControlPlugin">
           <ros>

File: sobit_pro_description/urdf/gazebo.urdf.xacro (robot description, xacro)
@@ -8,7 +8,6 @@
         <sensor name="head_camera_color" type="camera">
           <pose>0.0 0.0 ${0.0175/2} ${M_PI/2} -${M_PI/2} 0.0</pose>
-          <!-- <ignition_frame_id>${robot_name}/head_camera_link</ignition_frame_id> -->
           <gz_frame_id>${robot_name}/head_camera_link</gz_frame_id>
-          <topic>${robot_name}/head_camera/rgb/image_raw</topic>
+          <topic>${robot_name}/head_camera/color</topic>
           <always_on>1</always_on>
           <visualize>true</visualize>
@@ -34,7 +33,6 @@
         <sensor name="head_camera_depth" type="depth">
           <pose>0.0 0.0 ${0.0175/2} ${M_PI/2} -${M_PI/2} 0.0</pose>
-          <!-- <ignition_frame_id>${robot_name}/head_camera_link</ignition_frame_id> -->
           <gz_frame_id>${robot_name}/head_camera_link</gz_frame_id>
-          <topic>${robot_name}/head_camera/depth_registered/image_raw</topic>
+          <topic>${robot_name}/head_camera/depth</topic>
           <always_on>1</always_on>
           <visualize>true</visualize>
@@ -59,5 +57,4 @@
         <sensor name="lidar" type="gpu_lidar">
           <pose>0 0 0 0 0 0</pose>
-          <!-- <ignition_frame_id>${robot_name}/lidar_laser</ignition_frame_id> -->
           <gz_frame_id>${robot_name}/lidar_laser</gz_frame_id>
           <!-- <qos>
