Commit message: Enhance simulation parameters and configurations for Gazebo integration
- Updated .gitignore to include Python bytecode files.
- Added angular_z_sign parameter to manage cmd_vel angular.z sign in simulation.
- Adjusted P-gain for position-commanded joints in controllers.yaml for better control.
- Modified robot.launch.py to include comments clarifying Gazebo to ROS message bridging.
- Cleaned up controllers.urdf.xacro by removing unnecessary mimic joint parameters.
- Increased physics simulation step size in empty_w_physics.sdf for improved performance.

File: sobit_pro_description/urdf/controllers.urdf.xacro (robot description, xacro)
@@ -164,51 +164,34 @@
           <state_interface name="effort"/>
         </joint>
-        <!-- <xacro:if value="${$(arg enable_gz)}"> TODO
+        <!-- Passive mimic finger joints (gz only): dartsim cannot create
+             mimic constraints from the SDF, so without this the fingers are
+             completely uncontrolled and sag open under gravity. Registering
+             them state-only lets gz_ros2_control detect the URDF <mimic>
+             tag (multiplier/offset included) and enforce the coupling
+             itself. The real robot has a physical linkage, so this section
+             must stay gz-only. Command interfaces are intentionally absent:
+             ros2_control rejects mimic joints that declare them. -->
+        <xacro:if value="${$(arg enable_gz)}">
           <joint name="hand_inner_l_joint">
-            <param name="mimic">hand_joint</param>
-            <param name="multiplier">-1</param>
-            <command_interface name="position"/>
-            <command_interface name="velocity"/>
-            <state_interface name="position"/>
-            <state_interface name="velocity"/>
-            <state_interface name="effort"/>
-          </joint>
-            Outer Left
+            <state_interface name="position"/>
+            <state_interface name="velocity"/>
+          </joint>
           <joint name="hand_outer_l_joint">
-            <param name="mimic">hand_joint</param>
-            <param name="multiplier">-1</param> flip if needed
-            <command_interface name="position"/>
-            <state_interface name="position"/>
-            <state_interface name="velocity"/>
-            <state_interface name="effort"/>
-          </joint>
-          Outer Right
+            <state_interface name="position"/>
+            <state_interface name="velocity"/>
+          </joint>
           <joint name="hand_outer_r_joint">
-            <param name="mimic">hand_joint</param>
-            <param name="multiplier">1</param> same direction as hand_joint
-            <command_interface name="position"/>
-            <state_interface name="position"/>
-            <state_interface name="velocity"/>
-            <state_interface name="effort"/>
-        </joint>
-                  Outer Left
+            <state_interface name="position"/>
+            <state_interface name="velocity"/>
+          </joint>
           <joint name="hand_finger_l_joint">
-            <param name="mimic">hand_joint</param>
-            <param name="multiplier">-0.5</param> flip if needed
-            <command_interface name="position"/>
-            <state_interface name="position"/>
-            <state_interface name="velocity"/>
-            <state_interface name="effort"/>
-          </joint>
-          Outer Right
+            <state_interface name="position"/>
+            <state_interface name="velocity"/>
+          </joint>
           <joint name="hand_finger_r_joint">
-            <param name="mimic">hand_joint</param>
-            <param name="multiplier">0.5</param> same direction as hand_joint
-            <command_interface name="position"/>
-            <state_interface name="position"/>
-            <state_interface name="velocity"/>
-            <state_interface name="effort"/>
-        </joint>
-        </xacro:if> -->
+            <state_interface name="position"/>
+            <state_interface name="velocity"/>
+          </joint>
+        </xacro:if>
       </xacro:if>
       <!-- Position Drive: Head -->
