Commit message: azure_kinectのurdfの連携処理を追加

File: sobit_pro_description/robots/sobit_pro.urdf.xacro (robot description, xacro)
@@ -11,11 +11,4 @@
   <xacro:include filename="$(find sobit_pro_description)/urdf/head/head.urdf.xacro" />
   <xacro:include filename="$(find sobit_pro_description)/urdf/sensor/azure_kinect.urdf.xacro" />
-  <!--
-  <xacro:include filename="$(find sobit_pro_description)/urdf/arm/arm.urdf.xacro" />
-  <xacro:include filename="$(find sobit_pro_description)/urdf/gripper/gripper.urdf.xacro" />
-  <xacro:include filename="$(find sobit_pro_description)/urdf/head/head.urdf.xacro" />
-  <xacro:include filename="$(find sobit_pro_description)/urdf/pole/pole.urdf.xacro" />
-  <xacro:include filename="$(find sobit_pro_description)/urdf/sensor/sensor.urdf.xacro" />
-  -->
   <xacro:base/>
   <xacro:wheel parent="base_link" />
@@ -24,14 +17,3 @@
   <xacro:head prefix="head_camera" parent="base_link" />
   <xacro:azure_kinect prefix="head_camera" parent="head_camera_tilt_link" />
-  <!--
-  <stack_hexagons parent="base_link" />
-  <xacro:arm prefix="arm" parent="plate_top_link"/>
-  <xacro:hand prefix="hand_motor" parent="wrist_flex_link"/>
-  <xacro:pole parent="plate_top_link"/>
-  <xacro:xtion_motor prefix="xtion" parent="base_pole_link"/>
-  <xacro:sensor_asus_xtion_pro parent="xtion_double_sided_tape_link"/>
-  <xacro:mic parent="base_pole_link"/>
-  <xacro:matrix parent="base_pole_link"/>
-  <xacro:urg parent="base_link"/>
-  -->
 </robot>

File: sobit_pro_description/urdf/sensor/azure_kinect.urdf.xacro (robot description, xacro)
@@ -16,4 +16,22 @@
       </visual>
     </link>
+    <joint name="${prefix}_base_joint" type="fixed">
+      <parent link="${prefix}_link" />
+      <child link="${prefix}_base" />
+      <origin xyz="0. -0.055 0.04" rpy="0. 0. ${-M_PI / 2}" />
+    </joint>
+    <link name="${prefix}_body" />
+    <joint name="${prefix}_base_to_body" type="fixed">
+      <parent link="${prefix}_base" />
+      <child link="${prefix}_body" />
+      <origin xyz="-0.0757 0. 0.008" rpy="0. 0. 0." />
+    </joint>
+    <link name="${prefix}_base" />
+    <joint name="${prefix}_base_to_visor" type="fixed">
+      <parent link="${prefix}_base" />
+      <child link="${prefix}_visor" />
+      <origin xyz="0. 0. 0." rpy="0. 0. 0." />
+    </joint>
+    <link name="${prefix}_visor" />
   </xacro:macro>
 </robot>

Commit message: update/l515_xaxro

File: sobit_pro_description/robots/sobit_pro.urdf.xacro (robot description, xacro)
@@ -12,4 +12,5 @@
   <xacro:include filename="$(find sobit_pro_description)/urdf/sensor/azure_kinect.urdf.xacro" />
   <xacro:include filename="$(find sobit_pro_description)/urdf/sensor/urg.urdf.xacro" />
+  <xacro:include filename="$(find sobit_pro_description)/urdf/sensor/realsense_l515.urdf.xacro" />
   <!--
   <xacro:include filename="$(find sobit_pro_description)/urdf/arm/arm.urdf.xacro" />
@@ -26,4 +27,7 @@
   <xacro:azure_kinect prefix="head_camera" parent="head_camera_tilt_link" />
   <xacro:urg parent="base_link"/>
+  <xacro:realsense_l515 parent="arm4_link" name="camera_l515" use_nominal_extrinsics="false" add_plug="false" use_mesh="true">
+    <origin xyz="0 -0.10 -0.03" rpy="0 0 -${M_PI/2.0}"/>
+  </xacro:realsense_l515>
   <!--
   <stack_hexagons parent="base_link" />

Commit message: add : realsense

File: sobit_pro_description/robots/sobit_pro.urdf.xacro (robot description, xacro)
@@ -27,6 +27,6 @@
   <xacro:azure_kinect prefix="head_camera" parent="head_camera_tilt_link" />
   <xacro:urg parent="base_link"/>
-  <xacro:realsense_l515 parent="arm4_link" name="camera_l515" use_nominal_extrinsics="false" add_plug="false" use_mesh="true">
-    <origin xyz="0 -0.10 -0.03" rpy="0 0 -${M_PI/2.0}"/>
+  <xacro:realsense_l515 parent="arm4_link" name="camera_l515" use_nominal_extrinsics="true" add_plug="false" use_mesh="true">
+    <origin xyz="0 -0.09625 -0.0305" rpy="0 0 -${M_PI/2.0}"/>
   </xacro:realsense_l515>
   <!--

Commit message: update robots urdf

File: sobit_pro_description/robots/sobit_pro.urdf.xacro (robot description, xacro)
@@ -1,43 +1,35 @@
 <?xml version="1.0" ?>
 <robot name="sobit_pro" xmlns:controller="http://playerstage.sourceforge.net/gazebo/xmlschema/#controller" xmlns:interface="http://playerstage.sourceforge.net/gazebo/xmlschema/#interface" xmlns:sensor="http://playerstage.sourceforge.net/gazebo/xmlschema/#sensor" xmlns:xacro="http://www.ros.org/wiki/xacro">
-  <!-- common xacro -->
+  <!-- Add Common Xacro: transmissions, colors -->
   <xacro:include filename="$(find sobit_pro_description)/urdf/common.xacro" />
   <xacro:include filename="$(find sobit_pro_description)/urdf/materials.urdf.xacro" />
-  <!-- links and joints -->
+  <!-- Add URDF: links, joints -->
   <xacro:include filename="$(find sobit_pro_description)/urdf/base/base.urdf.xacro" />
+  <xacro:include filename="$(find sobit_pro_description)/urdf/body/plate.urdf.xacro" />
+  <xacro:include filename="$(find sobit_pro_description)/urdf/body/cover.urdf.xacro" />
+  <xacro:include filename="$(find sobit_pro_description)/urdf/back/back.urdf.xacro" />
   <xacro:include filename="$(find sobit_pro_description)/urdf/wheel/wheel.urdf.xacro" />
   <xacro:include filename="$(find sobit_pro_description)/urdf/arm/arm.urdf.xacro" />
-  <xacro:include filename="$(find sobit_pro_description)/urdf/gripper/gripper.urdf.xacro" />
+  <xacro:include filename="$(find sobit_pro_description)/urdf/hand/hand.urdf.xacro" />
   <xacro:include filename="$(find sobit_pro_description)/urdf/head/head.urdf.xacro" />
   <xacro:include filename="$(find sobit_pro_description)/urdf/sensor/azure_kinect.urdf.xacro" />
-  <xacro:include filename="$(find sobit_pro_description)/urdf/sensor/urg.urdf.xacro" />
+  <xacro:include filename="$(find sobit_pro_description)/urdf/sensor/matrix.urdf.xacro" />
+  <xacro:include filename="$(find sobit_pro_description)/urdf/sensor/mic.urdf.xacro" />
+  <xacro:include filename="$(find sobit_pro_description)/urdf/sensor/lidar.urdf.xacro" />
   <xacro:include filename="$(find sobit_pro_description)/urdf/sensor/realsense_l515.urdf.xacro" />
-  <!--
-  <xacro:include filename="$(find sobit_pro_description)/urdf/arm/arm.urdf.xacro" />
-  <xacro:include filename="$(find sobit_pro_description)/urdf/gripper/gripper.urdf.xacro" />
-  <xacro:include filename="$(find sobit_pro_description)/urdf/head/head.urdf.xacro" />
-  <xacro:include filename="$(find sobit_pro_description)/urdf/pole/pole.urdf.xacro" />
-  <xacro:include filename="$(find sobit_pro_description)/urdf/sensor/sensor.urdf.xacro" />
-  -->
+  <xacro:include filename="$(find urg_node)/urdf/hokuyo_ust.urdf.xacro" />
+  <xacro:include filename="$(find realsense2_description)/urdf/_l515.urdf.xacro" />
   <xacro:base/>
-  <xacro:wheel parent="base_link" />
-  <xacro:arm prefix="arm" parent="base_link" />
-  <xacro:gripper prefix_grip="gripper" prefix_finger="finger" parent="arm4_link" />
-  <xacro:head prefix="head_camera" parent="base_link" />
+  <xacro:plate prefix="plate" parent="base_link" />
+  <xacro:wheel prefix="wheel" parent="plate_middle_link" />
+  <xacro:cover prefix="cover" parent="plate_top_link" />
+  <xacro:back  prefix="back" parent="plate_top_link" />
+  <xacro:head  prefix="head" parent="back_base_link" />
+  <xacro:mic   prefix="mic"  parent="back_base_link" />
+  <xacro:arm   prefix="arm"  parent="plate_top_link" />
+  <xacro:hand  prefix_hand="hand" prefix_finger="finger" parent="arm_wrist_tilt_link" />
+  <xacro:lidar prefix="lidar" parent="plate_bottom_link" />
   <xacro:azure_kinect prefix="head_camera" parent="head_camera_tilt_link" />
-  <xacro:urg parent="base_link"/>
-  <xacro:realsense_l515 parent="arm4_link" name="camera_l515" use_nominal_extrinsics="true" add_plug="false" use_mesh="true">
-    <origin xyz="0 -0.09625 -0.0305" rpy="0 0 -${M_PI/2.0}"/>
-  </xacro:realsense_l515>
-  <!--
-  <stack_hexagons parent="base_link" />
-  <xacro:arm prefix="arm" parent="plate_top_link"/>
-  <xacro:hand prefix="hand_motor" parent="wrist_flex_link"/>
-  <xacro:pole parent="plate_top_link"/>
-  <xacro:xtion_motor prefix="xtion" parent="base_pole_link"/>
-  <xacro:sensor_asus_xtion_pro parent="xtion_double_sided_tape_link"/>
-  <xacro:mic parent="base_pole_link"/>
-  <xacro:matrix parent="base_pole_link"/>
-  <xacro:urg parent="base_link"/>
-  -->
+  <xacro:matrix prefix="matrix" parent="head_camera_link" />
+  <xacro:realsense_l515 prefix="hand_camera" parent="arm_wrist_tilt_link" />
 </robot>

Commit message: update urdf

File: sobit_pro_description/robots/sobit_pro.urdf.xacro (robot description, xacro)
@@ -34,5 +34,5 @@
   <xacro:lidar prefix="lidar" parent="plate_bottom_link" />
   <xacro:azure_camera prefix="head_camera" parent="head_camera_tilt_link" />
-  <xacro:matrix prefix="matrix" parent="head_camera_link" />
+  <xacro:matrix prefix="matrix" parent="head_camera_base" />
   <!-- <xacro:realsense_l515 prefix="hand_camera" parent="arm_wrist_tilt_link" /> -->
   <xacro:realsense_d405 prefix="hand_camera" parent="arm_wrist_tilt_link" />

File: sobit_pro_description/urdf/sensor/azure_camera.urdf.xacro (robot description, xacro)
@@ -4,9 +4,9 @@
     <joint name="${prefix}_joint" type="fixed">
       <parent link="${parent}" />
-      <child link="${prefix}_link" />
+      <child link="${prefix}_base" />
       <origin xyz="-0.0065 0.0 0.0395" rpy="0.0 0.0 0.0" />
     </joint>
-    <link name="${prefix}_link"/>
-    <xacro:azure_kinect parent="${prefix}_link" tf_prefix="${prefix}_" add_cover="false">
+    <link name="${prefix}_base"/>
+    <xacro:azure_kinect parent="${prefix}_base" tf_prefix="${prefix}_" add_cover="false">
       <origin xyz="0.0 0 0.0" rpy="0 0 0"/>
     </xacro:azure_kinect>

Commit message: update urdf model

File: sobit_pro_description/robots/sobit_pro.urdf.xacro (robot description, xacro)
@@ -26,14 +26,14 @@
   <xacro:plate prefix="plate" parent="base_link" />
   <xacro:wheel prefix="wheel" parent="plate_middle_link" />
-  <xacro:cover prefix="cover" parent="plate_top_link" />
-  <xacro:back  prefix="back" parent="plate_top_link" />
-  <xacro:head  prefix="head" parent="back_base_link" />
-  <xacro:mic   prefix="mic"  parent="back_base_link" />
-  <xacro:arm   prefix="arm"  parent="plate_top_link" />
-  <xacro:hand  prefix_hand="hand" prefix_finger="finger" parent="arm_wrist_tilt_link" />
+  <!-- <xacro:cover prefix="cover" parent="plate_top_link" /> -->
+  <!-- <xacro:back  prefix="back" parent="plate_top_link" /> -->
+  <!-- <xacro:head  prefix="head" parent="back_base_link" /> -->
+  <!-- <xacro:mic   prefix="mic"  parent="back_base_link" /> -->
+  <!-- <xacro:arm   prefix="arm"  parent="plate_top_link" /> -->
+  <!-- <xacro:hand  prefix_hand="hand" prefix_finger="finger" parent="arm_wrist_tilt_link" /> -->
   <xacro:lidar prefix="lidar" parent="plate_bottom_link" />
-  <xacro:azure_camera prefix="head_camera" parent="head_camera_tilt_link" />
-  <xacro:matrix prefix="matrix" parent="head_camera_base" />
+  <!-- <xacro:azure_camera prefix="head_camera" parent="head_camera_tilt_link" /> -->
+  <!-- <xacro:matrix prefix="matrix" parent="head_camera_base" /> -->
   <!-- <xacro:realsense_l515 prefix="hand_camera" parent="arm_wrist_tilt_link" /> -->
-  <xacro:realsense_d405 prefix="hand_camera" parent="arm_wrist_tilt_link" />
+  <!-- <xacro:realsense_d405 prefix="hand_camera" parent="arm_wrist_tilt_link" /> -->
 </robot>

File: sobit_pro_description/urdf/body/plate.urdf.xacro (robot description, xacro)
@@ -1,5 +1,5 @@
 <?xml version="1.0" encoding="UTF-8" ?>
 <robot name="plate" xmlns:xacro="http://ros.org/wiki/xacro">
-    <xacro:macro name="plate" params="prefix parent">>
+    <xacro:macro name="plate" params="prefix parent">
     <joint name="${prefix}_bottom_joint" type="fixed">
       <origin xyz="0.0 0.0 0.0" rpy="0.0 0.0 0.0" />
@@ -56,5 +56,5 @@
       </inertial>
     </link>
-    <joint name="${prefix}_top_joint" type="fixed">
+    <!-- <joint name="${prefix}_top_joint" type="fixed">
       <origin xyz="0.0 0.0 0.4800" rpy="0.0 0.0 0.0" />
       <parent link="${prefix}_middle_link" />
@@ -82,5 +82,5 @@
                  izz="1.0" />
       </inertial>
-    </link>
+    </link> -->
     </xacro:macro>
 </robot>

Commit message: [UPD] head_camera_xxxx_->head_xxx_

File: sobit_pro_description/robots/sobit_pro.urdf.xacro (robot description, xacro)
@@ -33,5 +33,5 @@
   <xacro:hand  prefix_hand="hand" prefix_finger="finger" parent="arm_wrist_tilt_link" />
   <xacro:lidar prefix="lidar" parent="plate_bottom_link" />
-  <xacro:azure_camera prefix="head_camera" parent="head_camera_tilt_link" />
+  <xacro:azure_camera prefix="head_camera" parent="head_tilt_link" />
   <xacro:matrix prefix="matrix" parent="head_camera_base" />
   <!-- <xacro:realsense_l515 prefix="hand_camera" parent="arm_wrist_tilt_link" /> -->

File: sobit_pro_description/robots/sobit_pro_arm.urdf.xacro (robot description, xacro)
@@ -33,5 +33,5 @@
   <xacro:hand  prefix_hand="hand" prefix_finger="finger" parent="arm_wrist_tilt_link" />
   <!-- <xacro:lidar prefix="lidar" parent="plate_bottom_link" /> -->
-  <!-- <xacro:azure_camera prefix="head_camera" parent="head_camera_tilt_link" /> -->
+  <!-- <xacro:azure_camera prefix="head_camera" parent="head_tilt_link" /> -->
   <!-- <xacro:matrix prefix="matrix" parent="head_camera_base" /> -->
   <!-- <xacro:realsense_l515 prefix="hand_camera" parent="arm_wrist_tilt_link" /> -->

File: sobit_pro_description/robots/sobit_pro_arm_head.urdf.xacro (robot description, xacro)
@@ -33,5 +33,5 @@
   <xacro:hand  prefix_hand="hand" prefix_finger="finger" parent="arm_wrist_tilt_link" />
   <!-- <xacro:lidar prefix="lidar" parent="plate_bottom_link" /> -->
-  <xacro:azure_camera prefix="head_camera" parent="head_camera_tilt_link" />
+  <xacro:azure_camera prefix="head_camera" parent="head_tilt_link" />
   <xacro:matrix prefix="matrix" parent="head_camera_base" />
   <!-- <xacro:realsense_l515 prefix="hand_camera" parent="arm_wrist_tilt_link" /> -->

File: sobit_pro_description/robots/sobit_pro_arm_mb.urdf.xacro (robot description, xacro)
@@ -33,5 +33,5 @@
   <xacro:hand  prefix_hand="hand" prefix_finger="finger" parent="arm_wrist_tilt_link" />
   <xacro:lidar prefix="lidar" parent="plate_bottom_link" />
-  <!-- <xacro:azure_camera prefix="head_camera" parent="head_camera_tilt_link" /> -->
+  <!-- <xacro:azure_camera prefix="head_camera" parent="head_tilt_link" /> -->
   <!-- <xacro:matrix prefix="matrix" parent="head_camera_base" /> -->
   <!-- <xacro:realsense_l515 prefix="hand_camera" parent="arm_wrist_tilt_link" /> -->

File: sobit_pro_description/robots/sobit_pro_head_mb.urdf.xacro (robot description, xacro)
@@ -33,5 +33,5 @@
   <!-- <xacro:hand  prefix_hand="hand" prefix_finger="finger" parent="arm_wrist_tilt_link" /> -->
   <xacro:lidar prefix="lidar" parent="plate_bottom_link" />
-  <xacro:azure_camera prefix="head_camera" parent="head_camera_tilt_link" />
+  <xacro:azure_camera prefix="head_camera" parent="head_tilt_link" />
   <xacro:matrix prefix="matrix" parent="head_camera_base" />
   <!-- <xacro:realsense_l515 prefix="hand_camera" parent="arm_wrist_tilt_link" /> -->

File: sobit_pro_description/urdf/head/head.urdf.xacro (robot description, xacro)
@@ -3,10 +3,13 @@
   <xacro:include filename="$(find sobit_pro_description)/urdf/head/head.transmission.xacro" />
   <xacro:macro name="head" params="prefix parent">
-    <joint name="${prefix}_camera_base_joint" type="fixed">
+    <joint name="${prefix}_base_joint" type="fixed">
+    <!-- <joint name="${prefix}_camera_base_joint" type="fixed"> -->
       <parent link="${parent}" />
-      <child link="${prefix}_camera_base_link" />
+      <!-- <child link="${prefix}_camera_base_link" /> -->
+      <child link="${prefix}_base_link" />
       <origin xyz="0.0900 0.0 0.5270" rpy="0.0 0.0 0.0" />
     </joint>
-    <link name="${prefix}_camera_base_link">
+    <link name="${prefix}_base_link">
+    <!-- <link name="${prefix}_camera_base_link"> -->
       <visual>
         <origin xyz="0.0 0.0 0.0" rpy="${M_PI/2.0} 0.0 ${M_PI/2.0}" />
@@ -30,12 +33,16 @@
       </inertial>
     </link>
-    <joint name="${prefix}_camera_pan_joint" type="revolute">
-      <parent link="${prefix}_camera_base_link" />
-      <child link="${prefix}_camera_pan_link" />
+    <!-- <joint name="${prefix}_camera_pan_joint" type="revolute"> -->
+    <joint name="${prefix}_pan_joint" type="revolute">
+      <parent link="${prefix}_base_link" />
+      <!-- <parent link="${prefix}_camera_base_link" /> -->
+      <child link="${prefix}_pan_link" />
+      <!-- <child link="${prefix}_camera_pan_link" /> -->
       <origin xyz="0.03985 0.0 0.0190" rpy="0.0 0.0 0.0" />
       <axis xyz="0 0 1" />
       <limit effort="30" lower="${-M_PI/2.0}" upper="${M_PI/2.0}" velocity="${M_PI/2.0}" />
     </joint>
-    <link name="${prefix}_camera_pan_link">
+    <link name="${prefix}_pan_link">
+    <!-- <link name="${prefix}_camera_pan_link"> -->
       <visual>
         <origin xyz="0.0 0.0 0.0" rpy="0.0 0.0 ${M_PI/2.0}" />
@@ -59,12 +66,16 @@
       </inertial>
     </link>
-    <joint name="${prefix}_camera_tilt_joint" type="revolute">
-      <parent link="${prefix}_camera_pan_link" />
-      <child link="${prefix}_camera_tilt_link" />
+    <joint name="${prefix}_tilt_joint" type="revolute">
+    <!-- <joint name="${prefix}_camera_tilt_joint" type="revolute"> -->
+      <parent link="${prefix}_pan_link" />
+      <!-- <parent link="${prefix}_camera_pan_link" /> -->
+      <child link="${prefix}_tilt_link" />
+      <!-- <child link="${prefix}_camera_tilt_link" /> -->
       <origin xyz="0.0 0.0 0.0405" rpy="0.0 0.0 0.0" />
       <axis xyz="0 -1 0" />
       <limit effort="30" lower="${-M_PI/2.0}" upper="${M_PI/2.0}" velocity="${M_PI/2.0}" />
     </joint>
-    <link name="${prefix}_camera_tilt_link">
+    <link name="${prefix}_tilt_link">
+    <!-- <link name="${prefix}_camera_tilt_link"> -->
       <visual>
         <origin xyz="0.0 0.0 0.0" rpy="0.0 0.0 ${M_PI/2.0}" />
