Commit message: merge develop_lib

File: sobit_pro_description/robots/sobit_pro.urdf (robot description, URDF)
Before this commit: robot sobit_pro, 23 links, 22 joints
Links:
- removed link AzureKinect_link
- removed link arm_wrist_link
- removed link hand_main_l_link
- removed link hand_main_r_link
- removed link hand_sub_l_link
- removed link hand_sub_r_link
- removed link neck_link
- added link arm4_link; visual mesh filename=package://sobit_pro_description/meshes/arm/sobit_pro_arm4.d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
- added link gripper_inner_l_link; visual mesh filename=package://sobit_pro_description/meshes/gripper/sobit_pro_gr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
- added link gripper_inner_r_link; visual mesh filename=package://sobit_pro_description/meshes/gripper/sobit_pro_gr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
- added link gripper_link
- added link gripper_outer_l_link; visual mesh filename=package://sobit_pro_description/meshes/gripper/sobit_pro_gr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
- added link gripper_outer_r_link; visual mesh filename=package://sobit_pro_description/meshes/gripper/sobit_pro_gr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
- added link head_camera_link; visual mesh filename=package://sobit_pro_description/meshes/sensor/azure_kinect.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
- added link head_camera_pan_link; visual mesh filename=package://sobit_pro_description/meshes/head/sobit_pro_head_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
- added link head_camera_tilt_link
- link arm1_link: geometry visual mesh filename=package://sobit_pro_description/meshes/arm/sobit_pro_arm1.d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
- link arm2_link: geometry visual mesh filename=package://sobit_pro_description/meshes/arm/sobit_pro_arm2.d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
- link arm3_link: geometry visual mesh filename=package://sobit_pro_description/meshes/arm/sobit_pro_arm3.d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
- link arm_base_link: geometry visual mesh filename=package://sobit_pro_description/meshes/arm/sobit_pro_arm_ba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
- link base_link: geometry visual mesh filename=package://sobit_pro_description/meshes/base/sobit_pro_body.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
- link finger_l_link: geometry visual mesh filename=package://sobit_pro_description/meshes/gripper/sobit_pro_fi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
- link finger_r_link: geometry visual mesh filename=package://sobit_pro_description/meshes/gripper/sobit_pro_fi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
- link steer_b_l_link: geometry visual mesh filename=package://sobit_pro_description/meshes/wheel/sobit_pro_stee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
- link steer_b_r_link: geometry visual mesh filename=package://sobit_pro_description/meshes/wheel/sobit_pro_stee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
- link steer_f_l_link: geometry visual mesh filename=package://sobit_pro_description/meshes/wheel/sobit_pro_stee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
- link steer_f_r_link: geometry visual mesh filename=package://sobit_pro_description/meshes/wheel/sobit_pro_stee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
- link wheel_b_l_link: geometry visual mesh filename=package://sobit_pro_description/meshes/wheel/sobit_pro_whee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
- link wheel_b_r_link: geometry visual mesh filename=package://sobit_pro_description/meshes/wheel/sobit_pro_whee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
- link wheel_f_l_link: geometry visual mesh filename=package://sobit_pro_description/meshes/wheel/sobit_pro_whee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
- link wheel_f_r_link: geometry visual mesh filename=package://sobit_pro_description/meshes/wheel/sobit_pro_whee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
Joints:
- removed joint AzureKinect_joint
- removed joint arm_wrist_joint
- removed joint hand_main_l_joint
- removed joint hand_main_r_joint
- removed joint hand_sub_l_joint
- removed joint hand_sub_r_joint
- removed joint neck_joint
- added joint arm4_joint: type revolute, parent arm3_link, child arm4_link, origin xyz=0 -0.09641814 -0.11490667 rpy=0.87 0 0, axis -1 0 0, limit lower=-1.5707963268 upper=1.5707963268 effort=10 velocity=10
- added joint gripper_inner_l_joint: type revolute, parent arm4_link, child gripper_inner_l_link, origin xyz=0.015 -0.07811569 0.02333593 rpy=0 0 0, axis 0 0 1, limit lower=-1.570796327 upper=0 effort=1 velocity=1, mimic joint=gripper_joint multiplier=-1.0 offset=0
- added joint gripper_inner_r_joint: type revolute, parent arm4_link, child gripper_inner_r_link, origin xyz=-0.015 -0.07811569 0.02333593 rpy=0 0 0, axis 0 0 1, limit lower=-1.570796327 upper=0 effort=1 velocity=1, mimic joint=gripper_joint multiplier=1.0 offset=0
- added joint gripper_joint: type revolute, parent arm4_link, child gripper_link, origin xyz=0.0 0.0 0.0 rpy=0 0 0, axis 0 0 1, limit lower=-1.570796327 upper=0 effort=1 velocity=1
- added joint gripper_outer_l_joint: type revolute, parent arm4_link, child gripper_outer_l_link, origin xyz=0.04 -0.0580698 0.02333593 rpy=0 0 0, axis 0 0 1, limit lower=-1.570796327 upper=0 effort=1 velocity=1, mimic joint=gripper_joint multiplier=-1.12 offset=0
- added joint gripper_outer_r_joint: type revolute, parent arm4_link, child gripper_outer_r_link, origin xyz=-0.04 -0.0580698 0.02333593 rpy=0 0 0, axis 0 0 1, limit lower=-1.570796327 upper=0 effort=1 velocity=1, mimic joint=gripper_joint multiplier=1.12 offset=0
- added joint head_camera_joint: type fixed, parent head_camera_tilt_link, child head_camera_link, origin xyz=0 0 0 rpy=0 0 0
- added joint head_camera_pan_joint: type revolute, parent base_link, child head_camera_pan_link, origin xyz=0 -0.12985 1.117 rpy=0 0 0, axis 0 0 1, limit lower=-1.5707963268 upper=1.5707963268 effort=10 velocity=10
- added joint head_camera_tilt_joint: type revolute, parent head_camera_pan_link, child head_camera_tilt_link, origin xyz=0 0 0.041 rpy=0 0 0, axis -1 0 0, limit lower=-1.5707963268 upper=1.5707963268 effort=10 velocity=10
- joint arm1_joint: axis 1 0 0 -> -1 0 0; limit lower=0 upper=3.14 effort=10 velocity=10 -> lower=-1.5707963268 upper=1.5707963268 effort=10 velocity=10; origin xyz=0 0 0 rpy=0 0 0 -> xyz=0 0 0 rpy=1.5707963268 0 0
- joint arm2_joint: axis 1 0 0 -> -1 0 0; limit lower=-2.2 upper=0.42 effort=10 velocity=10 -> lower=-1.5707963268 upper=1.5707963268 effort=10 velocity=10; origin xyz=0 0 0.15 rpy=0 0 0 -> xyz=0 0 0.15 rpy=-1.137 0 0
- joint arm3_joint: axis 1 0 0 -> -1 0 0; limit lower=-2.5 upper=0.36 effort=10 velocity=10 -> lower=-1.5707963268 upper=1.5707963268 effort=10 velocity=10; origin xyz=0 -0.13594617 0.06339274 rpy=0 0 0 -> xyz=0 -0.13594617 0.06339274 rpy=-1.30 0 0
- joint finger_l_joint: mimic joint=hand_main_r_joint multiplier=0.84 offset=0 -> joint=gripper_joint multiplier=0.84 offset=0; parent hand_main_l_link -> gripper_inner_l_link
- joint finger_r_joint: mimic joint=hand_main_r_joint multiplier=-0.84 offset=0 -> joint=gripper_joint multiplier=-0.84 offset=0; parent hand_main_r_link -> gripper_inner_r_link

File: sobit_pro_description/robots/sobit_pro.urdf.xacro (robot description, xacro)
@@ -11,4 +11,12 @@
   <xacro:include filename="$(find sobit_pro_description)/urdf/head/head.urdf.xacro" />
   <xacro:include filename="$(find sobit_pro_description)/urdf/sensor/azure_kinect.urdf.xacro" />
+  <xacro:include filename="$(find sobit_pro_description)/urdf/sensor/urg.urdf.xacro" />
+  <!--
+  <xacro:include filename="$(find sobit_pro_description)/urdf/arm/arm.urdf.xacro" />
+  <xacro:include filename="$(find sobit_pro_description)/urdf/gripper/gripper.urdf.xacro" />
+  <xacro:include filename="$(find sobit_pro_description)/urdf/head/head.urdf.xacro" />
+  <xacro:include filename="$(find sobit_pro_description)/urdf/pole/pole.urdf.xacro" />
+  <xacro:include filename="$(find sobit_pro_description)/urdf/sensor/sensor.urdf.xacro" />
+  -->
   <xacro:base/>
   <xacro:wheel parent="base_link" />
@@ -17,3 +25,15 @@
   <xacro:head prefix="head_camera" parent="base_link" />
   <xacro:azure_kinect prefix="head_camera" parent="head_camera_tilt_link" />
+  <xacro:urg parent="base_link"/>
+  <!--
+  <stack_hexagons parent="base_link" />
+  <xacro:arm prefix="arm" parent="plate_top_link"/>
+  <xacro:hand prefix="hand_motor" parent="wrist_flex_link"/>
+  <xacro:pole parent="plate_top_link"/>
+  <xacro:xtion_motor prefix="xtion" parent="base_pole_link"/>
+  <xacro:sensor_asus_xtion_pro parent="xtion_double_sided_tape_link"/>
+  <xacro:mic parent="base_pole_link"/>
+  <xacro:matrix parent="base_pole_link"/>
+  <xacro:urg parent="base_link"/>
+  -->
 </robot>

File: sobit_pro_description/urdf/arm/arm.urdf.xacro (robot description, xacro)
@@ -17,4 +17,10 @@
       </visual>
     </link>
+    <joint name="${prefix}_fixed_joint" type="fixed">
+      <parent link="${prefix}_base_link" />
+      <child link="${prefix}_fixed_link" />
+      <origin xyz="0 0 0" rpy="0 0 ${-M_PI / 2}" />
+    </joint>
+    <link name="${prefix}_fixed_link" />
     <joint name="${prefix}1_joint" type="revolute">
       <parent link="${prefix}_base_link" />

File: sobit_pro_description/urdf/base/base.urdf.xacro (robot description, xacro)
@@ -7,5 +7,5 @@
       <parent link="base_footprint" />
       <child link="base_link" />
-      <origin xyz="0 0 0.143" rpy="0 0 0" />
+      <origin xyz="0 0 0.143" rpy="0 0 ${M_PI / 2}" />
     </joint>
     <link name="base_link">

File: sobit_pro_description/urdf/sensor/azure_kinect.urdf.xacro (robot description, xacro)
@@ -16,22 +16,4 @@
       </visual>
     </link>
-    <joint name="${prefix}_base_joint" type="fixed">
-      <parent link="${prefix}_link" />
-      <child link="${prefix}_base" />
-      <origin xyz="0. -0.055 0.04" rpy="0. 0. ${-M_PI / 2}" />
-    </joint>
-    <link name="${prefix}_body" />
-    <joint name="${prefix}_base_to_body" type="fixed">
-      <parent link="${prefix}_base" />
-      <child link="${prefix}_body" />
-      <origin xyz="-0.0757 0. 0.008" rpy="0. 0. 0." />
-    </joint>
-    <link name="${prefix}_base" />
-    <joint name="${prefix}_base_to_visor" type="fixed">
-      <parent link="${prefix}_base" />
-      <child link="${prefix}_visor" />
-      <origin xyz="0. 0. 0." rpy="0. 0. 0." />
-    </joint>
-    <link name="${prefix}_visor" />
   </xacro:macro>
 </robot>
