Commit message: [UPD] migration from ROS 1

File: sobit_pro_description/robots/sobit_pro.urdf (robot description, URDF)
Before this commit: robot sobit_pro, 64 links, 63 joints
Links:
- link arm_base_link: geometry collision box size=0.140 0.156 0.043; visual mesh filename=file://$(find sobit_pro_description)/meshes/arm/arm_base.stl scale=0.001 0.001 0.001
- link arm_elbow_lower_pan_link: geometry collision box size=0.120 0.048 0.03975; visual mesh filename=file://$(find sobit_pro_description)/meshes/arm/arm_elbow_l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 scale=0.001 0.001 0.001
- link arm_elbow_lower_tilt_link: geometry collision box size=0.005 0.041 0.024; visual mesh filename=file://$(find sobit_pro_description)/meshes/arm/arm_elbow_l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 scale=0.001 0.001 0.001
- link arm_elbow_upper_1_tilt_link: geometry collision box size=0.127 0.048 0.035; visual mesh filename=file://$(find sobit_pro_description)/meshes/arm/arm_inner.s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 scale=0.001 0.001 0.001
- link arm_shoulder_1_tilt_link: geometry collision box size=0.1166 0.124 0.043; visual mesh filename=file://$(find sobit_pro_description)/meshes/arm/arm_upper.s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 scale=0.001 0.001 0.001
- link back_base_link: geometry collision box size=0.02 0.02 0.517; visual mesh filename=file://$(find sobit_pro_description)/meshes/back/back_base.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 scale=0.001 0.001 0.001
- link cover_link: geometry collision box size=0.35786 0.3965 0.489; visual mesh filename=file://$(find sobit_pro_description)/meshes/body/cover.stl scale=0.001 0.001 0.001
- link hand_base_link: geometry collision box size=0.06102 0.102 0.0745; visual mesh filename=file://$(find sobit_pro_description)/meshes/hand/hand_base.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 scale=0.001 0.001 0.001
- link hand_finger_l_link: geometry collision box size=0.07317 0.01137 0.044; visual mesh filename=file://$(find sobit_pro_description)/meshes/hand/hand_finge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 scale=0.001 0.001 0.001
- link hand_finger_r_link: geometry collision box size=0.07317 0.01137 0.044; visual mesh filename=file://$(find sobit_pro_description)/meshes/hand/hand_finge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 scale=0.001 0.001 0.001
- link hand_inner_l_link: geometry collision box size=0.05296 0.01 0.066; visual mesh filename=file://$(find sobit_pro_description)/meshes/hand/hand_inner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 scale=0.001 0.001 0.001
- link hand_link: geometry collision box size=0.05296 0.01 0.066; visual mesh filename=file://$(find sobit_pro_description)/meshes/hand/hand_inner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 scale=0.001 0.001 0.001
- link hand_outer_l_link: geometry collision box size=0.04281 0.01 0.056; visual mesh filename=file://$(find sobit_pro_description)/meshes/hand/hand_outer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 scale=0.001 0.001 0.001
- link hand_outer_r_link: geometry collision box size=0.04281 0.01 0.056; visual mesh filename=file://$(find sobit_pro_description)/meshes/hand/hand_outer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 scale=0.001 0.001 0.001
- link head_base_link: geometry collision box size=0.15125 0.0285 0.044; visual mesh filename=file://$(find sobit_pro_description)/meshes/head/head_camer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 scale=0.001 0.001 0.001
- link head_camera_plug_base_link: geometry collision box size=0.0994 0.09637 0.0222; visual mesh filename=file://$(find sobit_pro_description)/meshes/akdk_camera.dae
- link head_pan_link: geometry collision box size=0.0285 0.037 0.03525; visual mesh filename=file://$(find sobit_pro_description)/meshes/head/head_camer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 scale=0.001 0.001 0.001
- link head_tilt_link: geometry collision box size=0.046 0.0466 0.0115; visual mesh filename=file://$(find sobit_pro_description)/meshes/head/head_camer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 scale=0.001 0.001 0.001
- link lidar_base_link: geometry collision box size=0.092 0.184 0.007; visual mesh filename=file://$(find sobit_pro_description)/meshes/sensor/lidar_ba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 scale=0.001 0.001 0.001
- link mic_base_link: geometry collision box size=0.0292 0.12919999999999998 0.03; visual mesh filename=file://$(find sobit_pro_description)/meshes/sensor/mic_base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 scale=0.001 0.001 0.001
- link mic_link: geometry collision cylinder length=0.281 radius=0.011; visual mesh filename=file://$(find sobit_pro_description)/meshes/sensor/mic.stl scale=0.001 0.001 0.001
- link plate_bottom_link: geometry collision box size=0.3 0.3 0.009; visual mesh filename=file://$(find sobit_pro_description)/meshes/body/plate_bott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 scale=0.001 0.001 0.001
- link plate_middle_link: geometry collision box size=0.3 0.3 0.009; visual mesh filename=file://$(find sobit_pro_description)/meshes/body/plate_midd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 scale=0.001 0.001 0.001
- link plate_top_link: geometry collision box size=0.3 0.3 0.009; visual mesh filename=file://$(find sobit_pro_description)/meshes/body/plate_top.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 scale=0.001 0.001 0.001
- link wheel_b_l_drive_link: geometry collision cylinder length=0.029 radius=0.072; visual mesh filename=file://$(find sobit_pro_description)/meshes/wheel/wheel_dri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 scale=0.001 0.001 0.001
- link wheel_b_l_steer_base_link: geometry collision box size=0.05525 0.0285 0.084; visual mesh filename=file://$(find sobit_pro_description)/meshes/wheel/wheel_bas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 scale=0.001 0.001 0.001
- link wheel_b_l_steer_link: geometry collision box size=0.0436 0.0495 0.1766; visual mesh filename=file://$(find sobit_pro_description)/meshes/wheel/wheel_ste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 scale=0.001 0.001 0.001
- link wheel_b_r_drive_link: geometry collision cylinder length=0.029 radius=0.072; visual mesh filename=file://$(find sobit_pro_description)/meshes/wheel/wheel_dri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 scale=0.001 0.001 0.001
- link wheel_b_r_steer_base_link: geometry collision box size=0.05525 0.0285 0.084; visual mesh filename=file://$(find sobit_pro_description)/meshes/wheel/wheel_bas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 scale=0.001 0.001 0.001
- link wheel_b_r_steer_link: geometry collision box size=0.0436 0.0495 0.1766; visual mesh filename=file://$(find sobit_pro_description)/meshes/wheel/wheel_ste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 scale=0.001 0.001 0.001
- link wheel_f_l_drive_link: geometry collision cylinder length=0.029 radius=0.072; visual mesh filename=file://$(find sobit_pro_description)/meshes/wheel/wheel_dri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 scale=0.001 0.001 0.001
- link wheel_f_l_steer_base_link: geometry collision box size=0.05525 0.0285 0.084; visual mesh filename=file://$(find sobit_pro_description)/meshes/wheel/wheel_bas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 scale=0.001 0.001 0.001
- link wheel_f_l_steer_link: geometry collision box size=0.0436 0.0495 0.1766; visual mesh filename=file://$(find sobit_pro_description)/meshes/wheel/wheel_ste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 scale=0.001 0.001 0.001
- link wheel_f_r_drive_link: geometry collision cylinder length=0.029 radius=0.072; visual mesh filename=file://$(find sobit_pro_description)/meshes/wheel/wheel_dri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 scale=0.001 0.001 0.001
- link wheel_f_r_steer_base_link: geometry collision box size=0.05525 0.0285 0.084; visual mesh filename=file://$(find sobit_pro_description)/meshes/wheel/wheel_bas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 scale=0.001 0.001 0.001
- link wheel_f_r_steer_link: geometry collision box size=0.0436 0.0495 0.1766; visual mesh filename=file://$(find sobit_pro_description)/meshes/wheel/wheel_ste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 scale=0.001 0.001 0.001

File: sobit_pro_description/robots/sobit_pro_robot.urdf.xacro (robot description, xacro)
@@ -22,5 +22,6 @@
   <xacro:include filename="$(find sobit_pro_description)/urdf/sensor/realsense_d415.urdf.xacro" />
   <xacro:include filename="$(find urg_node)/urdf/hokuyo_ust.urdf.xacro" />
-  <xacro:include filename="$(find azure_kinect_ros_driver)/urdf/azure_kinect.urdf.xacro" />
+  <xacro:include filename="$(find sobit_pro_description)/urdf/azure_kinect.urdf.xacro" />
+  <!-- <xacro:include filename="$(find azure_kinect_ros_driver)/urdf/azure_kinect.urdf.xacro" /> -->
   <!-- <xacro:include filename="$(find realsense2_description)/urdf/_l515.urdf.xacro" /> -->
   <xacro:include filename="$(find realsense2_description)/urdf/_d405.urdf.xacro" />
@@ -43,5 +44,5 @@
     <xacro:arm   prefix="arm"   parent="plate_top_link" />
     <xacro:hand  prefix_hand="hand" prefix_finger="finger" parent="arm_wrist_tilt_link" />
-    <xacro:lidar prefix="lidar" parent="plate_bottom_link" robot_namespace="$(arg robot_namespace)" />
+    <xacro:lidar prefix="lidar" parent="plate_bottom_link" />
     <xacro:azure_camera prefix="head_camera" parent="head_tilt_link" />
     <xacro:matrix prefix="matrix" parent="head_camera_base" />
@@ -58,5 +59,5 @@
     <xacro:arm   prefix="arm"   parent="plate_top_link" />
     <xacro:hand  prefix_hand="hand" prefix_finger="finger" parent="arm_wrist_tilt_link" />
-    <xacro:lidar prefix="lidar" parent="plate_bottom_link" robot_namespace="$(arg robot_namespace)" />
+    <xacro:lidar prefix="lidar" parent="plate_bottom_link" />
     <!-- <xacro:realsense_l515 prefix="hand_camera" parent="arm_wrist_tilt_link" /> -->
     <xacro:realsense_d405 prefix="hand_camera" parent="arm_wrist_tilt_link" />
@@ -72,5 +73,5 @@
     <xacro:head  prefix="head"  parent="back_base_link" />
     <xacro:mic   prefix="mic"   parent="back_base_link" />
-    <xacro:lidar prefix="lidar" parent="plate_bottom_link" robot_namespace="$(arg robot_namespace)" />
+    <xacro:lidar prefix="lidar" parent="plate_bottom_link" />
     <xacro:azure_camera prefix="head_camera" parent="head_tilt_link" />
     <xacro:matrix prefix="matrix" parent="head_camera_base" />
@@ -83,5 +84,5 @@
     <xacro:wheel prefix="wheel" parent="plate_middle_link" />
     <xacro:cover prefix="cover" parent="plate_top_link" />
-    <xacro:lidar prefix="lidar" parent="plate_bottom_link" robot_namespace="$(arg robot_namespace)" />
+    <xacro:lidar prefix="lidar" parent="plate_bottom_link" />
   </xacro:if>
   <!-- enable_mb: false, enable_arm: true, enable_head: true -->
@@ -95,5 +96,5 @@
     <xacro:arm   prefix="arm"   parent="plate_top_link" />
     <xacro:hand  prefix_hand="hand" prefix_finger="finger" parent="arm_wrist_tilt_link" />
-    <xacro:azure_camera prefix="head_camera" parent="head_tilt_link" />
+    <!-- <xacro:azure_camera prefix="head_camera" parent="head_tilt_link" /> -->
     <xacro:matrix prefix="matrix" parent="head_camera_base" />
     <!-- <xacro:realsense_l515 prefix="hand_camera" parent="arm_wrist_tilt_link" /> -->
@@ -120,11 +121,11 @@
     <xacro:head  prefix="head"  parent="back_base_link" />
     <xacro:mic   prefix="mic"   parent="back_base_link" />
-    <xacro:azure_camera prefix="head_camera" parent="head_tilt_link" />
+    <!-- <xacro:azure_camera prefix="head_camera" parent="head_tilt_link" /> -->
     <xacro:matrix prefix="matrix" parent="head_camera_base" />
   </xacro:if>
   <!-- enable_gz: true -->
-  <xacro:if value="${$(arg enable_gz)}">
+  <!-- <xacro:if value="${$(arg enable_gz)}">
     <xacro:include filename="$(find sobit_pro_sim_description)/urdf/gazebo.urdf.xacro" />
     <xacro:gazebo/>
-  </xacro:if>
+  </xacro:if> -->
 </robot>

File: sobit_pro_description/urdf/arm/arm.urdf.xacro (robot description, xacro)
@@ -13,5 +13,5 @@
         <origin xyz="0.0 0.0 0.0" rpy="${M_PI/2} 0.0 0.0" />
         <geometry>
-          <mesh filename="package://sobit_pro_description/meshes/arm/arm_base.stl" scale="0.001 0.001 0.001" />
+          <mesh filename="file://$(find sobit_pro_description)/meshes/arm/arm_base.stl" scale="0.001 0.001 0.001" />
         </geometry>
         <material name="black" />
@@ -43,5 +43,5 @@
         <origin xyz="0.0 0.0 0.0" rpy="${M_PI/2} 0.0 ${M_PI/2}" />
         <geometry>
-          <mesh filename="package://sobit_pro_description/meshes/arm/arm_upper.stl" scale="0.001 0.001 0.001" />
+          <mesh filename="file://$(find sobit_pro_description)/meshes/arm/arm_upper.stl" scale="0.001 0.001 0.001" />
         </geometry>
         <material name="black" />
@@ -83,5 +83,5 @@
         <origin xyz="0.0 0.0 0.0" rpy="${M_PI/2} 0.0 ${M_PI/2}" />
         <geometry>
-          <mesh filename="package://sobit_pro_description/meshes/arm/arm_inner.stl" scale="0.001 0.001 0.001" />
+          <mesh filename="file://$(find sobit_pro_description)/meshes/arm/arm_inner.stl" scale="0.001 0.001 0.001" />
         </geometry>
         <material name="black" />
@@ -123,5 +123,5 @@
         <origin xyz="0.0 0.0 0.0" rpy="${M_PI/2} 0.0 ${M_PI/2}" />
         <geometry>
-          <mesh filename="package://sobit_pro_description/meshes/arm/arm_elbow_lower_tilt.stl" scale="0.001 0.001 0.001" />
+          <mesh filename="file://$(find sobit_pro_description)/meshes/arm/arm_elbow_lower_tilt.stl" scale="0.001 0.001 0.001" />
         </geometry>
         <material name="black" />
@@ -153,5 +153,5 @@
         <origin xyz="0.0 0.0 0.0" rpy="${M_PI/2} 0.0 ${M_PI/2}" />
         <geometry>
-          <mesh filename="package://sobit_pro_description/meshes/arm/arm_elbow_lower_pan.stl" scale="0.001 0.001 0.001" />
+          <mesh filename="file://$(find sobit_pro_description)/meshes/arm/arm_elbow_lower_pan.stl" scale="0.001 0.001 0.001" />
         </geometry>
         <material name="black" />

File: sobit_pro_description/urdf/back/back.urdf.xacro (robot description, xacro)
@@ -12,5 +12,5 @@
         <origin xyz="0.0 0.0 0.0" rpy="0.0 0.0 ${M_PI}" />
         <geometry>
-          <mesh filename="package://sobit_pro_description/meshes/back/back_base.stl" scale="0.001 0.001 0.001" />
+          <mesh filename="file://$(find sobit_pro_description)/meshes/back/back_base.stl" scale="0.001 0.001 0.001" />
         </geometry>
         <material name="grey" />

File: sobit_pro_description/urdf/body/cover.urdf.xacro (robot description, xacro)
@@ -12,5 +12,5 @@
         <origin xyz="0.0 0.0 0.0" rpy="${M_PI/2} 0.0 ${M_PI/2}" />
         <geometry>
-          <mesh filename="package://sobit_pro_description/meshes/body/cover.stl" scale="0.001 0.001 0.001" />
+          <mesh filename="file://$(find sobit_pro_description)/meshes/body/cover.stl" scale="0.001 0.001 0.001" />
         </geometry>
         <material name="blue" />

File: sobit_pro_description/urdf/body/plate.urdf.xacro (robot description, xacro)
@@ -12,5 +12,5 @@
         <origin xyz="0.0 0.0 0.0" rpy="0.0 0.0 0.0" />
         <geometry>
-          <mesh filename="package://sobit_pro_description/meshes/body/plate_bottom.stl" scale="0.001 0.001 0.001" />
+          <mesh filename="file://$(find sobit_pro_description)/meshes/body/plate_bottom.stl" scale="0.001 0.001 0.001" />
         </geometry>
         <material name="black" />
@@ -39,5 +39,5 @@
         <origin xyz="0.0 0.0 0.0" rpy="0.0 0.0 0.0" />
         <geometry>
-          <mesh filename="package://sobit_pro_description/meshes/body/plate_middle.stl" scale="0.001 0.001 0.001" />
+          <mesh filename="file://$(find sobit_pro_description)/meshes/body/plate_middle.stl" scale="0.001 0.001 0.001" />
         </geometry>
         <material name="black" />
@@ -66,5 +66,5 @@
         <origin xyz="0.0 0.0 0.0" rpy="0.0 0.0 ${M_PI/2}" />
         <geometry>
-          <mesh filename="package://sobit_pro_description/meshes/body/plate_top.stl" scale="0.001 0.001 0.001" />
+          <mesh filename="file://$(find sobit_pro_description)/meshes/body/plate_top.stl" scale="0.001 0.001 0.001" />
         </geometry>
         <material name="black" />

File: sobit_pro_description/urdf/hand/hand.urdf.xacro (robot description, xacro)
@@ -13,5 +13,5 @@
         <origin xyz="0.0 0.0 0.0" rpy="${M_PI/2.0} 0.0 ${M_PI/2.0}" />
         <geometry>
-          <mesh filename="package://sobit_pro_description/meshes/hand/hand_base.stl" scale="0.001 0.001 0.001" />
+          <mesh filename="file://$(find sobit_pro_description)/meshes/hand/hand_base.stl" scale="0.001 0.001 0.001" />
         </geometry>
         <material name="black" />
@@ -42,5 +42,5 @@
         <origin xyz="0.0 0.0 0.0" rpy="0.0 0.0 ${M_PI/2.0}" />
         <geometry>
-          <mesh filename="package://sobit_pro_description/meshes/hand/hand_inner_l.stl" scale="0.001 0.001 0.001" />
+          <mesh filename="file://$(find sobit_pro_description)/meshes/hand/hand_inner_l.stl" scale="0.001 0.001 0.001" />
         </geometry>
         <material name="black" />
@@ -71,5 +71,5 @@
         <origin xyz="0.0 0.0 0.0" rpy="0.0 0.0 ${M_PI/2.0}" />
         <geometry>
-          <mesh filename="package://sobit_pro_description/meshes/hand/hand_inner_r.stl" scale="0.001 0.001 0.001" />
+          <mesh filename="file://$(find sobit_pro_description)/meshes/hand/hand_inner_r.stl" scale="0.001 0.001 0.001" />
         </geometry>
         <material name="black" />
@@ -100,5 +100,5 @@
         <origin xyz="0.0 0.0 0.0" rpy="0.0 0.0 ${M_PI/2.0}" />
         <geometry>
-          <mesh filename="package://sobit_pro_description/meshes/hand/hand_outer_l.stl" scale="0.001 0.001 0.001" />
+          <mesh filename="file://$(find sobit_pro_description)/meshes/hand/hand_outer_l.stl" scale="0.001 0.001 0.001" />
         </geometry>
         <material name="black" />
@@ -129,5 +129,5 @@
         <origin xyz="0.0 0.0 0.0" rpy="0.0 0.0 ${M_PI/2.0}" />
         <geometry>
-          <mesh filename="package://sobit_pro_description/meshes/hand/hand_outer_r.stl" scale="0.001 0.001 0.001" />
+          <mesh filename="file://$(find sobit_pro_description)/meshes/hand/hand_outer_r.stl" scale="0.001 0.001 0.001" />
         </geometry>
         <material name="black" />
@@ -158,5 +158,5 @@
         <origin xyz="-0.029998 0.025 0.0" rpy="0.0 0.0 ${M_PI/2.0}" />
         <geometry>
-          <mesh filename="package://sobit_pro_description/meshes/hand/hand_finger_l.stl" scale="0.001 0.001 0.001" />
+          <mesh filename="file://$(find sobit_pro_description)/meshes/hand/hand_finger_l.stl" scale="0.001 0.001 0.001" />
         </geometry>
         <material name="black" />
@@ -187,5 +187,5 @@
         <origin xyz="-0.029998 -0.025 0.0" rpy="0.0 0.0 ${M_PI/2.0}" />
         <geometry>
-          <mesh filename="package://sobit_pro_description/meshes/hand/hand_finger_r.stl" scale="0.001 0.001 0.001" />
+          <mesh filename="file://$(find sobit_pro_description)/meshes/hand/hand_finger_r.stl" scale="0.001 0.001 0.001" />
         </geometry>
         <material name="black" />

File: sobit_pro_description/urdf/head/head.urdf.xacro (robot description, xacro)
@@ -13,5 +13,5 @@
         <origin xyz="0.0 0.0 0.0" rpy="${M_PI/2.0} 0.0 ${M_PI/2.0}" />
         <geometry>
-          <mesh filename="package://sobit_pro_description/meshes/head/head_camera_base.stl" scale="0.001 0.001 0.001" />
+          <mesh filename="file://$(find sobit_pro_description)/meshes/head/head_camera_base.stl" scale="0.001 0.001 0.001" />
         </geometry>
         <material name="black" />
@@ -42,5 +42,5 @@
         <origin xyz="0.0 0.0 0.0" rpy="0.0 0.0 ${M_PI/2.0}" />
         <geometry>
-          <mesh filename="package://sobit_pro_description/meshes/head/head_camera_pan.stl" scale="0.001 0.001 0.001" />
+          <mesh filename="file://$(find sobit_pro_description)/meshes/head/head_camera_pan.stl" scale="0.001 0.001 0.001" />
         </geometry>
         <material name="black" />
@@ -71,5 +71,5 @@
         <origin xyz="0.0 0.0 0.0" rpy="0.0 0.0 ${M_PI/2.0}" />
         <geometry>
-          <mesh filename="package://sobit_pro_description/meshes/head/head_camera_tilt.stl" scale="0.001 0.001 0.001" />
+          <mesh filename="file://$(find sobit_pro_description)/meshes/head/head_camera_tilt.stl" scale="0.001 0.001 0.001" />
         </geometry>
         <material name="black" />

File: sobit_pro_description/urdf/sensor/azure_camera.urdf.xacro (robot description, xacro)
@@ -9,7 +9,7 @@
     </joint>
     <link name="${prefix}_base"/>
-    <xacro:azure_kinect parent="${prefix}_base" tf_prefix="${prefix}_" add_cover="false">
+    <!-- <xacro:azure_kinect parent="${prefix}_base" tf_prefix="${prefix}_" add_cover="false">
       <origin xyz="0.0 0 0.0" rpy="0 0 0"/>
-    </xacro:azure_kinect>
+    </xacro:azure_kinect> -->
   </xacro:macro>
 </robot>

File: sobit_pro_description/urdf/sensor/lidar.urdf.xacro (robot description, xacro)
@@ -2,5 +2,5 @@
 <robot name="sobit_pro"
        xmlns:xacro="http://ros.org/wiki/xacro">
-  <xacro:macro name="lidar" params="prefix parent robot_namespace">
+  <xacro:macro name="lidar" params="prefix parent">
     <joint name="${prefix}_base_joint" type="fixed">
       <parent link="${parent}" />
@@ -12,5 +12,5 @@
         <origin xyz="0.0 0.0 0.0" rpy="${M_PI/2} 0.0 ${M_PI}" />
         <geometry>
-          <mesh filename="package://sobit_pro_description/meshes/sensor/lidar_base.stl" scale="0.001 0.001 0.001" />
+          <mesh filename="file://$(find sobit_pro_description)/meshes/sensor/lidar_base.stl" scale="0.001 0.001 0.001" />
         </geometry>
         <material name="black" />
@@ -30,5 +30,5 @@
       </inertial>
     </link>
-    <xacro:hokuyo_ust_mount prefix="${prefix}" parent="${prefix}_base_link" topic="scan" robot_namespace="${robot_namespace}/" model="ust-10" min_angle="-${M_PI/2}" max_angle="${M_PI/2}" >
+    <xacro:hokuyo_ust_mount prefix="${prefix}" parent="${prefix}_base_link" topic="scan" >
       <origin xyz="0.067 0.0 0.0" rpy="0.0 0.0 0.0" />
     </xacro:hokuyo_ust_mount>

File: sobit_pro_description/urdf/sensor/mic.urdf.xacro (robot description, xacro)
@@ -12,5 +12,5 @@
         <origin xyz="0.0 0.0 0.0" rpy="${M_PI/2} 0.0 ${M_PI}" />
         <geometry>
-          <mesh filename="package://sobit_pro_description/meshes/sensor/mic_base.stl" scale="0.001 0.001 0.001" />
+          <mesh filename="file://$(find sobit_pro_description)/meshes/sensor/mic_base.stl" scale="0.001 0.001 0.001" />
         </geometry>
         <material name="black" />
@@ -41,5 +41,5 @@
         <origin xyz="0.0 0.0 0.0" rpy="${M_PI/2} 0.0 ${M_PI}" />
         <geometry>
-          <mesh filename="package://sobit_pro_description/meshes/sensor/mic.stl" scale="0.001 0.001 0.001" />
+          <mesh filename="file://$(find sobit_pro_description)/meshes/sensor/mic.stl" scale="0.001 0.001 0.001" />
         </geometry>
         <material name="black" />

File: sobit_pro_description/urdf/sensor/realsense_d405.urdf.xacro (robot description, xacro)
@@ -9,5 +9,5 @@
     </joint>
     <link name="${prefix}_base_link" />
-    <xacro:sensor_d405 parent="${prefix}_base_link" name="${prefix}" use_nominal_extrinsics="true" use_mesh="true">
+    <xacro:sensor_d405 parent="${prefix}_base_link" name="${prefix}" use_nominal_extrinsics="true" >
       <origin xyz="0.0 0.0 0.0" rpy="0.0 0.0 0.0" />
     </xacro:sensor_d405>

File: sobit_pro_description/urdf/sensor/realsense_d415.urdf.xacro (robot description, xacro)
@@ -11,5 +11,5 @@
         <origin xyz="0.15 0.15 -0.0155" rpy="0.0 0.0 ${90*M_PI/180}" />
         <geometry>
-          <mesh filename="package://sobit_pro_description/meshes/body/plate_top_camera_mount.stl" scale="1.0 1.0 1.0" />
+          <mesh filename="file://$(find sobit_pro_description)/meshes/body/plate_top_camera_mount.stl" scale="1.0 1.0 1.0" />
         </geometry>
         <material name="black" />

File: sobit_pro_description/urdf/sensor/realsense_l515.urdf.xacro (robot description, xacro)
@@ -9,5 +9,5 @@
     </joint>
     <link name="${prefix}_base_link" />
-    <xacro:sensor_l515 parent="${prefix}_base_link" name="${prefix}" use_nominal_extrinsics="true" add_plug="false" use_mesh="true">
+    <xacro:sensor_l515 parent="${prefix}_base_link" name="${prefix}" use_nominal_extrinsics="true" add_plug="false" >
       <origin xyz="0.0 0.0 0.0" rpy="0.0 0.0 0.0" />
     </xacro:sensor_l515>
