Commit message: [UPD] migration from ROS 1

File: sobit_pro_description/urdf/wheel/wheel.urdf.xacro (robot description, xacro)
@@ -13,5 +13,5 @@
         <origin xyz="0.0 0.0 0.0" rpy="${M_PI/2.0} 0.0 ${M_PI/2.0}" />
         <geometry>
-          <mesh filename="package://sobit_pro_description/meshes/wheel/wheel_base.stl" scale="0.001 0.001 0.001" />
+          <mesh filename="file://$(find sobit_pro_description)/meshes/wheel/wheel_base.stl" scale="0.001 0.001 0.001" />
         </geometry>
         <material name="black" />
@@ -45,5 +45,5 @@
         <origin xyz="0.0 0.0 0.0" rpy="${M_PI/2} 0.0 ${M_PI/2}" />
         <geometry>
-          <mesh filename="package://sobit_pro_description/meshes/wheel/wheel_steer.stl" scale="0.001 0.001 0.001" />
+          <mesh filename="file://$(find sobit_pro_description)/meshes/wheel/wheel_steer.stl" scale="0.001 0.001 0.001" />
         </geometry>
         <material name="black" />
@@ -76,5 +76,5 @@
         <origin xyz="0.0 0.0 0.0" rpy="${M_PI/2} 0.0 ${M_PI+M_PI/2.0}" />
         <geometry>
-          <mesh filename="package://sobit_pro_description/meshes/wheel/wheel_drive.stl" scale="0.001 0.001 0.001" />
+          <mesh filename="file://$(find sobit_pro_description)/meshes/wheel/wheel_drive.stl" scale="0.001 0.001 0.001" />
         </geometry>
         <material name="wheel" />
