Commit message: update controller

File: sobit_pro_description/robots/sobit_pro_robot.urdf.xacro (robot description, xacro)
@@ -12,5 +12,5 @@
   <xacro:include filename="$(find sobit_pro_description)/urdf/body/cover.urdf.xacro" />
   <xacro:include filename="$(find sobit_pro_description)/urdf/back/back.urdf.xacro" />
-  <xacro:include filename="$(find sobit_pro_description)/urdf/wheel/wheel.urdf.xacro" />
+  <!-- <xacro:include filename="$(find sobit_pro_description)/urdf/wheel/wheel.urdf.xacro" /> -->
   <xacro:include filename="$(find sobit_pro_description)/urdf/arm/arm.urdf.xacro" />
   <xacro:include filename="$(find sobit_pro_description)/urdf/hand/hand.urdf.xacro" />
@@ -39,5 +39,5 @@
     <xacro:base/>
     <xacro:plate prefix="plate" parent="base_link" />
-    <xacro:wheel prefix="wheel" parent="plate_middle_link" />
+    <!-- <xacro:wheel prefix="wheel" parent="plate_middle_link" /> -->
     <xacro:cover prefix="cover" parent="plate_top_link" />
     <xacro:back  prefix="back"  parent="plate_top_link" />
@@ -57,5 +57,5 @@
     <xacro:base/>
     <xacro:plate prefix="plate" parent="base_link" />
-    <xacro:wheel prefix="wheel" parent="plate_middle_link" />
+    <!-- <xacro:wheel prefix="wheel" parent="plate_middle_link" /> -->
     <xacro:cover prefix="cover" parent="plate_top_link" />
     <xacro:arm   prefix="arm"   parent="plate_top_link" />
@@ -70,5 +70,5 @@
     <xacro:base/>
     <xacro:plate prefix="plate" parent="base_link" />
-    <xacro:wheel prefix="wheel" parent="plate_middle_link" />
+    <!-- <xacro:wheel prefix="wheel" parent="plate_middle_link" /> -->
     <xacro:cover prefix="cover" parent="plate_top_link" />
     <xacro:back  prefix="back"  parent="plate_top_link" />
@@ -84,5 +84,5 @@
     <xacro:base/>
     <xacro:plate prefix="plate" parent="base_link" />
-    <xacro:wheel prefix="wheel" parent="plate_middle_link" />
+    <!-- <xacro:wheel prefix="wheel" parent="plate_middle_link" /> -->
     <xacro:cover prefix="cover" parent="plate_top_link" />
     <xacro:lidar prefix="lidar" parent="plate_bottom_link" />

File: sobit_pro_description/urdf/controllers.urdf.xacro (robot description, xacro)
@@ -1,170 +1,185 @@
 <?xml version="1.0" encoding="UTF-8" ?>
-<!-- SOBIT PRO (Dynamixel Control) -->
+<!-- SOBIT Light (Dynamixel Control) -->
 <robot name="sobit_pro_controllers" xmlns:xacro="http://www.ros.org/wiki/xacro">
-    <xacro:macro name="controllers" params="name enable_gz:=False robot_name:=sobit_pro">
-        <ros2_control name="${name}_arg" type="system">
-            <hardware>
-                <xacro:if value="${$(arg enable_gz)}">
-                    <plugin>ign_ros2_control/IgnitionSystem</plugin>
-                </xacro:if>
-                <xacro:unless value="${$(arg enable_gz)}">
-                    <plugin>dynamixel_hardware/DynamixelHardware</plugin>
-                    <param name="usv_port">/dev/ttyUSB0</param>
-                    <param name="baud_rate">3000000</param>
-                </xacro:unless>
-            </hardware>
-            <!-- Position Drive: Arm -->
-            <joint name="arm_shoulder_1_tilt_joint">
-                <xacro:unless value="${$(arg enable_gz)}">
-                    <param name="id">11</param>
-                </xacro:unless>
-                <command_interface name="position">
-                    <param name="min">-1.570796327</param>
-                    <param name="max">1.570796327</param>
-                </command_interface>
-                <command_interface name="velocity"/>
-                <state_interface name="position">
-                    <param name="initial_value">0.0</param>
-                </state_interface>
-                <state_interface name="velocity"/>
-                <state_interface name="effort"/>
-            </joint>
-            <joint name="arm_shoulder_2_tilt_joint">
-                <xacro:unless value="${$(arg enable_gz)}">
-                    <param name="id">12</param>
-                </xacro:unless>
-                <command_interface name="position">
-                    <param name="min">-1.570796327</param>
-                    <param name="max">1.570796327</param>
-                </command_interface>
-                <command_interface name="velocity"/>
-                <state_interface name="position">
-                    <param name="initial_value">0.0</param>
-                </state_interface>
-                <state_interface name="velocity"/>
-                <state_interface name="effort"/>
-            </joint>
-            <joint name="arm_elbow_upper_1_tilt_joint">
-                <xacro:unless value="${$(arg enable_gz)}">
-                    <param name="id">13</param>
-                </xacro:unless>
-                <command_interface name="position">
-                    <param name="min">-1.570796327</param>
-                    <param name="max">1.570796327</param>
-                </command_interface>
-                <command_interface name="velocity"/>
-                <state_interface name="position">
-                    <param name="initial_value">0.0</param>
-                </state_interface>
-                <state_interface name="velocity"/>
-                <state_interface name="effort"/>
-            </joint>
-            <joint name="arm_elbow_upper_2_tilt_joint">
-                <xacro:unless value="${$(arg enable_gz)}">
-                    <param name="id">14</param>
-                </xacro:unless>
-                <command_interface name="position">
-                    <param name="min">-1.570796327</param>
-                    <param name="max">1.570796327</param>
-                </command_interface>
-                <command_interface name="velocity"/>
-                <state_interface name="position">
-                    <param name="initial_value">0.0</param>
-                </state_interface>
-                <state_interface name="velocity"/>
-                <state_interface name="effort"/>
-            </joint>
-            <joint name="arm_elbow_lower_tilt_joint">
-                <xacro:unless value="${$(arg enable_gz)}">
-                    <param name="id">15</param>
-                </xacro:unless>
-                <command_interface name="position">
-                    <param name="min">-1.570796327</param>
-                    <param name="max">1.570796327</param>
-                </command_interface>
-                <command_interface name="velocity"/>
-                <state_interface name="position">
-                    <param name="initial_value">0.0</param>
-                </state_interface>
-                <state_interface name="velocity"/>
-                <state_interface name="effort"/>
-            </joint>
-            <joint name="arm_elbow_lower_pan_joint">
-                <xacro:unless value="${$(arg enable_gz)}">
-                    <param name="id">16</param>
-                </xacro:unless>
-                <command_interface name="position">
-                    <param name="min">-1.570796327</param>
-                    <param name="max">1.570796327</param>
-                </command_interface>
-                <command_interface name="velocity"/>
-                <state_interface name="position">
-                    <param name="initial_value">0.0</param>
-                </state_interface>
-                <state_interface name="velocity"/>
-                <state_interface name="effort"/>
-            </joint>
-            <joint name="arm_wrist_tilt_joint">
-                <xacro:unless value="${$(arg enable_gz)}">
-                    <param name="id">17</param>
-                </xacro:unless>
-                <command_interface name="position">
-                    <param name="min">-1.570796327</param>
-                    <param name="max">1.570796327</param>
-                </command_interface>
-                <command_interface name="velocity"/>
-                <state_interface name="position">
-                    <param name="initial_value">0.0</param>
-                </state_interface>
-                <state_interface name="velocity"/>
-                <state_interface name="effort"/>
-            </joint>
-            <joint name="hand_joint">
-                <xacro:unless value="${$(arg enable_gz)}">
-                    <param name="id">18</param>
-                </xacro:unless>
-                <command_interface name="position">
-                    <param name="min">-1.570796327</param>
-                    <param name="max">0</param>
-                </command_interface>
-                <command_interface name="velocity"/>
-                <state_interface name="position">
-                    <param name="initial_value">0.0</param>
-                </state_interface>
-                <state_interface name="velocity"/>
-                <state_interface name="effort"/>
-            </joint>
-            <!-- Position Drive: Head -->
-            <joint name="head_pan_joint">
-                <xacro:unless value="${$(arg enable_gz)}">
-                    <param name="id">21</param>
-                </xacro:unless>
-                <command_interface name="position">
-                    <param name="min">-1.570796327</param>
-                    <param name="max">1.570796327</param>
-                </command_interface>
-                <command_interface name="velocity"/>
-                <state_interface name="position">
-                    <param name="initial_value">0.0</param>
-                </state_interface>
-                <state_interface name="velocity"/>
-                <state_interface name="effort"/>
-            </joint>
-            <joint name="head_tilt_joint">
-                <xacro:unless value="${$(arg enable_gz)}">
-                    <param name="id">22</param>
-                </xacro:unless>
-                <command_interface name="position">
-                    <param name="min">-1.570796327</param>
-                    <param name="max">0.57</param>
-                </command_interface>
-                <command_interface name="velocity"/>
-                <state_interface name="position">
-                    <param name="initial_value">0.0</param>
-                </state_interface>
-                <state_interface name="velocity"/>
-                <state_interface name="effort"/>
-            </joint>
-        </ros2_control>
-    </xacro:macro>
+  <xacro:macro name="controllers" params="name enable_gz:=False robot_name:=sobit_pro">
+    <ros2_control name="${name}_arm" type="system">
+    <!-- <ros2_control name="joints_control" type="system"> -->
+      <hardware>
+        <xacro:if value="${$(arg enable_gz)}">
+          <plugin>ign_ros2_control/IgnitionSystem</plugin>
+          <!-- <plugin>gazebo_ros2_control/GazeboHardware</plugin> -->
+        </xacro:if>
+        <xacro:unless value="${$(arg enable_gz)}">
+          <plugin>dynamixel_hardware/DynamixelHardware</plugin>
+          <param name="usb_port">/dev/ttyUSB0</param>
+          <param name="baud_rate">1000000</param>
+          <param name="use_dummy">true</param>
+        </xacro:unless>
+      </hardware>
+      <!-- Position Drive: Arm -->
+      <joint name="arm_shoulder_1_tilt_joint">
+        <xacro:unless value="${$(arg enable_gz)}">
+          <param name="id">11</param>
+        </xacro:unless>
+        <command_interface name="position">
+          <param name="min">-1.570796327</param>
+          <param name="max">1.570796327</param>
+        </command_interface>
+        <command_interface name="velocity"/>
+        <state_interface name="position">
+          <param name="initial_value">0.0</param>
+        </state_interface>
+        <state_interface name="velocity"/>
+        <state_interface name="effort"/>
+      </joint>
+      <joint name="arm_shoulder_2_tilt_joint">
+        <xacro:unless value="${$(arg enable_gz)}">
+          <param name="id">12</param>
+        </xacro:unless>
+        <!-- <param name="mimic">arm_shoulder_pitch_joint</param>
+        <param name="multiplier">-1</param> -->
+        <!-- <command_interface name="position"/> -->
+        <command_interface name="position">
+          <param name="min">-1.570796327</param>
+          <param name="max">1.570796327</param>
+        </command_interface>
+        <command_interface name="velocity"/>
+        <state_interface name="position">
+          <param name="initial_value">1.57</param>
+        </state_interface>
+        <!-- <state_interface name="position"/> -->
+        <state_interface name="velocity"/>
+        <state_interface name="effort"/>
+      </joint>
+      <joint name="arm_elbow_upper_1_tilt_joint">
+        <xacro:unless value="${$(arg enable_gz)}">
+          <param name="id">13</param>
+        </xacro:unless>
+        <command_interface name="position">
+          <param name="min">-1.570796327</param>
+          <param name="max">1.570796327</param>
+        </command_interface>
+        <command_interface name="velocity"/>
+        <state_interface name="position">
+          <param name="initial_value">-1.57</param>
+        </state_interface>
+        <state_interface name="velocity"/>
+        <state_interface name="effort"/>
+      </joint>
+      <joint name="arm_elbow_upper_2_tilt_joint">
+        <xacro:unless value="${$(arg enable_gz)}">
+          <param name="id">14</param>
+        </xacro:unless>
+        <command_interface name="position">
+          <param name="min">-1.570796327</param>
+          <param name="max">1.570796327</param>
+        </command_interface>
+        <command_interface name="velocity"/>
+        <state_interface name="position">
+          <param name="initial_value">0.0</param>
+        </state_interface>
+        <state_interface name="velocity"/>
+        <state_interface name="effort"/>
+      </joint>
+      <joint name="arm_elbow_lower_tilt_joint">
+        <xacro:unless value="${$(arg enable_gz)}">
+          <param name="id">15</param>
+        </xacro:unless>
+        <command_interface name="position">
+          <param name="min">-1.570796327</param>
+          <param name="max">1.570796327</param>
+        </command_interface>
+        <command_interface name="velocity"/>
+        <state_interface name="position">
+          <param name="initial_value">0.0</param>
+        </state_interface>
+        <state_interface name="velocity"/>
+        <state_interface name="effort"/>
+      </joint>
+      <joint name="arm_elbow_lower_pan_joint">
+        <xacro:unless value="${$(arg enable_gz)}">
+          <param name="id">16</param>
+        </xacro:unless>
+        <command_interface name="position">
+          <param name="min">-1.570796327</param>
+          <param name="max">1.570796327</param>
+        </command_interface>
+        <command_interface name="velocity"/>
+        <state_interface name="position">
+          <param name="initial_value">0.0</param>
+        </state_interface>
+        <state_interface name="velocity"/>
+        <state_interface name="effort"/>
+      </joint>
+      <joint name="arm_wrist_tilt_joint">
+        <xacro:unless value="${$(arg enable_gz)}">
+          <param name="id">17</param>
+        </xacro:unless>
+        <command_interface name="position">
+          <param name="min">-1.570796327</param>
+          <param name="max">1.570796327</param>
+        </command_interface>
+        <command_interface name="velocity"/>
+        <state_interface name="position">
+          <param name="initial_value">0.0</param>
+        </state_interface>
+        <state_interface name="velocity"/>
+        <state_interface name="effort"/>
+      </joint>
+      <!-- Position Drive: Hand -->
+      <joint name="hand_joint">
+        <xacro:unless value="${$(arg enable_gz)}">
+          <param name="id">18</param>
+        </xacro:unless>
+        <command_interface name="position">
+            <param name="min">-1.570796327</param>
+            <param name="max">0.0</param>
+        </command_interface>
+        <command_interface name="velocity"/>
+        <state_interface name="position">
+          <param name="initial_value">0.0</param>
+        </state_interface>
+        <state_interface name="velocity"/>
+        <state_interface name="effort"/>
+      </joint>
+      <xacro:if value="${$(arg enable_gz)}">
+        <joint name="hand_sub_joint">
+          <param name="mimic">hand_joint</param>
+          <param name="multiplier">-1</param>
+          <command_interface name="position"/>
+          <command_interface name="velocity"/>
+          <state_interface name="position"/>
+          <state_interface name="velocity"/>
+          <state_interface name="effort"/>
+        </joint>
+      </xacro:if>
+      <!-- Position Drive: Head -->
+      <joint name="head_pan_joint">
+        <param name="id">21</param>
+        <command_interface name="position">
+            <param name="min">-1.570796327</param>
+            <param name="max">1.570796327</param>
+        </command_interface>
+        <command_interface name="velocity"/>
+        <state_interface name="position">
+          <param name="initial_value">0.0</param>
+        </state_interface>
+        <state_interface name="velocity"/>
+        <state_interface name="effort"/>
+      </joint>
+      <joint name="head_tilt_joint">
+        <param name="id">22</param>
+        <command_interface name="position">
+          <param name="min">-1.570796327</param>
+          <param name="max">0.570796327</param>
+        </command_interface>
+        <command_interface name="velocity"/>
+        <state_interface name="position">
+          <param name="initial_value">0.0</param>
+        </state_interface>
+        <state_interface name="velocity"/>
+        <state_interface name="effort"/>
+      </joint>
+    </ros2_control>
+  </xacro:macro>
 </robot>
