Commit message: update ros2_controll

File: sobit_pro_description/robots/sobit_pro_robot.urdf.xacro (robot description, xacro)
@@ -1,5 +1,4 @@
 <?xml version="1.0" ?>
-<robot name="sobit_pro"
-       xmlns:xacro="http://www.ros.org/wiki/xacro" >
+<robot name="sobit_pro" xmlns:xacro="http://www.ros.org/wiki/xacro">
   <!-- Add Common Xacro: transmissions, colors -->
   <xacro:include filename="$(find sobit_pro_description)/urdf/common.xacro" />
@@ -24,5 +23,6 @@
   <xacro:include filename="$(find sobit_pro_description)/urdf/sensor/realsense_d415.urdf.xacro" />
   <xacro:include filename="$(find urg_node)/urdf/hokuyo_ust.urdf.xacro" />
-  <xacro:include filename="$(find sobit_pro_description)/urdf/azure_kinect.urdf.xacro" />
+  <!-- <xacro:include filename="$(find sobit_pro_description)/urdf/azure_kinect.urdf.xacro" /> -->
+  <xacro:include filename="$(find azure_kinect_ros_driver)/urdf/azure_kinect.urdf.xacro" />
   <!-- <xacro:include filename="$(find azure_kinect_ros_driver)/urdf/azure_kinect.urdf.xacro" /> -->
   <!-- <xacro:include filename="$(find realsense2_description)/urdf/_l515.urdf.xacro" /> -->
@@ -33,6 +33,11 @@
   <xacro:arg name="enable_arm"  default="True" />
   <xacro:arg name="enable_head" default="True" />
-  <xacro:arg name="enable_gz"   default="False" />
-  <xacro:arg name="robot_namespace" default="sobit_pro" />
+  <!-- Add variables -->
+  <xacro:arg name="enable_gz"                 default="False" />
+  <xacro:arg name="enable_gz_lidar"           default="True" />
+  <xacro:arg name="robot_name"                default="sobit_pro" />
+  <!-- <xacro:controllers name="joints_control" enable_gz="$(arg enable_gz)" robot_name="$(arg robot_name)" /> -->
+  <!-- <xacro:open_manipulator_x_ros2_control name="open_manipulator_x_ros2_control" /> -->
+  <xacro:controllers name="joints_control" enable_gz="$(arg enable_gz)" robot_name="$(arg robot_name)" />
   <!-- enable_mb: true, enable_arm: true, enable_head: true -->
   <xacro:if value="${$(arg enable_mb) and $(arg enable_arm) and $(arg enable_head)}">

File: sobit_pro_description/urdf/controllers.urdf.xacro (robot description, xacro)
@@ -1,28 +1,17 @@
 <?xml version="1.0" encoding="UTF-8" ?>
-<!-- SOBIT Light (Dynamixel Control) -->
 <robot name="sobit_pro_controllers" xmlns:xacro="http://www.ros.org/wiki/xacro">
   <xacro:macro name="controllers" params="name enable_gz:=False robot_name:=sobit_pro">
-    <ros2_control name="${name}_arm" type="system">
-    <!-- <ros2_control name="joints_control" type="system"> -->
+    <ros2_control name="${name}" type="system">
       <hardware>
-        <xacro:if value="${$(arg enable_gz)}">
-          <plugin>ign_ros2_control/IgnitionSystem</plugin>
-          <!-- <plugin>gazebo_ros2_control/GazeboHardware</plugin> -->
-        </xacro:if>
-        <xacro:unless value="${$(arg enable_gz)}">
-          <plugin>dynamixel_hardware/DynamixelHardware</plugin>
-          <param name="usb_port">/dev/ttyUSB0</param>
-          <param name="baud_rate">1000000</param>
-          <param name="use_dummy">true</param>
-        </xacro:unless>
+        <plugin>dynamixel_hardware/DynamixelHardware</plugin>
+        <param name="usb_port">/dev/ttyUSB0</param>
+        <param name="baud_rate">1000000</param>
+        <!-- <param name="use_dummy">true</param> -->
       </hardware>
-      <!-- Position Drive: Arm -->
       <joint name="arm_shoulder_1_tilt_joint">
-        <xacro:unless value="${$(arg enable_gz)}">
-          <param name="id">11</param>
-        </xacro:unless>
+        <param name="id">11</param>
         <command_interface name="position">
-          <param name="min">-1.570796327</param>
-          <param name="max">1.570796327</param>
+          <param name="min">-1.57</param>
+          <param name="max">1.57</param>  <!-- 1.57 -->
         </command_interface>
         <command_interface name="velocity"/>
@@ -34,33 +23,25 @@
       </joint>
       <joint name="arm_shoulder_2_tilt_joint">
-        <xacro:unless value="${$(arg enable_gz)}">
-          <param name="id">12</param>
-        </xacro:unless>
-        <!-- <param name="mimic">arm_shoulder_pitch_joint</param>
-        <param name="multiplier">-1</param> -->
-        <!-- <command_interface name="position"/> -->
+        <param name="id">12</param>
         <command_interface name="position">
-          <param name="min">-1.570796327</param>
-          <param name="max">1.570796327</param>
+          <param name="min">-1.57</param>
+          <param name="max">1.57</param>  <!-- 1.57 -->
         </command_interface>
         <command_interface name="velocity"/>
         <state_interface name="position">
-          <param name="initial_value">1.57</param>
+          <param name="initial_value">0.0</param>
         </state_interface>
-        <!-- <state_interface name="position"/> -->
         <state_interface name="velocity"/>
         <state_interface name="effort"/>
       </joint>
       <joint name="arm_elbow_upper_1_tilt_joint">
-        <xacro:unless value="${$(arg enable_gz)}">
-          <param name="id">13</param>
-        </xacro:unless>
+        <param name="id">13</param>
         <command_interface name="position">
-          <param name="min">-1.570796327</param>
-          <param name="max">1.570796327</param>
+          <param name="min">-1.57</param>
+          <param name="max">1.57</param>  <!-- 1.57 -->
         </command_interface>
         <command_interface name="velocity"/>
         <state_interface name="position">
-          <param name="initial_value">-1.57</param>
+          <param name="initial_value">0.0</param>
         </state_interface>
         <state_interface name="velocity"/>
@@ -68,10 +49,8 @@
       </joint>
       <joint name="arm_elbow_upper_2_tilt_joint">
-        <xacro:unless value="${$(arg enable_gz)}">
-          <param name="id">14</param>
-        </xacro:unless>
+        <param name="id">14</param>
         <command_interface name="position">
-          <param name="min">-1.570796327</param>
-          <param name="max">1.570796327</param>
+          <param name="min">-1.57</param>
+          <param name="max">1.57</param>  <!-- 1.57 -->
         </command_interface>
         <command_interface name="velocity"/>
@@ -83,10 +62,8 @@
       </joint>
       <joint name="arm_elbow_lower_tilt_joint">
-        <xacro:unless value="${$(arg enable_gz)}">
-          <param name="id">15</param>
-        </xacro:unless>
+        <param name="id">15</param>
         <command_interface name="position">
-          <param name="min">-1.570796327</param>
-          <param name="max">1.570796327</param>
+          <param name="min">-1.57</param>
+          <param name="max">1.57</param>  <!-- 1.57 -->
         </command_interface>
         <command_interface name="velocity"/>
@@ -98,10 +75,8 @@
       </joint>
       <joint name="arm_elbow_lower_pan_joint">
-        <xacro:unless value="${$(arg enable_gz)}">
-          <param name="id">16</param>
-        </xacro:unless>
+        <param name="id">16</param>
         <command_interface name="position">
-          <param name="min">-1.570796327</param>
-          <param name="max">1.570796327</param>
+          <param name="min">-1.57</param>
+          <param name="max">1.57</param>  <!-- 1.57 -->
         </command_interface>
         <command_interface name="velocity"/>
@@ -113,10 +88,8 @@
       </joint>
       <joint name="arm_wrist_tilt_joint">
-        <xacro:unless value="${$(arg enable_gz)}">
-          <param name="id">17</param>
-        </xacro:unless>
+        <param name="id">17</param>
         <command_interface name="position">
-          <param name="min">-1.570796327</param>
-          <param name="max">1.570796327</param>
+          <param name="min">-1.57</param>
+          <param name="max">1.57</param>  <!-- 1.57 -->
         </command_interface>
         <command_interface name="velocity"/>
@@ -127,12 +100,9 @@
         <state_interface name="effort"/>
       </joint>
-      <!-- Position Drive: Hand -->
       <joint name="hand_joint">
-        <xacro:unless value="${$(arg enable_gz)}">
-          <param name="id">18</param>
-        </xacro:unless>
+        <param name="id">18</param>
         <command_interface name="position">
-            <param name="min">-1.570796327</param>
-            <param name="max">0.0</param>
+          <param name="min">-1.57</param>
+          <param name="max">0.0</param>  <!-- 1.57 -->
         </command_interface>
         <command_interface name="velocity"/>
@@ -143,21 +113,9 @@
         <state_interface name="effort"/>
       </joint>
-      <xacro:if value="${$(arg enable_gz)}">
-        <joint name="hand_sub_joint">
-          <param name="mimic">hand_joint</param>
-          <param name="multiplier">-1</param>
-          <command_interface name="position"/>
-          <command_interface name="velocity"/>
-          <state_interface name="position"/>
-          <state_interface name="velocity"/>
-          <state_interface name="effort"/>
-        </joint>
-      </xacro:if>
-      <!-- Position Drive: Head -->
       <joint name="head_pan_joint">
         <param name="id">21</param>
         <command_interface name="position">
-            <param name="min">-1.570796327</param>
-            <param name="max">1.570796327</param>
+          <param name="min">-1.57</param>
+          <param name="max">1.57</param>  <!-- 1.57 -->
         </command_interface>
         <command_interface name="velocity"/>
@@ -171,6 +129,6 @@
         <param name="id">22</param>
         <command_interface name="position">
-          <param name="min">-1.570796327</param>
-          <param name="max">0.570796327</param>
+          <param name="min">-1.57</param>
+          <param name="max">0.57</param>  <!-- 1.57 -->
         </command_interface>
         <command_interface name="velocity"/>

File: sobit_pro_description/urdf/sensor/azure_camera.urdf.xacro (robot description, xacro)
@@ -12,4 +12,7 @@
       <origin xyz="0.0 0 0.0" rpy="0 0 0"/>
     </xacro:azure_kinect> -->
+    <xacro:azure_kinect parent="${prefix}_base" tf_prefix="${prefix}_" add_cover="false">
+      <origin xyz="0.0 0 0.0" rpy="0 0 0"/>
+    </xacro:azure_kinect>
   </xacro:macro>
 </robot>

Commit message: update file

File: sobit_pro_description/robots/sobit_pro_robot.urdf.xacro (robot description, xacro)
@@ -5,5 +5,6 @@
   <xacro:include filename="$(find sobit_pro_description)/urdf/materials.urdf.xacro" />
   <xacro:include filename="$(find sobit_pro_description)/urdf/transmission.urdf.xacro" />
-  <xacro:include filename="$(find sobit_pro_description)/urdf/controllers.urdf.xacro" />
+  <xacro:include filename="$(find sobit_pro_description)/urdf/controllers_upper.urdf.xacro" />
+  <xacro:include filename="$(find sobit_pro_description)/urdf/controllers_lower.urdf.xacro" />
   <!-- Add URDF: links, joints -->
   <xacro:include filename="$(find sobit_pro_description)/urdf/base/base.urdf.xacro" />
@@ -11,5 +12,6 @@
   <xacro:include filename="$(find sobit_pro_description)/urdf/body/cover.urdf.xacro" />
   <xacro:include filename="$(find sobit_pro_description)/urdf/back/back.urdf.xacro" />
-  <!-- <xacro:include filename="$(find sobit_pro_description)/urdf/wheel/wheel.urdf.xacro" /> -->
+  <xacro:include filename="$(find sobit_pro_description)/urdf/wheel/wheel.urdf.xacro" />
+  <!-- <xacro:include filename="$(find sobit_pro_description)/urdf/wheel/wheel_2.urdf.xacro" /> -->
   <xacro:include filename="$(find sobit_pro_description)/urdf/arm/arm.urdf.xacro" />
   <xacro:include filename="$(find sobit_pro_description)/urdf/hand/hand.urdf.xacro" />
@@ -39,10 +41,11 @@
   <!-- <xacro:controllers name="joints_control" enable_gz="$(arg enable_gz)" robot_name="$(arg robot_name)" /> -->
   <!-- <xacro:open_manipulator_x_ros2_control name="open_manipulator_x_ros2_control" /> -->
-  <xacro:controllers name="joints_control" enable_gz="$(arg enable_gz)" robot_name="$(arg robot_name)" />
+  <xacro:controllers_DxUpper name="joints_control_upper" enable_gz="$(arg enable_gz)" robot_name="$(arg robot_name)" />
+  <xacro:controllers_DxLower name="joints_control_lower" enable_gz="$(arg enable_gz)" robot_name="$(arg robot_name)" />
   <!-- enable_mb: true, enable_arm: true, enable_head: true -->
   <xacro:if value="${$(arg enable_mb) and $(arg enable_arm) and $(arg enable_head)}">
     <xacro:base/>
     <xacro:plate prefix="plate" parent="base_link" />
-    <!-- <xacro:wheel prefix="wheel" parent="plate_middle_link" /> -->
+    <xacro:wheel prefix="wheel" parent="plate_middle_link" />
     <xacro:cover prefix="cover" parent="plate_top_link" />
     <xacro:back  prefix="back"  parent="plate_top_link" />
@@ -62,5 +65,5 @@
     <xacro:base/>
     <xacro:plate prefix="plate" parent="base_link" />
-    <!-- <xacro:wheel prefix="wheel" parent="plate_middle_link" /> -->
+    <xacro:wheel prefix="wheel" parent="plate_middle_link" />
     <xacro:cover prefix="cover" parent="plate_top_link" />
     <xacro:arm   prefix="arm"   parent="plate_top_link" />
@@ -75,5 +78,5 @@
     <xacro:base/>
     <xacro:plate prefix="plate" parent="base_link" />
-    <!-- <xacro:wheel prefix="wheel" parent="plate_middle_link" /> -->
+    <xacro:wheel prefix="wheel" parent="plate_middle_link" />
     <xacro:cover prefix="cover" parent="plate_top_link" />
     <xacro:back  prefix="back"  parent="plate_top_link" />
@@ -89,5 +92,5 @@
     <xacro:base/>
     <xacro:plate prefix="plate" parent="base_link" />
-    <!-- <xacro:wheel prefix="wheel" parent="plate_middle_link" /> -->
+    <xacro:wheel prefix="wheel" parent="plate_middle_link" />
     <xacro:cover prefix="cover" parent="plate_top_link" />
     <xacro:lidar prefix="lidar" parent="plate_bottom_link" />

File: sobit_pro_description/urdf/controllers_upper.urdf.xacro (robot description, xacro)
@@ -1,5 +1,5 @@
 <?xml version="1.0" encoding="UTF-8" ?>
 <robot name="sobit_pro_controllers" xmlns:xacro="http://www.ros.org/wiki/xacro">
-  <xacro:macro name="controllers" params="name enable_gz:=False robot_name:=sobit_pro">
+  <xacro:macro name="controllers_DxUpper" params="name enable_gz:=False robot_name:=sobit_pro">
     <ros2_control name="${name}" type="system">
       <hardware>

File: sobit_pro_description/urdf/wheel/wheel.urdf.xacro (robot description, xacro)
@@ -64,5 +64,5 @@
     </link>
   </xacro:macro>
-  <xacro:macro name="stack_wheel_drive" params="parent prefix number x_loc y_loc z_loc roll=0.0 pitch=0.0 yaw=0.0">
+  <!-- <xacro:macro name="stack_wheel_drive" params="parent prefix number x_loc y_loc z_loc roll=0.0 pitch=0.0 yaw=0.0">
     <joint name="wheel_${prefix}_drive_joint" type="continuous">
       <origin xyz="${x_loc+0.0019} ${y_loc} ${z_loc}" rpy="${roll} ${pitch} ${yaw}" />
@@ -94,5 +94,5 @@
       </inertial>
     </link>
-  </xacro:macro>
+  </xacro:macro> -->
   <xacro:macro name="wheel" params="parent prefix">
     <xacro:stack_wheel_steer_base parent="${parent}" prefix="f_l" number="1" x_loc= " ${0.210*cos(radians(45.))}" y_loc= " ${0.210*cos(radians(45.))}" z_loc="-0.019" />
@@ -104,8 +104,8 @@
     <xacro:stack_wheel_steer parent="wheel_b_r_steer_base_link" prefix="b_r" number="3" x_loc= "0.013875" y_loc= "0.0" z_loc="-0.032" />
     <xacro:stack_wheel_steer parent="wheel_f_r_steer_base_link" prefix="f_r" number="4" x_loc= "0.013875" y_loc= "0.0" z_loc="-0.032" />
-    <xacro:stack_wheel_drive parent="wheel_f_l_steer_link" prefix="f_l" number="1" x_loc= "0.02" y_loc= "0.0" z_loc="-0.118" />
+    <!-- <xacro:stack_wheel_drive parent="wheel_f_l_steer_link" prefix="f_l" number="1" x_loc= "0.02" y_loc= "0.0" z_loc="-0.118" />
     <xacro:stack_wheel_drive parent="wheel_b_l_steer_link" prefix="b_l" number="2" x_loc= "0.02" y_loc= "0.0" z_loc="-0.118" />
     <xacro:stack_wheel_drive parent="wheel_b_r_steer_link" prefix="b_r" number="3" x_loc= "0.02" y_loc= "0.0" z_loc="-0.118" />
-    <xacro:stack_wheel_drive parent="wheel_f_r_steer_link" prefix="f_r" number="4" x_loc= "0.02" y_loc= "0.0" z_loc="-0.118" />
+    <xacro:stack_wheel_drive parent="wheel_f_r_steer_link" prefix="f_r" number="4" x_loc= "0.02" y_loc= "0.0" z_loc="-0.118" /> -->
     <xacro:wheel_transmission prefix="${prefix}" />
   </xacro:macro>

Commit message: update control

File: sobit_pro_description/robots/sobit_pro_robot.urdf.xacro (robot description, xacro)
@@ -13,5 +13,5 @@
   <xacro:include filename="$(find sobit_pro_description)/urdf/back/back.urdf.xacro" />
   <xacro:include filename="$(find sobit_pro_description)/urdf/wheel/wheel.urdf.xacro" />
-  <!-- <xacro:include filename="$(find sobit_pro_description)/urdf/wheel/wheel_2.urdf.xacro" /> -->
+  <xacro:include filename="$(find sobit_pro_description)/urdf/wheel/wheel_2.urdf.xacro" />
   <xacro:include filename="$(find sobit_pro_description)/urdf/arm/arm.urdf.xacro" />
   <xacro:include filename="$(find sobit_pro_description)/urdf/hand/hand.urdf.xacro" />
@@ -42,5 +42,5 @@
   <!-- <xacro:open_manipulator_x_ros2_control name="open_manipulator_x_ros2_control" /> -->
   <xacro:controllers_DxUpper name="joints_control_upper" enable_gz="$(arg enable_gz)" robot_name="$(arg robot_name)" />
-  <xacro:controllers_DxLower name="joints_control_lower" enable_gz="$(arg enable_gz)" robot_name="$(arg robot_name)" />
+  <!-- <xacro:controllers_DxLower name="joints_control_lower" enable_gz="$(arg enable_gz)" robot_name="$(arg robot_name)" /> -->
   <!-- enable_mb: true, enable_arm: true, enable_head: true -->
   <xacro:if value="${$(arg enable_mb) and $(arg enable_arm) and $(arg enable_head)}">

File: sobit_pro_description/urdf/wheel/wheel_2.urdf.xacro (robot description, xacro)
@@ -2,7 +2,7 @@
 <robot name="sobit_pro"
        xmlns:xacro="http://ros.org/wiki/xacro">
-  <xacro:property name="M_PI" value="3.14159265359" />
+  <!-- <xacro:property name="M_PI" value="3.14159265359" />
   <xacro:include filename="$(find sobit_pro_description)/urdf/wheel/wheel.transmission.xacro" />
-  <xacro:include filename="$(find sobit_pro_description)/urdf/materials.urdf.xacro" />
+  <xacro:include filename="$(find sobit_pro_description)/urdf/materials.urdf.xacro" /> -->
   <xacro:macro name="stack_wheel_drive" params="parent prefix number x_loc y_loc z_loc roll=0.0 pitch=0.0 yaw=0.0">
     <joint name="wheel_${prefix}_drive_joint" type="continuous">
