Commit message: config + temp/wheel = this branch

File: sobit_pro_description/robots/sobit_pro_robot.urdf.xacro (robot description, xacro)
@@ -13,5 +13,5 @@
   <xacro:include filename="$(find sobit_pro_description)/urdf/back/back.urdf.xacro" />
   <xacro:include filename="$(find sobit_pro_description)/urdf/wheel/wheel.urdf.xacro" />
-  <xacro:include filename="$(find sobit_pro_description)/urdf/wheel/wheel_2.urdf.xacro" />
+  <!-- <xacro:include filename="$(find sobit_pro_description)/urdf/wheel/wheel_2.urdf.xacro" /> -->
   <xacro:include filename="$(find sobit_pro_description)/urdf/arm/arm.urdf.xacro" />
   <xacro:include filename="$(find sobit_pro_description)/urdf/hand/hand.urdf.xacro" />
@@ -42,5 +42,5 @@
   <!-- <xacro:open_manipulator_x_ros2_control name="open_manipulator_x_ros2_control" /> -->
   <xacro:controllers_DxUpper name="joints_control_upper" enable_gz="$(arg enable_gz)" robot_name="$(arg robot_name)" />
-  <!-- <xacro:controllers_DxLower name="joints_control_lower" enable_gz="$(arg enable_gz)" robot_name="$(arg robot_name)" /> -->
+  <xacro:controllers_DxLower name="joints_control_lower" enable_gz="$(arg enable_gz)" robot_name="$(arg robot_name)" />
   <!-- enable_mb: true, enable_arm: true, enable_head: true -->
   <xacro:if value="${$(arg enable_mb) and $(arg enable_arm) and $(arg enable_head)}">

File: sobit_pro_description/urdf/controllers_lower.urdf.xacro (robot description, xacro)
@@ -9,5 +9,5 @@
         <!-- <param name="use_dummy">true</param> -->
       </hardware>
-      <joint name="wheel_f_l_steer_joint">
+      <joint name="wheel_f_r_steer_joint">
         <param name="id">5</param>
         <command_interface name="position">
@@ -15,5 +15,5 @@
           <param name="max">1.57</param>  <!-- 1.57 -->
         </command_interface>
-        <command_interface name="velocity"/>
+        <!-- <command_interface name="velocity"/> -->
         <state_interface name="position">
           <param name="initial_value">0.0</param>
@@ -22,5 +22,5 @@
         <state_interface name="effort"/>
       </joint>
-      <joint name="wheel_f_r_steer_joint">
+      <joint name="wheel_f_l_steer_joint">
         <param name="id">6</param>
         <command_interface name="position">
@@ -28,5 +28,18 @@
           <param name="max">1.57</param>  <!-- 1.57 -->
         </command_interface>
-        <command_interface name="velocity"/>
+        <!-- <command_interface name="velocity"/> -->
+        <state_interface name="position">
+          <param name="initial_value">0.0</param>
+        </state_interface>
+        <state_interface name="velocity"/>
+        <state_interface name="effort"/>
+      </joint>
+      <joint name="wheel_b_r_steer_joint">
+        <param name="id">7</param>
+        <command_interface name="position">
+          <param name="min">-1.57</param>
+          <param name="max">1.57</param>  <!-- 1.57 -->
+        </command_interface>
+        <!-- <command_interface name="velocity"/> -->
         <state_interface name="position">
           <param name="initial_value">0.0</param>
@@ -36,17 +49,4 @@
       </joint>
       <joint name="wheel_b_l_steer_joint">
-        <param name="id">7</param>
-        <command_interface name="position">
-          <param name="min">-1.57</param>
-          <param name="max">1.57</param>  <!-- 1.57 -->
-        </command_interface>
-        <command_interface name="velocity"/>
-        <state_interface name="position">
-          <param name="initial_value">0.0</param>
-        </state_interface>
-        <state_interface name="velocity"/>
-        <state_interface name="effort"/>
-      </joint>
-      <joint name="wheel_b_r_steer_joint">
         <param name="id">8</param>
         <command_interface name="position">
@@ -54,5 +54,5 @@
           <param name="max">1.57</param>  <!-- 1.57 -->
         </command_interface>
-        <command_interface name="velocity"/>
+        <!-- <command_interface name="velocity"/> -->
         <state_interface name="position">
           <param name="initial_value">0.0</param>

File: sobit_pro_description/urdf/controllers_upper.urdf.xacro (robot description, xacro)
@@ -15,7 +15,7 @@
           <param name="max">1.57</param>  <!-- 1.57 -->
         </command_interface>
-        <command_interface name="velocity"/>
+        <!-- <command_interface name="velocity"/> -->
         <state_interface name="position">
-          <param name="initial_value">0.0</param>
+          <param name="initial_value">1.57</param>
         </state_interface>
         <state_interface name="velocity"/>
@@ -28,7 +28,7 @@
           <param name="max">1.57</param>  <!-- 1.57 -->
         </command_interface>
-        <command_interface name="velocity"/>
+        <!-- <command_interface name="velocity"/> -->
         <state_interface name="position">
-          <param name="initial_value">0.0</param>
+          <param name="initial_value">-1.57</param>
         </state_interface>
         <state_interface name="velocity"/>
@@ -41,7 +41,7 @@
           <param name="max">1.57</param>  <!-- 1.57 -->
         </command_interface>
-        <command_interface name="velocity"/>
+        <!-- <command_interface name="velocity"/> -->
         <state_interface name="position">
-          <param name="initial_value">0.0</param>
+          <param name="initial_value">1.57</param>
         </state_interface>
         <state_interface name="velocity"/>
@@ -54,7 +54,7 @@
           <param name="max">1.57</param>  <!-- 1.57 -->
         </command_interface>
-        <command_interface name="velocity"/>
+        <!-- <command_interface name="velocity"/> -->
         <state_interface name="position">
-          <param name="initial_value">0.0</param>
+          <param name="initial_value">-1.57</param>
         </state_interface>
         <state_interface name="velocity"/>
@@ -67,7 +67,7 @@
           <param name="max">1.57</param>  <!-- 1.57 -->
         </command_interface>
-        <command_interface name="velocity"/>
+        <!-- <command_interface name="velocity"/> -->
         <state_interface name="position">
-          <param name="initial_value">0.0</param>
+          <param name="initial_value">-1.57</param>
         </state_interface>
         <state_interface name="velocity"/>
@@ -80,5 +80,5 @@
           <param name="max">1.57</param>  <!-- 1.57 -->
         </command_interface>
-        <command_interface name="velocity"/>
+        <!-- <command_interface name="velocity"/> -->
         <state_interface name="position">
           <param name="initial_value">0.0</param>
@@ -93,7 +93,7 @@
           <param name="max">1.57</param>  <!-- 1.57 -->
         </command_interface>
-        <command_interface name="velocity"/>
+        <!-- <command_interface name="velocity"/> -->
         <state_interface name="position">
-          <param name="initial_value">0.0</param>
+          <param name="initial_value">-1.57</param>
         </state_interface>
         <state_interface name="velocity"/>
@@ -106,5 +106,5 @@
           <param name="max">0.0</param>  <!-- 1.57 -->
         </command_interface>
-        <command_interface name="velocity"/>
+        <!-- <command_interface name="velocity"/> -->
         <state_interface name="position">
           <param name="initial_value">0.0</param>
@@ -119,5 +119,5 @@
           <param name="max">1.57</param>  <!-- 1.57 -->
         </command_interface>
-        <command_interface name="velocity"/>
+        <!-- <command_interface name="velocity"/> -->
         <state_interface name="position">
           <param name="initial_value">0.0</param>
@@ -132,5 +132,5 @@
           <param name="max">0.57</param>  <!-- 1.57 -->
         </command_interface>
-        <command_interface name="velocity"/>
+        <!-- <command_interface name="velocity"/> -->
         <state_interface name="position">
           <param name="initial_value">0.0</param>

File: sobit_pro_description/urdf/wheel/wheel.urdf.xacro (robot description, xacro)
@@ -64,5 +64,5 @@
     </link>
   </xacro:macro>
-  <!-- <xacro:macro name="stack_wheel_drive" params="parent prefix number x_loc y_loc z_loc roll=0.0 pitch=0.0 yaw=0.0">
+  <xacro:macro name="stack_wheel_drive" params="parent prefix number x_loc y_loc z_loc roll=0.0 pitch=0.0 yaw=0.0">
     <joint name="wheel_${prefix}_drive_joint" type="continuous">
       <origin xyz="${x_loc+0.0019} ${y_loc} ${z_loc}" rpy="${roll} ${pitch} ${yaw}" />
@@ -94,5 +94,5 @@
       </inertial>
     </link>
-  </xacro:macro> -->
+  </xacro:macro>
   <xacro:macro name="wheel" params="parent prefix">
     <xacro:stack_wheel_steer_base parent="${parent}" prefix="f_l" number="1" x_loc= " ${0.210*cos(radians(45.))}" y_loc= " ${0.210*cos(radians(45.))}" z_loc="-0.019" />
@@ -104,8 +104,8 @@
     <xacro:stack_wheel_steer parent="wheel_b_r_steer_base_link" prefix="b_r" number="3" x_loc= "0.013875" y_loc= "0.0" z_loc="-0.032" />
     <xacro:stack_wheel_steer parent="wheel_f_r_steer_base_link" prefix="f_r" number="4" x_loc= "0.013875" y_loc= "0.0" z_loc="-0.032" />
-    <!-- <xacro:stack_wheel_drive parent="wheel_f_l_steer_link" prefix="f_l" number="1" x_loc= "0.02" y_loc= "0.0" z_loc="-0.118" />
+    <xacro:stack_wheel_drive parent="wheel_f_l_steer_link" prefix="f_l" number="1" x_loc= "0.02" y_loc= "0.0" z_loc="-0.118" />
     <xacro:stack_wheel_drive parent="wheel_b_l_steer_link" prefix="b_l" number="2" x_loc= "0.02" y_loc= "0.0" z_loc="-0.118" />
     <xacro:stack_wheel_drive parent="wheel_b_r_steer_link" prefix="b_r" number="3" x_loc= "0.02" y_loc= "0.0" z_loc="-0.118" />
-    <xacro:stack_wheel_drive parent="wheel_f_r_steer_link" prefix="f_r" number="4" x_loc= "0.02" y_loc= "0.0" z_loc="-0.118" /> -->
+    <xacro:stack_wheel_drive parent="wheel_f_r_steer_link" prefix="f_r" number="4" x_loc= "0.02" y_loc= "0.0" z_loc="-0.118" />
     <xacro:wheel_transmission prefix="${prefix}" />
   </xacro:macro>

Commit message: add xtion update ros2_control

File: sobit_pro_description/robots/sobit_pro_robot.urdf.xacro (robot description, xacro)
@@ -22,4 +22,6 @@
   <xacro:include filename="$(find sobit_pro_description)/urdf/sensor/realsense_d405.urdf.xacro" />
   <xacro:include filename="$(find sobit_pro_description)/urdf/sensor/realsense_d415.urdf.xacro" />
+  <xacro:include filename="$(find sobit_pro_description)/urdf/sensor/xtion.urdf.xacro" />
+  <xacro:include filename="$(find sobit_pro_description)/urdf/sensor/xtion_fixed.urdf.xacro" />
   <xacro:include filename="$(find urg_node)/urdf/hokuyo_ust.urdf.xacro" />
   <xacro:include filename="$(find azure_kinect_ros_driver)/urdf/azure_kinect.urdf.xacro" />
@@ -47,6 +49,7 @@
     <xacro:hand  prefix_hand="hand" prefix_finger="finger" parent="arm_wrist_tilt_link" />
     <xacro:lidar prefix="lidar" parent="plate_bottom_link" />
-    <xacro:azure_camera prefix="head_camera" parent="head_tilt_link" />
-    <xacro:matrix prefix="matrix" parent="head_camera_base" />
+    <!-- <xacro:azure_camera prefix="head_camera" parent="head_tilt_link" /> -->
+    <xacro:xtion_fixed prefix="head_camera" parent="head_tilt_link"/>
+    <!-- <xacro:matrix prefix="matrix" parent="head_camera_base" /> -->
     <!-- <xacro:realsense_l515 prefix="hand_camera" parent="arm_wrist_tilt_link" /> -->
     <xacro:realsense_d405 prefix="hand_camera" parent="arm_wrist_tilt_link" />

File: sobit_pro_description/urdf/head/head.urdf.xacro (robot description, xacro)
@@ -71,5 +71,6 @@
         <origin xyz="0.0 0.0 0.0" rpy="0.0 0.0 ${M_PI/2.0}" />
         <geometry>
-          <mesh filename="file://$(find sobit_pro_description)/meshes/head/head_camera_tilt.stl" scale="0.001 0.001 0.001" />
+          <!-- <mesh filename="file://$(find sobit_pro_description)/meshes/head/head_camera_tilt.stl" scale="0.001 0.001 0.001" /> -->
+          <mesh filename="file://$(find sobit_pro_description)/meshes/head/head_camera_tilt_xtion.stl" scale="0.001 0.001 0.001" />
         </geometry>
         <material name="black" />
