Commit message: [ADD] minimal bringup mode of only mobile base, arm and head. and debug of switch camera of [Xtion and AzureKinect]. Add Gazebo color image and depth image of Sim2Real for Xtion.

File: sobit_pro_description/robots/sobit_pro_robot.urdf.xacro (robot description, xacro)
@@ -15,5 +15,4 @@
   <xacro:include filename="$(find sobit_pro_description)/urdf/hand/hand.urdf.xacro" />
   <xacro:include filename="$(find sobit_pro_description)/urdf/head/head.urdf.xacro" />
-  <xacro:include filename="$(find sobit_pro_description)/urdf/sensor/azure_camera.urdf.xacro" />
   <xacro:include filename="$(find sobit_pro_description)/urdf/sensor/matrix.urdf.xacro" />
   <xacro:include filename="$(find sobit_pro_description)/urdf/sensor/mic.urdf.xacro" />
@@ -22,6 +21,4 @@
   <xacro:include filename="$(find sobit_pro_description)/urdf/sensor/realsense_d405.urdf.xacro" />
   <xacro:include filename="$(find sobit_pro_description)/urdf/sensor/realsense_d415.urdf.xacro" />
-  <xacro:include filename="$(find sobit_pro_description)/urdf/sensor/xtion.urdf.xacro" />
-  <xacro:include filename="$(find sobit_pro_description)/urdf/sensor/xtion_fixed.urdf.xacro" />
   <xacro:include filename="$(find urg_node)/urdf/hokuyo_ust.urdf.xacro" />
   <xacro:include filename="$(find azure_kinect_ros_driver)/urdf/azure_kinect.urdf.xacro" />
@@ -36,4 +33,6 @@
   <xacro:arg name="enable_gz"                 default="False" />
   <xacro:arg name="enable_gz_lidar"           default="True" />
+  <xacro:arg name="enable_gz_head_cam_color"  default="True" />
+  <xacro:arg name="enable_gz_head_cam_depth"  default="True" />
   <xacro:arg name="robot_name"                default="sobit_pro" />
   <xacro:arg name="head_camera_name"          default="xtion" />
@@ -50,13 +49,4 @@
     <xacro:hand  prefix_hand="hand" prefix_finger="finger" parent="arm_wrist_tilt_link" />
     <xacro:lidar prefix="lidar" parent="plate_bottom_link" />
-    <!-- <xacro:xtion_fixed prefix="head_camera" parent="head_tilt_link"/> -->
-    <!-- Xtion -->
-    <xacro:if value="$(eval head_camera_name == 'xtion')">
-      <xacro:xtion_fixed prefix="head_camera" parent="head_tilt_link"/>
-    </xacro:if>
-    <!-- Azure Kinect -->
-    <xacro:if value="$(eval head_camera_name == 'azure_kinect')">
-      <xacro:azure_camera prefix="camera" parent="head_tilt_link" />
-    </xacro:if>
     <!-- <xacro:matrix prefix="matrix" parent="head_camera_base" /> -->
     <!-- <xacro:realsense_l515 prefix="hand_camera" parent="arm_wrist_tilt_link" /> -->
@@ -87,5 +77,4 @@
     <xacro:mic   prefix="mic"   parent="back_base_link" />
     <xacro:lidar prefix="lidar" parent="plate_bottom_link" />
-    <xacro:azure_camera prefix="head_camera" parent="head_tilt_link" />
     <xacro:matrix prefix="matrix" parent="head_camera_base" />
     <xacro:realsense_d415 prefix="plate_top_camera" parent="plate_top_link" />
@@ -109,5 +98,4 @@
     <xacro:arm   prefix="arm"   parent="plate_top_link" />
     <xacro:hand  prefix_hand="hand" prefix_finger="finger" parent="arm_wrist_tilt_link" />
-    <!-- <xacro:azure_camera prefix="head_camera" parent="head_tilt_link" /> -->
     <xacro:matrix prefix="matrix" parent="head_camera_base" />
     <!-- <xacro:realsense_l515 prefix="hand_camera" parent="arm_wrist_tilt_link" /> -->
@@ -134,6 +122,18 @@
     <xacro:head  prefix="head"  parent="back_base_link" />
     <xacro:mic   prefix="mic"   parent="back_base_link" />
-    <!-- <xacro:azure_camera prefix="head_camera" parent="head_tilt_link" /> -->
     <xacro:matrix prefix="matrix" parent="head_camera_base" />
+  </xacro:if>
+  <xacro:if value="${$(arg enable_head)}">
+    <!-- Xtion -->
+    <xacro:if value="$(eval head_camera_name == 'xtion')">
+    <xacro:include filename="$(find sobit_pro_description)/urdf/sensor/xtion.urdf.xacro" />
+    <xacro:include filename="$(find sobit_pro_description)/urdf/sensor/xtion_fixed.urdf.xacro" />
+      <xacro:xtion_fixed prefix="head_camera" parent="head_tilt_link"/>
+    </xacro:if>
+    <!-- Azure Kinect -->
+    <xacro:if value="$(eval head_camera_name == 'azure_kinect')">
+      <xacro:include filename="$(find sobit_pro_description)/urdf/sensor/azure_camera.urdf.xacro" />
+      <xacro:azure_camera prefix="head_camera" parent="head_tilt_link" />
+    </xacro:if>
   </xacro:if>
   <!-- Add Dynamixel plugins -->
@@ -142,5 +142,5 @@
   <xacro:if value="${$(arg enable_gz)}">
     <xacro:include filename="$(find sobit_pro_description)/urdf/gazebo.urdf.xacro" />
-    <xacro:gazebo_sensors robot_name="$(arg robot_name)" />
+    <xacro:gazebo_sensors robot_name="$(arg robot_name)" enable_gz_lidar="$(arg enable_gz_lidar)" enable_gz_head_cam_color="$(arg enable_gz_head_cam_color)" enable_gz_head_cam_depth="$(arg enable_gz_head_cam_depth)" />
   </xacro:if>
 </robot>

File: sobit_pro_description/urdf/controllers.urdf.xacro (robot description, xacro)
@@ -1,5 +1,5 @@
 <?xml version="1.0" encoding="UTF-8" ?>
 <robot name="sobit_pro_controllers" xmlns:xacro="http://www.ros.org/wiki/xacro">
-  <xacro:macro name="controllers" params="name enable_gz:=False robot_name:=sobit_pro">
+  <xacro:macro name="controllers" params="name enable_gz:=False enable_mb:=True enable_arm:=True enable_head:=True robot_name:=sobit_pro">
     <ros2_control name="${name}" type="system">
       <hardware>
@@ -16,334 +16,340 @@
       </hardware>
        <!-- Position Drive - Arm -->
-      <joint name="arm_shoulder_1_tilt_joint">
-        <xacro:unless value="${$(arg enable_gz)}">
-          <param name="id">11</param>
-          <param name="control_mode">0</param>
-          <param name="interface">rs</param>
-        </xacro:unless>
-        <command_interface name="position">
-          <param name="min">-1.570796327</param>
-          <param name="max">1.570796327</param>
-        </command_interface>
-        <!-- <command_interface name="velocity"/> -->
-        <state_interface name="position">
-          <param name="initial_value">1.57</param>
-        </state_interface>
-        <state_interface name="velocity"/>
-        <state_interface name="effort"/>
-      </joint>
-      <joint name="arm_shoulder_2_tilt_joint">
-        <xacro:unless value="${$(arg enable_gz)}">
-          <param name="id">12</param>
-          <param name="control_mode">0</param>
-          <param name="interface">rs</param>
-        </xacro:unless>
-        <command_interface name="position">
-          <param name="min">-1.570796327</param>
-          <param name="max">1.570796327</param>
-        </command_interface>
-        <!-- <command_interface name="velocity"/> -->
-        <state_interface name="position">
-          <param name="initial_value">-1.57</param>
-        </state_interface>
-        <state_interface name="velocity"/>
-        <state_interface name="effort"/>
-      </joint>
-      <joint name="arm_elbow_upper_1_tilt_joint">
-        <xacro:unless value="${$(arg enable_gz)}">
-          <param name="id">13</param>
-          <param name="control_mode">0</param>
-          <param name="interface">rs</param>
-        </xacro:unless>
-        <command_interface name="position">
-          <param name="min">-1.570796327</param>
-          <param name="max">1.570796327</param>
-        </command_interface>
-        <!-- <command_interface name="velocity"/> -->
-        <state_interface name="position">
-          <param name="initial_value">1.57</param>
-        </state_interface>
-        <state_interface name="velocity"/>
-        <state_interface name="effort"/>
-      </joint>
-      <joint name="arm_elbow_upper_2_tilt_joint">
-        <xacro:unless value="${$(arg enable_gz)}">
-          <param name="id">14</param>
-          <param name="control_mode">0</param>
-          <param name="interface">rs</param>
-        </xacro:unless>
-        <command_interface name="position">
-          <param name="min">-1.570796327</param>
-          <param name="max">1.570796327</param>
-        </command_interface>
-        <!-- <command_interface name="velocity"/> -->
-        <state_interface name="position">
-          <param name="initial_value">-1.57</param>
-        </state_interface>
-        <state_interface name="velocity"/>
-        <state_interface name="effort"/>
-      </joint>
-      <joint name="arm_elbow_lower_tilt_joint">
-        <xacro:unless value="${$(arg enable_gz)}">
-          <param name="id">15</param>
-          <param name="control_mode">0</param>
-          <param name="interface">rs</param>
-        </xacro:unless>
-        <command_interface name="position">
-          <param name="min">-1.570796327</param>
-          <param name="max">1.570796327</param>
-        </command_interface>
-        <!-- <command_interface name="velocity"/> -->
-        <state_interface name="position">
-          <param name="initial_value">-1.57</param>
-        </state_interface>
-        <state_interface name="velocity"/>
-        <state_interface name="effort"/>
-      </joint>
-      <joint name="arm_elbow_lower_pan_joint">
-        <xacro:unless value="${$(arg enable_gz)}">
-          <param name="id">16</param>
-          <param name="control_mode">0</param>
-          <param name="interface">rs</param>
-        </xacro:unless>
-        <command_interface name="position">
-          <param name="min">-1.570796327</param>
-          <param name="max">1.570796327</param>
-        </command_interface>
-        <!-- <command_interface name="velocity"/> -->
-        <state_interface name="position">
-          <param name="initial_value">0.0</param>
-        </state_interface>
-        <state_interface name="velocity"/>
-        <state_interface name="effort"/>
-      </joint>
-      <joint name="arm_wrist_tilt_joint">
-        <xacro:unless value="${$(arg enable_gz)}">
-          <param name="id">17</param>
-          <param name="control_mode">0</param>
-          <param name="interface">rs</param>
-        </xacro:unless>
-        <command_interface name="position">
-          <param name="min">-1.570796327</param>
-          <param name="max">1.570796327</param>
-        </command_interface>
-        <!-- <command_interface name="velocity"/> -->
-        <state_interface name="position">
-          <param name="initial_value">-1.57</param>
-        </state_interface>
-        <state_interface name="velocity"/>
-        <state_interface name="effort"/>
-      </joint>
-      <!-- Position Drive: Hand -->
-      <joint name="hand_joint">
-        <xacro:unless value="${$(arg enable_gz)}">
-          <param name="id">18</param>
-          <param name="control_mode">6</param>
-          <param name="Goal_Current">150</param>
-          <param name="interface">rs</param>
-          <param name="gear_ratio">1.0</param>
-        </xacro:unless>
-        <command_interface name="position">
-          <param name="min">-1.570796327</param>
-          <param name="max">0.0</param>
-        </command_interface>
-        <!-- <command_interface name="velocity"/> -->
-        <state_interface name="position">
-          <param name="initial_value">0.0</param>
-        </state_interface>
-        <state_interface name="velocity"/>
-        <state_interface name="effort"/>
-      </joint>
-      <xacro:if value="${$(arg enable_gz)}">
-        <joint name="hand_inner_l_joint">
-          <param name="mimic">hand_joint</param>
-          <param name="multiplier">-1</param>
-          <command_interface name="position"/>
-          <!-- <command_interface name="velocity"/> -->
-          <state_interface name="position"/>
-          <state_interface name="velocity"/>
-          <state_interface name="effort"/>
-        </joint>
-          <!-- Outer Left -->
-        <joint name="hand_outer_l_joint">
-          <param name="mimic">hand_joint</param>
-          <param name="multiplier">-1</param> <!-- flip if needed -->
-          <command_interface name="position"/>
-          <state_interface name="position"/>
-          <state_interface name="velocity"/>
-          <state_interface name="effort"/>
-        </joint>
-        <!-- Outer Right -->
-        <joint name="hand_outer_r_joint">
-          <param name="mimic">hand_joint</param>
-          <param name="multiplier">1</param> <!-- same direction as hand_joint -->
-          <command_interface name="position"/>
-          <state_interface name="position"/>
-          <state_interface name="velocity"/>
-          <state_interface name="effort"/>
-      </joint>
-                <!-- Outer Left -->
-        <joint name="hand_finger_l_joint">
-          <param name="mimic">hand_joint</param>
-          <param name="multiplier">-0.5</param> <!-- flip if needed -->
-          <command_interface name="position"/>
-          <state_interface name="position"/>
-          <state_interface name="velocity"/>
-          <state_interface name="effort"/>
-        </joint>
-        <!-- Outer Right -->
-        <joint name="hand_finger_r_joint">
-          <param name="mimic">hand_joint</param>
-          <param name="multiplier">0.5</param> <!-- same direction as hand_joint -->
-          <command_interface name="position"/>
-          <state_interface name="position"/>
-          <state_interface name="velocity"/>
-          <state_interface name="effort"/>
-      </joint>
+      <xacro:if value="${$(arg enable_arm)}">
+        <joint name="arm_shoulder_1_tilt_joint">
+          <xacro:unless value="${$(arg enable_gz)}">
+            <param name="id">11</param>
+            <param name="control_mode">0</param>
+            <param name="interface">rs</param>
+          </xacro:unless>
+          <command_interface name="position">
+            <param name="min">-1.570796327</param>
+            <param name="max">1.570796327</param>
+          </command_interface>
+          <!-- <command_interface name="velocity"/> -->
+          <state_interface name="position">
+            <param name="initial_value">1.57</param>
+          </state_interface>
+          <state_interface name="velocity"/>
+          <state_interface name="effort"/>
+        </joint>
+        <joint name="arm_shoulder_2_tilt_joint">
+          <xacro:unless value="${$(arg enable_gz)}">
+            <param name="id">12</param>
+            <param name="control_mode">0</param>
+            <param name="interface">rs</param>
+          </xacro:unless>
+          <command_interface name="position">
+            <param name="min">-1.570796327</param>
+            <param name="max">1.570796327</param>
+          </command_interface>
+          <!-- <command_interface name="velocity"/> -->
+          <state_interface name="position">
+            <param name="initial_value">-1.57</param>
+          </state_interface>
+          <state_interface name="velocity"/>
+          <state_interface name="effort"/>
+        </joint>
+        <joint name="arm_elbow_upper_1_tilt_joint">
+          <xacro:unless value="${$(arg enable_gz)}">
+            <param name="id">13</param>
+            <param name="control_mode">0</param>
+            <param name="interface">rs</param>
+          </xacro:unless>
+          <command_interface name="position">
+            <param name="min">-1.570796327</param>
+            <param name="max">1.570796327</param>
+          </command_interface>
+          <!-- <command_interface name="velocity"/> -->
+          <state_interface name="position">
+            <param name="initial_value">1.57</param>
+          </state_interface>
+          <state_interface name="velocity"/>
+          <state_interface name="effort"/>
+        </joint>
+        <joint name="arm_elbow_upper_2_tilt_joint">
+          <xacro:unless value="${$(arg enable_gz)}">
+            <param name="id">14</param>
+            <param name="control_mode">0</param>
+            <param name="interface">rs</param>
+          </xacro:unless>
+          <command_interface name="position">
+            <param name="min">-1.570796327</param>
+            <param name="max">1.570796327</param>
+          </command_interface>
+          <!-- <command_interface name="velocity"/> -->
+          <state_interface name="position">
+            <param name="initial_value">-1.57</param>
+          </state_interface>
+          <state_interface name="velocity"/>
+          <state_interface name="effort"/>
+        </joint>
+        <joint name="arm_elbow_lower_tilt_joint">
+          <xacro:unless value="${$(arg enable_gz)}">
+            <param name="id">15</param>
+            <param name="control_mode">0</param>
+            <param name="interface">rs</param>
+          </xacro:unless>
+          <command_interface name="position">
+            <param name="min">-1.570796327</param>
+            <param name="max">1.570796327</param>
+          </command_interface>
+          <!-- <command_interface name="velocity"/> -->
+          <state_interface name="position">
+            <param name="initial_value">-1.57</param>
+          </state_interface>
+          <state_interface name="velocity"/>
+          <state_interface name="effort"/>
+        </joint>
+        <joint name="arm_elbow_lower_pan_joint">
+          <xacro:unless value="${$(arg enable_gz)}">
+            <param name="id">16</param>
+            <param name="control_mode">0</param>
+            <param name="interface">rs</param>
+          </xacro:unless>
+          <command_interface name="position">
+            <param name="min">-1.570796327</param>
+            <param name="max">1.570796327</param>
+          </command_interface>
+          <!-- <command_interface name="velocity"/> -->
+          <state_interface name="position">
+            <param name="initial_value">0.0</param>
+          </state_interface>
+          <state_interface name="velocity"/>
+          <state_interface name="effort"/>
+        </joint>
+        <joint name="arm_wrist_tilt_joint">
+          <xacro:unless value="${$(arg enable_gz)}">
+            <param name="id">17</param>
+            <param name="control_mode">0</param>
+            <param name="interface">rs</param>
+          </xacro:unless>
+          <command_interface name="position">
+            <param name="min">-1.570796327</param>
+            <param name="max">1.570796327</param>
+          </command_interface>
+          <!-- <command_interface name="velocity"/> -->
+          <state_interface name="position">
+            <param name="initial_value">-1.57</param>
+          </state_interface>
+          <state_interface name="velocity"/>
+          <state_interface name="effort"/>
+        </joint>
+        <!-- Position Drive: Hand -->
+        <joint name="hand_joint">
+          <xacro:unless value="${$(arg enable_gz)}">
+            <param name="id">18</param>
+            <param name="control_mode">6</param>
+            <param name="Goal_Current">150</param>
+            <param name="interface">rs</param>
+            <param name="gear_ratio">1.0</param>
+          </xacro:unless>
+          <command_interface name="position">
+            <param name="min">-1.570796327</param>
+            <param name="max">0.0</param>
+          </command_interface>
+          <!-- <command_interface name="velocity"/> -->
+          <state_interface name="position">
+            <param name="initial_value">0.0</param>
+          </state_interface>
+          <state_interface name="velocity"/>
+          <state_interface name="effort"/>
+        </joint>
+        <xacro:if value="${$(arg enable_gz)}">
+          <joint name="hand_inner_l_joint">
+            <param name="mimic">hand_joint</param>
+            <param name="multiplier">-1</param>
+            <command_interface name="position"/>
+            <!-- <command_interface name="velocity"/> -->
+            <state_interface name="position"/>
+            <state_interface name="velocity"/>
+            <state_interface name="effort"/>
+          </joint>
+            <!-- Outer Left -->
+          <joint name="hand_outer_l_joint">
+            <param name="mimic">hand_joint</param>
+            <param name="multiplier">-1</param> <!-- flip if needed -->
+            <command_interface name="position"/>
+            <state_interface name="position"/>
+            <state_interface name="velocity"/>
+            <state_interface name="effort"/>
+          </joint>
+          <!-- Outer Right -->
+          <joint name="hand_outer_r_joint">
+            <param name="mimic">hand_joint</param>
+            <param name="multiplier">1</param> <!-- same direction as hand_joint -->
+            <command_interface name="position"/>
+            <state_interface name="position"/>
+            <state_interface name="velocity"/>
+            <state_interface name="effort"/>
+        </joint>
+                  <!-- Outer Left -->
+          <joint name="hand_finger_l_joint">
+            <param name="mimic">hand_joint</param>
+            <param name="multiplier">-0.5</param> <!-- flip if needed -->
+            <command_interface name="position"/>
+            <state_interface name="position"/>
+            <state_interface name="velocity"/>
+            <state_interface name="effort"/>
+          </joint>
+          <!-- Outer Right -->
+          <joint name="hand_finger_r_joint">
+            <param name="mimic">hand_joint</param>
+            <param name="multiplier">0.5</param> <!-- same direction as hand_joint -->
+            <command_interface name="position"/>
+            <state_interface name="position"/>
+            <state_interface name="velocity"/>
+            <state_interface name="effort"/>
+        </joint>
+        </xacro:if>
       </xacro:if>
       <!-- Position Drive: Head -->
-      <joint name="head_pan_joint">
-        <xacro:unless value="${$(arg enable_gz)}">
-          <param name="id">21</param>
-          <param name="control_mode">0</param>
-          <param name="interface">rs</param>
-        </xacro:unless>
-        <command_interface name="position">
-          <param name="min">-1.570796327</param>
-          <param name="max">1.570796327</param>
-        </command_interface>
-        <!-- <command_interface name="velocity"/> -->
-        <state_interface name="position">
-          <param name="initial_value">0.0</param>
-        </state_interface>
-        <state_interface name="velocity"/>
-        <state_interface name="effort"/>
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