Commit message: [ADD] minimal bringup mode of only mobile base, arm and head. and debug of switch camera of [Xtion and AzureKinect]. Add Gazebo color image and depth image of Sim2Real for Xtion.

File: sobit_pro_description/urdf/gazebo.urdf.xacro (robot description, xacro)
@@ -1,76 +1,13 @@
 <?xml version="1.0" encoding="UTF-8" ?>
-<!-- SOBIT Light (Gazebo) -->
+<!-- SOBIT PRO (Gazebo) -->
 <robot name="sobit_pro_gazebo" xmlns:xacro="http://ros.org/wiki/xacro">
-  <xacro:macro name="gazebo_sensors" params="robot_name enable_gz_front_cam_color:=True enable_gz_back_cam_color:=True enable_gz_head_cam_color:=True enable_gz_head_cam_depth:=True enable_gz_hand_cam_color:=True enable_gz_hand_cam_depth:=True enable_gz_lidar:=True enable_gz_imu:=True">
-    <!-- Sensor - Base Front Camera (Color) -->
-    <!-- <xacro:if value="${enable_gz_front_cam_color}">
-      <gazebo reference="imu_link">
-        <sensor name="imu_sensor" type="imu">
-          <pose>0 0 0 0 0 0</pose>
-          <ignition_frame_id>${robot_name}/imu_link</ignition_frame_id>
-          <topic>${robot_name}/imu</topic>
-          <always_on>1</always_on>
-          <visualize>true</visualize>
-          <update_rate>1</update_rate>
-        </sensor>
-      </gazebo>
-    </xacro:if> -->
-    <!-- Sensor - Base Front Camera (Color) -->
-    <!-- <xacro:if value="${enable_gz_front_cam_color}">
-      <gazebo reference="camera_front_link">
-        <sensor name="base_front_camera_color" type="camera">
-          <pose>0 0 ${0.0175/2} ${M_PI/2} -${M_PI/2} 0 </pose>
-          <ignition_frame_id>${robot_name}/base_front_camera_color</ignition_frame_id>
-          <topic>${robot_name}/base_front_camera/color</topic>
-          <always_on>1</always_on>
-          <visualize>true</visualize>
-          <update_rate>1</update_rate>
-          <camera name="base_front_camera">
-            <horizontal_fov>1.21126</horizontal_fov>
-            <image>
-              <width>640</width>
-              <height>480</height>
-              <format>RGB_INT8</format>
-            </image>
-            <clip>
-              <near>0.1</near>
-              <far>10</far>
-            </clip>
-          </camera>
-        </sensor>
-      </gazebo>
-    </xacro:if> -->
-    <!-- Sensor - Base Back Camera (Color) -->
-    <!-- <xacro:if value="${enable_gz_back_cam_color}">
-      <gazebo reference="camera_back_link">
-        <sensor name="base_back_camera_color" type="camera">
-          <pose>0 0 ${0.0175/2} ${M_PI/2} -${M_PI/2} 0 </pose>
-          <ignition_frame_id>${robot_name}/camera_back_link</ignition_frame_id>
-          <topic>${robot_name}/base_back_camera/color</topic>
-          <always_on>1</always_on>
-          <visualize>true</visualize>
-          <update_rate>1</update_rate>
-          <camera name="base_back_camera">
-            <horizontal_fov>1.21126</horizontal_fov>
-            <image>
-              <width>640</width>
-              <height>480</height>
-              <format>RGB_INT8</format>
-            </image>
-            <clip>
-              <near>0.1</near>
-              <far>10</far>
-            </clip>
-          </camera>
-        </sensor>
-      </gazebo>
-    </xacro:if> -->
+  <xacro:macro name="gazebo_sensors" params="robot_name enable_gz_head_cam_color:=True enable_gz_head_cam_depth:=True enable_gz_lidar:=True">
     <!-- Sensor - Head Camera (Color) -->
-    <!-- <xacro:if value="${enable_gz_head_cam_color}">
-      <gazebo reference="head_camera_color_optical_frame">
+    <xacro:if value="${enable_gz_head_cam_color}">
+      <gazebo reference="head_camera_link">
         <sensor name="head_camera_color" type="camera">
-          <pose>0 0 ${0.0175/2} ${M_PI/2} -${M_PI/2} 0 </pose>
-          <ignition_frame_id>${robot_name}/head_camera_color_optical_frame</ignition_frame_id>
-          <topic>${robot_name}/head_camera/color</topic>
+          <pose>0.0 0.0 ${0.0175/2} ${M_PI/2} -${M_PI/2} 0.0</pose>
+          <ignition_frame_id>${robot_name}/head_camera_link</ignition_frame_id>
+          <topic>${robot_name}/head_camera/rgb/image_raw</topic>
           <always_on>1</always_on>
           <visualize>true</visualize>
@@ -90,12 +27,12 @@
         </sensor>
       </gazebo>
-    </xacro:if> -->
+    </xacro:if>
     <!-- Sensor - Head Camera (Depth) -->
-    <!-- <xacro:if value="${enable_gz_head_cam_depth}">
+    <xacro:if value="${enable_gz_head_cam_depth}">
       <gazebo reference="head_camera_depth_optical_frame">
         <sensor name="head_camera_depth" type="depth">
-          <pose>0 0 ${0.0175/2} ${M_PI/2} -${M_PI/2} 0 </pose>
+          <pose>0.0 0.0 ${0.0175/2} ${M_PI/2} -${M_PI/2} 0.0</pose>
           <ignition_frame_id>${robot_name}/head_camera_depth_optical_frame</ignition_frame_id>
-          <topic>${robot_name}/head_camera/depth</topic>
+          <topic>${robot_name}/head_camera/depth_registered/image_raw</topic>
           <always_on>1</always_on>
           <visualize>true</visualize>
@@ -104,6 +41,6 @@
             <horizontal_fov>1.48702</horizontal_fov>
             <image>
-              <width>1280</width>
-              <height>720</height>
+              <width>640</width>
+              <height>480</height>
             </image>
             <clip>
@@ -114,54 +51,5 @@
         </sensor>
       </gazebo>
-    </xacro:if> -->
-    <!-- Sensor - Hand Camera (Color) -->
-    <!-- <xacro:if value="${enable_gz_hand_cam_color}">
-      <gazebo reference="hand_camera_color_optical_frame">
-        <sensor name="hand_camera_color" type="camera">
-          <pose>0 0 ${0.0175/2} ${M_PI/2} -${M_PI/2} 0 </pose>
-          <ignition_frame_id>${robot_name}/hand_camera_color_optical_frame</ignition_frame_id>
-          <topic>${robot_name}/hand_camera/color</topic>
-          <always_on>1</always_on>
-          <visualize>true</visualize>
-          <update_rate>1</update_rate>
-          <camera name="hand_camera_color">
-            <horizontal_fov>1.21126</horizontal_fov>
-            <image>
-              <width>640</width>
-              <height>480</height>
-              <format>RGB_INT8</format>
-            </image>
-            <clip>
-              <near>0.1</near>
-              <far>10</far>
-            </clip>
-          </camera>
-        </sensor>
-      </gazebo>
-    </xacro:if> -->
-    <!-- Sensor - Hand Camera (Depth) -->
-    <!-- <xacro:if value="${enable_gz_hand_cam_depth}">
-      <gazebo reference="hand_camera_depth_optical_frame">
-        <sensor name="hand_camera_depth" type="depth">
-          <pose>0 0 ${0.0175/2} ${M_PI/2} -${M_PI/2} 0 </pose>
-          <ignition_frame_id>${robot_name}/hand_camera_depth_optical_frame</ignition_frame_id>
-          <topic>${robot_name}/hand_camera/depth</topic>
-          <always_on>1</always_on>
-          <visualize>true</visualize>
-          <update_rate>1</update_rate>
-          <camera name="head_camera_depth">
-            <horizontal_fov>1.48702</horizontal_fov>
-            <image>
-              <width>1280</width>
-              <height>720</height>
-            </image>
-            <clip>
-              <near>0.1</near>
-              <far>10</far>
-            </clip>
-          </camera>
-        </sensor>
-      </gazebo>
-    </xacro:if> -->
+    </xacro:if>
     <!-- Sensor - LiDAR -->
     <xacro:if value="${enable_gz_lidar}">

Commit message: New branch created for jazzy

File: sobit_pro_description/robots/sobit_pro_robot.urdf.xacro (robot description, xacro)
@@ -22,5 +22,4 @@
   <xacro:include filename="$(find sobit_pro_description)/urdf/sensor/realsense_d415.urdf.xacro" />
   <xacro:include filename="$(find urg_node)/urdf/hokuyo_ust.urdf.xacro" />
-  <xacro:include filename="$(find azure_kinect_ros_driver)/urdf/azure_kinect.urdf.xacro" />
   <!-- <xacro:include filename="$(find realsense2_description)/urdf/_l515.urdf.xacro" /> -->
   <xacro:include filename="$(find realsense2_description)/urdf/_d405.urdf.xacro" />
@@ -48,5 +47,5 @@
     <xacro:arm   prefix="arm"   parent="plate_top_link" />
     <xacro:hand  prefix_hand="hand" prefix_finger="finger" parent="arm_wrist_tilt_link" />
-    <xacro:lidar prefix="lidar" parent="plate_bottom_link" />
+    <xacro:lidar prefix="lidar" parent="plate_bottom_link" robot_name="$(arg robot_name)" />
     <!-- <xacro:matrix prefix="matrix" parent="head_camera_base" /> -->
     <!-- <xacro:realsense_l515 prefix="hand_camera" parent="arm_wrist_tilt_link" /> -->
@@ -62,5 +61,5 @@
     <xacro:arm   prefix="arm"   parent="plate_top_link" />
     <xacro:hand  prefix_hand="hand" prefix_finger="finger" parent="arm_wrist_tilt_link" />
-    <xacro:lidar prefix="lidar" parent="plate_bottom_link" />
+    <xacro:lidar prefix="lidar" parent="plate_bottom_link" robot_name="$(arg robot_name)" />
     <!-- <xacro:realsense_l515 prefix="hand_camera" parent="arm_wrist_tilt_link" /> -->
     <xacro:realsense_d405 prefix="hand_camera" parent="arm_wrist_tilt_link" />
@@ -76,5 +75,5 @@
     <xacro:head  prefix="head"  parent="back_base_link" />
     <xacro:mic   prefix="mic"   parent="back_base_link" />
-    <xacro:lidar prefix="lidar" parent="plate_bottom_link" />
+    <xacro:lidar prefix="lidar" parent="plate_bottom_link" robot_name="$(arg robot_name)" />
     <xacro:matrix prefix="matrix" parent="head_camera_base" />
     <xacro:realsense_d415 prefix="plate_top_camera" parent="plate_top_link" />
@@ -86,5 +85,5 @@
     <xacro:wheel prefix="wheel" parent="plate_middle_link" />
     <xacro:cover prefix="cover" parent="plate_top_link" />
-    <xacro:lidar prefix="lidar" parent="plate_bottom_link" />
+    <xacro:lidar prefix="lidar" parent="plate_bottom_link" robot_name="$(arg robot_name)" />
   </xacro:if>
   <!-- enable_mb (false), enable_arm (true), enable_head (true) -->
@@ -133,4 +132,5 @@
     <!-- Azure Kinect -->
     <xacro:if value="$(eval head_camera_name == 'azure_kinect')">
+      <xacro:include filename="$(find azure_kinect_ros_driver)/urdf/azure_kinect.urdf.xacro" />
       <xacro:include filename="$(find sobit_pro_description)/urdf/sensor/azure_camera.urdf.xacro" />
       <xacro:azure_camera prefix="head_camera" parent="head_tilt_link" />

File: sobit_pro_description/urdf/controllers.urdf.xacro (robot description, xacro)
@@ -5,5 +5,6 @@
       <hardware>
         <xacro:if value="${$(arg enable_gz)}">
-          <plugin>ign_ros2_control/IgnitionSystem</plugin>
+          <!-- <plugin>ign_ros2_control/IgnitionSystem</plugin> -->
+          <plugin>gz_ros2_control/GazeboSimSystem</plugin>
         </xacro:if>
         <xacro:unless value="${$(arg enable_gz)}">
@@ -353,10 +354,11 @@
       </xacro:if>
     </ros2_control>
-    <!-- Ignition ROS2 Control -->
+    <!-- Gazebo Sim ROS2 Control -->
     <xacro:if value="${$(arg enable_gz)}">
       <gazebo>
-        <plugin filename="ign_ros2_control-system" name="ign_ros2_control::IgnitionROS2ControlPlugin">
+        <!-- <plugin filename="ign_ros2_control-system" name="ign_ros2_control::IgnitionROS2ControlPlugin"> -->
+        <plugin filename="gz_ros2_control-system" name="gz_ros2_control::GazeboSimROS2ControlPlugin">
           <ros>
-            <namespace>${robot_name}</namespace>
+            <namespace>$(arg robot_name)</namespace>
           </ros>
           <parameters>$(find sobit_pro_control)/config/controllers.yaml</parameters>

File: sobit_pro_description/urdf/gazebo.urdf.xacro (robot description, xacro)
@@ -8,5 +8,6 @@
         <sensor name="head_camera_color" type="camera">
           <pose>0.0 0.0 ${0.0175/2} ${M_PI/2} -${M_PI/2} 0.0</pose>
-          <ignition_frame_id>${robot_name}/head_camera_link</ignition_frame_id>
+          <!-- <ignition_frame_id>${robot_name}/head_camera_link</ignition_frame_id> -->
+          <gz_frame_id>${robot_name}/head_camera_link</gz_frame_id>
           <topic>${robot_name}/head_camera/rgb/image_raw</topic>
           <always_on>1</always_on>
@@ -33,5 +34,6 @@
         <sensor name="head_camera_depth" type="depth">
           <pose>0.0 0.0 ${0.0175/2} ${M_PI/2} -${M_PI/2} 0.0</pose>
-          <ignition_frame_id>${robot_name}/head_camera_link</ignition_frame_id>
+          <!-- <ignition_frame_id>${robot_name}/head_camera_link</ignition_frame_id> -->
+          <gz_frame_id>${robot_name}/head_camera_link</gz_frame_id>
           <topic>${robot_name}/head_camera/depth_registered/image_raw</topic>
           <always_on>1</always_on>
@@ -57,5 +59,6 @@
         <sensor name="lidar" type="gpu_lidar">
           <pose>0 0 0 0 0 0</pose>
-          <ignition_frame_id>${robot_name}/lidar_laser</ignition_frame_id>
+          <!-- <ignition_frame_id>${robot_name}/lidar_laser</ignition_frame_id> -->
+          <gz_frame_id>${robot_name}/lidar_laser</gz_frame_id>
           <!-- <qos>
             <topic name=${robot_name}/scan>

File: sobit_pro_description/urdf/sensor/lidar.urdf.xacro (robot description, xacro)
@@ -2,5 +2,5 @@
 <robot name="sobit_pro"
        xmlns:xacro="http://ros.org/wiki/xacro">
-  <xacro:macro name="lidar" params="prefix parent">
+  <xacro:macro name="lidar_edge" params="prefix parent robot_name">
     <joint name="${prefix}_base_joint" type="fixed">
       <parent link="${parent}" />
@@ -30,7 +30,10 @@
       </inertial>
     </link>
-    <xacro:hokuyo_ust_mount prefix="${prefix}" parent="${prefix}_base_link" topic="/scan" >
+    <xacro:hokuyo_ust_mount prefix="${prefix}" parent="${prefix}_base_link" topic="${prefix}/scan" robot_name="${robot_name}" >
       <origin xyz="0.067 0.0 0.0" rpy="0.0 0.0 0.0" />
     </xacro:hokuyo_ust_mount>
   </xacro:macro>
+  <xacro:macro name="lidar" params="parent prefix robot_name">
+    <xacro:lidar_edge prefix="${prefix}" parent="${parent}" robot_name="${robot_name}"/>
+  </xacro:macro>
 </robot>

Commit message: [FIX] update femtobolt/mic description meshes and alignment

File: sobit_pro_description/robots/sobit_pro_robot.urdf.xacro (robot description, xacro)
@@ -136,4 +136,9 @@
       <xacro:azure_camera prefix="head_camera" parent="head_tilt_link" />
     </xacro:if>
+    <!-- Orbbec FemtoBolt -->
+    <xacro:if value="$(eval head_camera_name == 'femtobolt' or head_camera_name == 'orbbec_femtobolt')">
+      <xacro:include filename="$(find sobit_pro_description)/urdf/sensor/femtobolt_camera.urdf.xacro" />
+      <xacro:femtobolt_camera prefix="head_camera" parent="head_tilt_link" />
+    </xacro:if>
   </xacro:if>
   <!-- Add Dynamixel plugins -->

File: sobit_pro_description/urdf/hand/hand.urdf.xacro (robot description, xacro)
@@ -43,5 +43,5 @@
       <axis xyz="0.0 0.0 1.0" />
       <limit lower="0" upper="${M_PI/2.0}" effort="1.0" velocity="4.796165"/>
-      <mimic joint="${prefix_hand}_joint" multiplier="1" offset="0" />
+      <mimic joint="${prefix_hand}_joint" multiplier="-1.0" offset="0" />
       <!-- <dynamics damping="50.0" friction="5.0"/> -->
     </joint>
@@ -104,5 +104,5 @@
       <origin xyz="0.043193 0.04015 0.0282231" rpy="0.0 0.0 0.0" />
       <axis xyz="0.0 0.0 1.0" />
-      <!-- <mimic joint="{prefix_hand}_joint" multiplier="1.0" offset="0" /> -->
+      <mimic joint="${prefix_hand}_joint" multiplier="-1.0" offset="0" />
       <limit lower="0" upper="${M_PI/2.0}" effort="1.0" velocity="4.796165"/>
     </joint>

File: sobit_pro_description/urdf/sensor/mic.urdf.xacro (robot description, xacro)
@@ -2,32 +2,37 @@
 <robot name="sobit_pro"
        xmlns:xacro="http://ros.org/wiki/xacro">
-  <xacro:macro name="mic" params="prefix parent">
+  <xacro:macro name="mic" params="prefix parent
+                                  mic_mount_offset_xyz:='0.0 0.0 0.5400'
+                                  mic_mount_visual_xyz:='0.017 0.015 0.12'
+                                  mic_mount_visual_rpy:='0.0 0.0 ${-M_PI/2.0}'
+                                  mic_on_mount_xyz:='0.0 0.005 0.280'
+                                  mic_on_mount_rpy:='0.0 0.0 0.0'">
     <joint name="${prefix}_base_joint" type="fixed">
       <parent link="${parent}" />
       <child link="${prefix}_base_link" />
-      <origin xyz="0.0 0.0 0.5400" rpy="0.0 0.0 0.0" />
+      <origin xyz="${mic_mount_offset_xyz}" rpy="0.0 0.0 0.0" />
     </joint>
     <link name="${prefix}_base_link">
       <visual>
-        <origin xyz="0.0 0.0 0.0" rpy="${M_PI/2} 0.0 ${M_PI}" />
+        <origin xyz="${mic_mount_visual_xyz}" rpy="${mic_mount_visual_rpy}" />
         <geometry>
-          <mesh filename="file://$(find sobit_pro_description)/meshes/sensor/mic_base.stl" scale="0.001 0.001 0.001" />
+          <mesh filename="file://$(find sobit_pro_description)/meshes/sensor/mic_mount.stl" scale="1.0 1.0 1.0" />
         </geometry>
         <material name="black" />
       </visual>
       <collision>
-        <origin xyz="0.0 ${(0.02-0.1146-0.0146)/2} -${0.02/2}" rpy="0.0 0.0 0.0" />
+        <origin xyz="-0.015 -0.0042 0.0005" rpy="0.0 0.0 0.0" />
         <geometry>
-          <box size="0.0292 ${0.1146+0.0146} 0.03"/>
+          <box size="0.03 0.3517 0.0655"/>
         </geometry>
         <material name="black" />
       </collision>
       <inertial>
-        <origin xyz="0.0 ${(0.02-0.1146-0.0146)/2} -${0.02/2}" rpy="0.0 0.0 0.0" />
+        <origin xyz="-0.015 -0.0042 0.0005" rpy="0.0 0.0 0.0" />
         <!-- APPROX -->
         <mass value="0.15" />
-        <inertia ixx="${1/12*0.15*(0.0292**2+0.03**2)}"            ixy="0.0" ixz="0.0"
-                 iyy="${1/12*0.15*((0.1146+0.0146)**2+0.03**2)}"   iyz="0.0"
-                 izz="${1/12*0.15*(0.0292**2+(0.1146+0.0146)**2)}" />
+        <inertia ixx="${1/12*0.15*(0.3517**2+0.0655**2)}" ixy="0.0" ixz="0.0"
+                 iyy="${1/12*0.15*(0.03**2+0.0655**2)}"   iyz="0.0"
+                 izz="${1/12*0.15*(0.03**2+0.3517**2)}" />
       </inertial>
     </link>
@@ -35,5 +40,5 @@
       <parent link="${prefix}_base_link" />
       <child link="${prefix}_link" />
-      <origin xyz="0.0 -0.099 0.0240" rpy="0.0 0.0 0.0" />
+      <origin xyz="${mic_on_mount_xyz}" rpy="${mic_on_mount_rpy}" />
     </joint>
     <link name="${prefix}_link">
