Commit message: [FIX]: Controllers and action server split (sobit_light-based)

File: sobit_pro_description/robots/sobit_pro_robot.urdf.xacro (robot description, xacro)
@@ -30,4 +30,5 @@
   <xacro:arg name="enable_arm"  default="True" />
   <xacro:arg name="enable_head" default="True" />
+  <xacro:arg name="enable_hand" default="True" />
   <!-- Add variables -->
   <xacro:arg name="enable_gz"                 default="False" />
@@ -47,5 +48,7 @@
     <xacro:mic   prefix="mic"   parent="back_base_link" />
     <xacro:arm   prefix="arm"   parent="plate_top_link" />
-    <xacro:hand  prefix_hand="hand" prefix_finger="finger" parent="arm_wrist_tilt_link" />
+    <xacro:if value="${$(arg enable_hand)}">
+      <xacro:hand  prefix_hand="hand" prefix_finger="finger" parent="arm_wrist_tilt_link" />
+    </xacro:if>
     <xacro:lidar prefix="lidar" parent="plate_bottom_link" />
     <!-- <xacro:matrix prefix="matrix" parent="head_camera_base" /> -->
@@ -61,5 +64,7 @@
     <xacro:cover prefix="cover" parent="plate_top_link" />
     <xacro:arm   prefix="arm"   parent="plate_top_link" />
-    <xacro:hand  prefix_hand="hand" prefix_finger="finger" parent="arm_wrist_tilt_link" />
+    <xacro:if value="${$(arg enable_hand)}">
+      <xacro:hand  prefix_hand="hand" prefix_finger="finger" parent="arm_wrist_tilt_link" />
+    </xacro:if>
     <xacro:lidar prefix="lidar" parent="plate_bottom_link" />
     <!-- <xacro:realsense_l515 prefix="hand_camera" parent="arm_wrist_tilt_link" /> -->
@@ -97,5 +102,7 @@
     <xacro:mic   prefix="mic"   parent="back_base_link" />
     <xacro:arm   prefix="arm"   parent="plate_top_link" />
-    <xacro:hand  prefix_hand="hand" prefix_finger="finger" parent="arm_wrist_tilt_link" />
+    <xacro:if value="${$(arg enable_hand)}">
+      <xacro:hand  prefix_hand="hand" prefix_finger="finger" parent="arm_wrist_tilt_link" />
+    </xacro:if>
     <xacro:matrix prefix="matrix" parent="head_camera_base" />
     <!-- <xacro:realsense_l515 prefix="hand_camera" parent="arm_wrist_tilt_link" /> -->
@@ -109,5 +116,7 @@
     <xacro:cover prefix="cover" parent="plate_top_link" />
     <xacro:arm   prefix="arm"   parent="plate_top_link" />
-    <xacro:hand  prefix_hand="hand" prefix_finger="finger" parent="arm_wrist_tilt_link" />
+    <xacro:if value="${$(arg enable_hand)}">
+      <xacro:hand  prefix_hand="hand" prefix_finger="finger" parent="arm_wrist_tilt_link" />
+    </xacro:if>
     <!-- <xacro:realsense_l515 prefix="hand_camera" parent="arm_wrist_tilt_link" /> -->
     <xacro:realsense_d405 prefix="hand_camera" parent="arm_wrist_tilt_link" />
@@ -143,5 +152,5 @@
   </xacro:if>
   <!-- Add Dynamixel plugins -->
-  <xacro:controllers name="joints_control" enable_gz="$(arg enable_gz)" robot_name="$(arg robot_name)" />
+  <xacro:controllers name="joints_control" enable_gz="$(arg enable_gz)" enable_hand="$(arg enable_hand)" robot_name="$(arg robot_name)" />
   <!-- Add Gazebo plugins -->
   <xacro:if value="${$(arg enable_gz)}">

File: sobit_pro_description/urdf/controllers.urdf.xacro (robot description, xacro)
@@ -1,5 +1,5 @@
 <?xml version="1.0" encoding="UTF-8" ?>
 <robot name="sobit_pro_controllers" xmlns:xacro="http://www.ros.org/wiki/xacro">
-  <xacro:macro name="controllers" params="name enable_gz:=False enable_mb:=True enable_arm:=True enable_head:=True robot_name:=sobit_pro">
+  <xacro:macro name="controllers" params="name enable_gz:=False enable_mb:=True enable_arm:=True enable_head:=True enable_hand:=True robot_name:=sobit_pro">
     <ros2_control name="${name}" type="system">
       <hardware>
@@ -136,70 +136,72 @@
           <state_interface name="effort"/>
         </joint>
-        <!-- Position Drive: Hand -->
-        <joint name="hand_joint">
-          <xacro:unless value="${$(arg enable_gz)}">
-            <param name="id">18</param>
-            <param name="control_mode">6</param>
-            <param name="Goal_Current">150</param>
-            <param name="interface">rs</param>
-            <param name="gear_ratio">1.0</param>
-          </xacro:unless>
-          <command_interface name="position">
-            <param name="min">-1.570796327</param>
-            <param name="max">0.0</param>
-          </command_interface>
-          <!-- <command_interface name="velocity"/> -->
-          <state_interface name="position">
-            <param name="initial_value">0.0</param>
-          </state_interface>
-          <state_interface name="velocity"/>
-          <state_interface name="effort"/>
-        </joint>
-        <xacro:if value="${$(arg enable_gz)}">
-          <joint name="hand_inner_l_joint">
-            <param name="mimic">hand_joint</param>
-            <param name="multiplier">-1</param>
-            <command_interface name="position"/>
+        <xacro:if value="${$(arg enable_hand)}">
+          <!-- Position Drive: Hand -->
+          <joint name="hand_joint">
+            <xacro:unless value="${$(arg enable_gz)}">
+              <param name="id">18</param>
+              <param name="control_mode">6</param>
+              <param name="Goal_Current">150</param>
+              <param name="interface">rs</param>
+              <param name="gear_ratio">1.0</param>
+            </xacro:unless>
+            <command_interface name="position">
+              <param name="min">-1.570796327</param>
+              <param name="max">0.0</param>
+            </command_interface>
             <!-- <command_interface name="velocity"/> -->
-            <state_interface name="position"/>
+            <state_interface name="position">
+              <param name="initial_value">0.0</param>
+            </state_interface>
             <state_interface name="velocity"/>
             <state_interface name="effort"/>
           </joint>
-            <!-- Outer Left -->
-          <joint name="hand_outer_l_joint">
-            <param name="mimic">hand_joint</param>
-            <param name="multiplier">-1</param> <!-- flip if needed -->
-            <command_interface name="position"/>
-            <state_interface name="position"/>
-            <state_interface name="velocity"/>
-            <state_interface name="effort"/>
+          <xacro:if value="${$(arg enable_gz)}">
+            <joint name="hand_inner_l_joint">
+              <param name="mimic">hand_joint</param>
+              <param name="multiplier">-1</param>
+              <command_interface name="position"/>
+              <!-- <command_interface name="velocity"/> -->
+              <state_interface name="position"/>
+              <state_interface name="velocity"/>
+              <state_interface name="effort"/>
+            </joint>
+              <!-- Outer Left -->
+            <joint name="hand_outer_l_joint">
+              <param name="mimic">hand_joint</param>
+              <param name="multiplier">-1</param> <!-- flip if needed -->
+              <command_interface name="position"/>
+              <state_interface name="position"/>
+              <state_interface name="velocity"/>
+              <state_interface name="effort"/>
+            </joint>
+            <!-- Outer Right -->
+            <joint name="hand_outer_r_joint">
+              <param name="mimic">hand_joint</param>
+              <param name="multiplier">1</param> <!-- same direction as hand_joint -->
+              <command_interface name="position"/>
+              <state_interface name="position"/>
+              <state_interface name="velocity"/>
+              <state_interface name="effort"/>
           </joint>
-          <!-- Outer Right -->
-          <joint name="hand_outer_r_joint">
-            <param name="mimic">hand_joint</param>
-            <param name="multiplier">1</param> <!-- same direction as hand_joint -->
-            <command_interface name="position"/>
-            <state_interface name="position"/>
-            <state_interface name="velocity"/>
-            <state_interface name="effort"/>
-        </joint>
-                  <!-- Outer Left -->
-          <joint name="hand_finger_l_joint">
-            <param name="mimic">hand_joint</param>
-            <param name="multiplier">-0.5</param> <!-- flip if needed -->
-            <command_interface name="position"/>
-            <state_interface name="position"/>
-            <state_interface name="velocity"/>
-            <state_interface name="effort"/>
+                    <!-- Outer Left -->
+            <joint name="hand_finger_l_joint">
+              <param name="mimic">hand_joint</param>
+              <param name="multiplier">-0.5</param> <!-- flip if needed -->
+              <command_interface name="position"/>
+              <state_interface name="position"/>
+              <state_interface name="velocity"/>
+              <state_interface name="effort"/>
+            </joint>
+            <!-- Outer Right -->
+            <joint name="hand_finger_r_joint">
+              <param name="mimic">hand_joint</param>
+              <param name="multiplier">0.5</param> <!-- same direction as hand_joint -->
+              <command_interface name="position"/>
+              <state_interface name="position"/>
+              <state_interface name="velocity"/>
+              <state_interface name="effort"/>
           </joint>
-          <!-- Outer Right -->
-          <joint name="hand_finger_r_joint">
-            <param name="mimic">hand_joint</param>
-            <param name="multiplier">0.5</param> <!-- same direction as hand_joint -->
-            <command_interface name="position"/>
-            <state_interface name="position"/>
-            <state_interface name="velocity"/>
-            <state_interface name="effort"/>
-        </joint>
+          </xacro:if>
         </xacro:if>
       </xacro:if>
