Commit message: update wheel urdf

File: sobit_pro_description/urdf/wheel/wheel.urdf.xacro (robot description, xacro)
@@ -9,5 +9,5 @@
       <origin xyz="0.15841 0.15841 0.07" rpy="0 0 0" />
       <axis xyz="0 0 1" />
-      <limit lower="-1.5" upper="1.5" effort="10" velocity="10"/>
+      <limit lower="-1.57" upper="1.57" effort="10" velocity="10"/>
       <dynamics damping="0.2" friction="0"/>
     </joint>
@@ -25,5 +25,5 @@
       <origin xyz="-0.15841 0.15841 0.07" rpy="0 0 0" />
       <axis xyz="0 0 1" />
-      <limit lower="-1.5" upper="1.5" effort="10" velocity="10"/>
+      <limit lower="-1.57" upper="1.57" effort="10" velocity="10"/>
       <dynamics damping="0.2" friction="0"/>
     </joint>
@@ -41,5 +41,5 @@
       <origin xyz="0.15841 -0.15841 0.07" rpy="0 0 0" />
       <axis xyz="0 0 1" />
-      <limit lower="-1.5" upper="1.5" effort="10" velocity="10"/>
+      <limit lower="-1.57" upper="1.57" effort="10" velocity="10"/>
       <dynamics damping="0.2" friction="0"/>
     </joint>
@@ -57,5 +57,5 @@
       <origin xyz="-0.15841 -0.15841 0.07" rpy="0 0 0" />
       <axis xyz="0 0 1" />
-      <limit lower="-1.5" upper="1.5" effort="10" velocity="10"/>
+      <limit lower="-1.57" upper="1.57" effort="10" velocity="10"/>
       <dynamics damping="0.2" friction="0"/>
     </joint>

Commit message: fix swivel motion: small radius

File: sobit_pro_description/urdf/wheel/wheel.urdf.xacro (robot description, xacro)
@@ -72,5 +72,5 @@
       <child link="wheel_b_l_link" />
       <origin xyz="0 0 -0.1414" rpy="0 0 0" />
-      <axis xyz="1 1 0" />
+      <axis xyz="-1 -1 0" />
     </joint>
     <link name="wheel_b_l_link">
@@ -86,5 +86,5 @@
       <child link="wheel_b_r_link" />
       <origin xyz="0 0 -0.1414" rpy="0 0 0" />
-      <axis xyz="-1 1 0" />
+      <axis xyz="1 -1 0" />
     </joint>
     <link name="wheel_b_r_link">

Commit message: [UPD] drive wheels are now

File: sobit_pro_description/urdf/wheel/wheel.urdf.xacro (robot description, xacro)
@@ -67,11 +67,10 @@
   </xacro:macro>
   <xacro:macro name="stack_wheel_drive" params="parent prefix number x_loc y_loc z_loc roll=0.0 pitch=0.0 yaw=0.0">
-    <joint name="wheel_${prefix}_drive_joint" type="revolute">
+    <joint name="wheel_${prefix}_drive_joint" type="continuous">
       <origin xyz="${x_loc+0.0019} ${y_loc} ${z_loc}" rpy="${roll} ${pitch} ${yaw}" />
       <parent link="${parent}" />
       <child link="wheel_${prefix}_drive_link" />
       <axis xyz="-1.0 0.0 0.0 " />
-      <limit lower="${-M_PI / 2}" upper="${M_PI/2}" effort="10" velocity="10" />
-      <!-- <dynamics damping="0.2" friction="0" /> -->
+      <limit effort="10" velocity="10" />
     </joint>
     <link name="wheel_${prefix}_drive_link">
