Commit message: urdfとros_controlの連携処理を追加

File: sobit_pro_description/urdf/arm/arm.urdf.xacro (robot description, xacro)
@@ -20,7 +20,7 @@
       <parent link="${prefix}_base_link" />
       <child link="${prefix}1_link" />
-      <origin xyz="0 0 0" rpy="0 0 0" />
-      <axis xyz="1 0 0" />
-      <limit lower="0" upper="3.14" effort="10" velocity="10"/>
+      <origin xyz="0 0 0" rpy="${M_PI / 2} 0 0" />
+      <axis xyz="-1 0 0" />
+      <limit lower="${-M_PI / 2}" upper="${M_PI / 2}" effort="10" velocity="10"/>
       <dynamics damping="0.2" friction="0"/>
     </joint>
@@ -36,7 +36,7 @@
       <parent link="${prefix}1_link" />
       <child link="${prefix}2_link" />
-      <origin xyz="0 0 0.15" rpy="0 0 0" />
-      <axis xyz="1 0 0" />
-      <limit lower="-2.2" upper="0.42" effort="10" velocity="10"/>
+      <origin xyz="0 0 0.15" rpy="-1.137 0 0" />
+      <axis xyz="-1 0 0" />
+      <limit lower="${-M_PI / 2}" upper="${M_PI / 2}" effort="10" velocity="10"/>
       <dynamics damping="0.2" friction="0"/>
     </joint>
@@ -52,7 +52,7 @@
       <parent link="${prefix}2_link" />
       <child link="${prefix}3_link" />
-      <origin xyz="0 -0.13594617 0.06339274" rpy="0 0 0" />
-      <axis xyz="1 0 0" />
-      <limit lower="-2.5" upper="0.36" effort="10" velocity="10"/>
+      <origin xyz="0 -0.13594617 0.06339274" rpy="-1.30 0 0" />
+      <axis xyz="-1 0 0" />
+      <limit lower="${-M_PI / 2}" upper="${M_PI / 2}" effort="10" velocity="10"/>
       <dynamics damping="0.2" friction="0"/>
     </joint>
@@ -68,7 +68,7 @@
       <parent link="${prefix}3_link" />
       <child link="${prefix}4_link" />
-      <origin xyz="0 -0.09641814 -0.11490667" rpy="0 0 0" />
-      <axis xyz="1 0 0" />
-      <limit lower="-0.62" upper="2.44" effort="10" velocity="10"/>
+      <origin xyz="0 -0.09641814 -0.11490667" rpy="0.87 0 0" />
+      <axis xyz="-1 0 0" />
+      <limit lower="${-M_PI / 2}" upper="${M_PI / 2}" effort="10" velocity="10"/>
       <dynamics damping="0.2" friction="0"/>
     </joint>

File: sobit_pro_description/urdf/head/head.urdf.xacro (robot description, xacro)
@@ -4,10 +4,10 @@
   <xacro:include filename="$(find sobit_pro_description)/urdf/head/head.transmission.xacro" />
   <xacro:macro name="head" params="prefix parent">
-    <joint name="${prefix}_pan_joint" type="continuous">
+    <joint name="${prefix}_pan_joint" type="revolute">
       <parent link="${parent}" />
       <child link="${prefix}_pan_link" />
       <origin xyz="0 -0.12985 1.117" rpy="0 0 0" />
       <axis xyz="0 0 1" />
-      <limit lower="-1.5" upper="1.5" effort="10" velocity="10"/>
+      <limit lower="${-M_PI / 2}" upper="${M_PI / 2}" effort="10" velocity="10"/>
       <dynamics damping="0.2" friction="0"/>
     </joint>
@@ -24,6 +24,6 @@
       <child link="${prefix}_tilt_link" />
       <origin xyz="0 0 0.041" rpy="0 0 0" />
-      <axis xyz="1 0 0" />
-      <limit lower="-0.65" upper="1.5" effort="10" velocity="10"/>
+      <axis xyz="-1 0 0" />
+      <limit lower="${-M_PI / 2}" upper="${M_PI / 2}" effort="10" velocity="10"/>
       <dynamics damping="0.2" friction="0"/>
     </joint>

Commit message: fix arm ud

File: sobit_pro_description/urdf/arm/arm.urdf.xacro (robot description, xacro)
@@ -23,7 +23,7 @@
     </joint>
     <link name="${prefix}_fixed_link" />
-    <joint name="${prefix}1_joint" type="revolute">
+    <joint name="${prefix}1_1_joint" type="revolute">
       <parent link="${prefix}_base_link" />
-      <child link="${prefix}1_link" />
+      <child link="${prefix}1_1_link" />
       <origin xyz="0 0 0" rpy="${M_PI / 2} 0 0" />
       <axis xyz="-1 0 0" />
@@ -31,5 +31,5 @@
       <dynamics damping="0.2" friction="0"/>
     </joint>
-    <link name="${prefix}1_link">
+    <link name="${prefix}1_1_link">
       <visual>
         <origin xyz="0 0 0" rpy="1.570796327 0 0" />
@@ -39,6 +39,17 @@
       </visual>
     </link>
+    <joint name="${prefix}1_2_joint" type="revolute">
+      <parent link="${prefix}1_1_link" />
+      <child link="${prefix}1_2_link" />
+      <origin xyz="0 0 0" rpy="${M_PI / 2} 0 0" />
+      <axis xyz="-1 0 0" />
+      <limit lower="${-M_PI / 2}" upper="${M_PI / 2}" effort="10" velocity="10"/>
+      <dynamics damping="0.2" friction="0"/>
+    </joint>
+    <link name="${prefix}1_2_link">
+      <origin xyz="0 0 0" rpy="1.570796327 0 0" />
+    </link>
     <joint name="${prefix}2_joint" type="revolute">
-      <parent link="${prefix}1_link" />
+      <parent link="${prefix}1_1_link" />
       <child link="${prefix}2_link" />
       <origin xyz="0 0 0.15" rpy="-1.137 0 0" />
