Commit message: [UPD] update collision with primitive shapes

File: sobit_pro_description/urdf/arm/arm.urdf.xacro (robot description, xacro)
@@ -17,7 +17,9 @@
       </visual>
       <collision>
-        <origin xyz="0.0 0.0 0.0" rpy="${M_PI/2} 0.0 0.0" />
+        <origin xyz="${0.140/2} 0.0 ${0.043/2}" rpy="0.0 0.0 0.0" />
+        <!-- <origin xyz="0.0 0.0 0.0" rpy="${M_PI/2} 0.0 0.0" /> -->
         <geometry>
-          <mesh filename="package://sobit_pro_description/meshes/arm/arm_base.stl" scale="0.001 0.001 0.001" />
+          <box size="0.140 0.156 0.043" />
+          <!-- <mesh filename="package://sobit_pro_description/meshes/arm/arm_base.stl" scale="0.001 0.001 0.001" /> -->
         </geometry>
       </collision>
@@ -47,7 +49,9 @@
       </visual>
       <collision>
-        <origin xyz="0.0 0.0 0.0" rpy="${M_PI/2} 0.0 ${M_PI/2}" />
+        <origin xyz="${0.1166/2+0.0224} 0.0 0.0" rpy="0.0 0.0 0.0" />
+        <!-- <origin xyz="0.0 0.0 0.0" rpy="${M_PI/2} 0.0 ${M_PI/2}" /> -->
         <geometry>
-          <mesh filename="package://sobit_pro_description/meshes/arm/arm_upper.stl" scale="0.001 0.001 0.001" />
+          <box size="0.1166 0.124 0.043" />
+          <!-- <mesh filename="package://sobit_pro_description/meshes/arm/arm_upper.stl" scale="0.001 0.001 0.001" /> -->
         </geometry>
       </collision>
@@ -60,5 +64,5 @@
       </inertial>
     </link>
-    <joint name="${prefix}_shoulder_2_tilt_joint" type="revolute" >
+    <!-- <joint name="${prefix}_shoulder_2_tilt_joint" type="revolute" >
       <parent link="${prefix}_base_link" />
       <child link="${prefix}_shoulder_2_tilt_link" />
@@ -67,7 +71,7 @@
       <mimic joint="${prefix}_shoulder_1_tilt_joint" multiplier="1" offset="0" />
       <limit lower="${-M_PI / 2}" upper="${M_PI/2}" effort="10" velocity="10" />
-      <!-- <dynamics damping="0.2" friction="0" /> -->
+      <dynamics damping="0.2" friction="0" />
     </joint>
-    <link name="${prefix}_shoulder_2_tilt_link" />
+    <link name="${prefix}_shoulder_2_tilt_link" /> -->
     <joint name="${prefix}_elbow_upper_1_tilt_joint" type="revolute" >
       <parent link="${prefix}_shoulder_1_tilt_link" />
@@ -87,7 +91,9 @@
       </visual>
       <collision>
-        <origin xyz="0.0 0.0 0.0" rpy="${M_PI/2} 0.0 ${M_PI/2}" />
+        <origin xyz="${0.023+0.127/2} 0.0 0.0" rpy="0.0 0.0 0.0" />
+        <!-- <origin xyz="0.0 0.0 0.0" rpy="${M_PI/2} 0.0 ${M_PI/2}" /> -->
         <geometry>
-          <mesh filename="package://sobit_pro_description/meshes/arm/arm_inner.stl" scale="0.001 0.001 0.001" />
+          <box size="0.127 0.048 0.035" />
+          <!-- <mesh filename="package://sobit_pro_description/meshes/arm/arm_inner.stl" scale="0.001 0.001 0.001" /> -->
         </geometry>
       </collision>
@@ -100,5 +106,5 @@
       </inertial>
     </link>
-    <joint name="${prefix}_elbow_upper_2_tilt_joint" type="revolute" >
+    <!-- <joint name="${prefix}_elbow_upper_2_tilt_joint" type="revolute" >
       <parent link="${prefix}_shoulder_1_tilt_link" />
       <child link="${prefix}_elbow_upper_2_tilt_link" />
@@ -107,7 +113,7 @@
       <mimic joint="${prefix}_elbow_upper_1_tilt_joint" multiplier="1" offset="0" />
       <limit lower="${-M_PI / 2}" upper="${M_PI/2}" effort="10" velocity="10" />
-      <!-- <dynamics damping="0.2" friction="0" /> -->
+      <dynamics damping="0.2" friction="0" />
     </joint>
-    <link name="${prefix}_elbow_upper_2_tilt_link" />
+    <link name="${prefix}_elbow_upper_2_tilt_link" /> -->
     <joint name="${prefix}_elbow_lower_tilt_joint" type="revolute" >
       <parent link="${prefix}_elbow_upper_1_tilt_link" />
@@ -127,7 +133,9 @@
       </visual>
       <collision>
-        <origin xyz="0.0 0.0 0.0" rpy="${M_PI/2} 0.0 ${M_PI/2}" />
+        <origin xyz="${0.03+0.120/2} 0.0 -${(0.0215-0.01825)/2}" rpy="0.0 0.0 0.0" />
+        <!-- <origin xyz="0.0 0.0 0.0" rpy="${M_PI/2} 0.0 ${M_PI/2}" /> -->
         <geometry>
-          <mesh filename="package://sobit_pro_description/meshes/arm/arm_elbow_lower_tilt.stl" scale="0.001 0.001 0.001" />
+          <box size="0.120 0.048 0.03975" />
+          <!-- <mesh filename="package://sobit_pro_description/meshes/arm/arm_elbow_lower_tilt.stl" scale="0.001 0.001 0.001" /> -->
         </geometry>
       </collision>
@@ -156,10 +164,10 @@
         <material name="black" />
       </visual>
-      <collision>
+      <!-- <collision>
         <origin xyz="0.0 0.0 0.0" rpy="${M_PI/2} 0.0 ${M_PI/2}" />
         <geometry>
           <mesh filename="package://sobit_pro_description/meshes/arm/arm_elbow_lower_pan.stl" scale="0.001 0.001 0.001" />
         </geometry>
-      </collision>
+      </collision> -->
       <inertial>
         <origin xyz="0.0 0.0 0.0" rpy="${M_PI/2} 0.0 ${M_PI/2}" />

File: sobit_pro_description/urdf/back/back.urdf.xacro (robot description, xacro)
@@ -16,7 +16,9 @@
       </visual>
       <collision>
-        <origin xyz="0.0 0.0 0.0" rpy="0.0 0.0 ${M_PI}" />
+        <origin xyz="0.0 0.0 ${0.517/2}" rpy="0.0 0.0 0.0" />
+        <!-- <origin xyz="0.0 0.0 0.0" rpy="0.0 0.0 ${M_PI}" /> -->
         <geometry>
-          <mesh filename="package://sobit_pro_description/meshes/back/back_base.stl" scale="0.001 0.001 0.001" />
+          <box size="0.02 0.02 0.517"/>
+          <!-- <mesh filename="package://sobit_pro_description/meshes/back/back_base.stl" scale="0.001 0.001 0.001" /> -->
         </geometry>
       </collision>

File: sobit_pro_description/urdf/body/cover.urdf.xacro (robot description, xacro)
@@ -16,7 +16,9 @@
       </visual>
       <collision>
-        <origin xyz="0.0 0.0 0.0" rpy="${M_PI/2} 0.0 ${M_PI/2}" />
+        <origin xyz="-${0.02893+0.3/2} 0.0 ${0.034-0.489/2}" rpy="0.0 0.0 0.0" />
+        <!-- <origin xyz="0.0 0.0 0.0" rpy="${M_PI/2} 0.0 ${M_PI/2}" /> -->
         <geometry>
-          <mesh filename="package://sobit_pro_description/meshes/body/cover.stl" scale="0.001 0.001 0.001" />
+          <box size="${(0.02893+0.3/2)*2} 0.3965 0.489"/>
+          <!-- <mesh filename="package://sobit_pro_description/meshes/body/cover.stl" scale="0.001 0.001 0.001" /> -->
         </geometry>
       </collision>

File: sobit_pro_description/urdf/body/plate.urdf.xacro (robot description, xacro)
@@ -1,5 +1,5 @@
 <?xml version="1.0" encoding="UTF-8" ?>
 <robot name="plate" xmlns:xacro="http://ros.org/wiki/xacro">
-    <xacro:macro name="plate" params="prefix parent">>
+    <xacro:macro name="plate" params="prefix parent">
     <joint name="${prefix}_bottom_joint" type="fixed">
       <origin xyz="0.0 0.0 0.0" rpy="0.0 0.0 0.0" />
@@ -16,7 +16,9 @@
       </visual>
       <collision>
-        <origin xyz="0.0 0.0 0.0" rpy="0.0 0.0 0.0" />
+        <origin xyz="0.0 0.0 -${0.009/2}" rpy="0.0 0.0 0.0" />
+        <!-- <origin xyz="0.0 0.0 0.0" rpy="0.0 0.0 0.0" /> -->
         <geometry>
-          <mesh filename="package://sobit_pro_description/meshes/body/plate_bottom.stl" scale="0.001 0.001 0.001" />
+          <box size="0.3 0.3 0.009" />
+          <!-- <mesh filename="package://sobit_pro_description/meshes/body/plate_bottom.stl" scale="0.001 0.001 0.001" /> -->
         </geometry>
       </collision>
@@ -43,7 +45,9 @@
       </visual>
       <collision>
-        <origin xyz="0.0 0.0 0.0" rpy="0.0 0.0 0.0" />
+        <origin xyz="0.0 0.0 -${0.009/2}" rpy="0.0 0.0 0.0" />
+        <!-- <origin xyz="0.0 0.0 0.0" rpy="0.0 0.0 0.0" /> -->
         <geometry>
-          <mesh filename="package://sobit_pro_description/meshes/body/plate_middle.stl" scale="0.001 0.001 0.001" />
+          <box size="0.3 0.3 0.009" />
+          <!-- <mesh filename="package://sobit_pro_description/meshes/body/plate_middle.stl" scale="0.001 0.001 0.001" /> -->
         </geometry>
       </collision>
@@ -70,7 +74,9 @@
       </visual>
       <collision>
-        <origin xyz="0.0 0.0 0.0" rpy="0.0 0.0 ${M_PI/2}" />
+        <origin xyz="0.0 0.0 -${0.009/2}" rpy="0.0 0.0 0.0" />
+        <!-- <origin xyz="0.0 0.0 0.0" rpy="0.0 0.0 ${M_PI/2}" /> -->
         <geometry>
-          <mesh filename="package://sobit_pro_description/meshes/body/plate_top.stl" scale="0.001 0.001 0.001" />
+          <box size="0.3 0.3 0.009" />
+          <!-- <mesh filename="package://sobit_pro_description/meshes/body/plate_top.stl" scale="0.001 0.001 0.001" /> -->
         </geometry>
       </collision>

File: sobit_pro_description/urdf/hand/hand.urdf.xacro (robot description, xacro)
@@ -17,7 +17,9 @@
       </visual>
       <collision>
-        <origin xyz="0.0 0.0 0.0" rpy="${M_PI/2.0} 0.0 ${M_PI/2.0}" />
-        <geometry>
-          <mesh filename="package://sobit_pro_description/meshes/hand/hand_base.stl" scale="0.001 0.001 0.001" />
+        <origin xyz="${0.0215+(0.08251-0.0215)/2} 0.0 ${(0.0415-0.033)/2}" rpy="0.0 0.0 0.0" />
+        <!-- <origin xyz="0.0 0.0 0.0" rpy="${M_PI/2.0} 0.0 ${M_PI/2.0}" /> -->
+        <geometry>
+          <box size="0.06102 0.102 0.0745" />
+          <!-- <mesh filename="package://sobit_pro_description/meshes/hand/hand_base.stl" scale="0.001 0.001 0.001" /> -->
         </geometry>
       </collision>
@@ -55,7 +57,9 @@
       </visual>
       <collision>
-        <origin xyz="0.0 0.0 0.0" rpy="0.0 0.0 ${M_PI/2.0}" />
-        <geometry>
-          <mesh filename="package://sobit_pro_description/meshes/hand/hand_inner_l.stl" scale="0.001 0.001 0.001" />
+        <origin xyz="${0.05408+(0.06006-0.00707)/2} 0.0 -${0.066/2}" rpy="0.0 0.0 0.0" />
+        <!-- <origin xyz="0.0 0.0 0.0" rpy="0.0 0.0 ${M_PI/2.0}" /> -->
+        <geometry>
+          <box size="${0.06006-0.0071} 0.01 0.066" />
+          <!-- <mesh filename="package://sobit_pro_description/meshes/hand/hand_inner_l.stl" scale="0.001 0.001 0.001" /> -->
         </geometry>
       </collision>
@@ -85,7 +89,9 @@
       </visual>
       <collision>
-        <origin xyz="0.0 0.0 0.0" rpy="0.0 0.0 ${M_PI/2.0}" />
-        <geometry>
-          <mesh filename="package://sobit_pro_description/meshes/hand/hand_inner_r.stl" scale="0.001 0.001 0.001" />
+        <origin xyz="${0.05408+(0.06006-0.00707)/2} 0.0 -${0.066/2}" rpy="0.0 0.0 0.0" />
+        <!-- <origin xyz="0.0 0.0 0.0" rpy="0.0 0.0 ${M_PI/2.0}" /> -->
+        <geometry>
+          <box size="${0.06006-0.0071} 0.01 0.066" />
+          <!-- <mesh filename="package://sobit_pro_description/meshes/hand/hand_inner_r.stl" scale="0.001 0.001 0.001" /> -->
         </geometry>
       </collision>
@@ -99,7 +105,9 @@
     </link>
     <joint name="${prefix_hand}_outer_l_joint" type="revolute">
-      <parent link="${prefix_hand}_base_link" />
+      <parent link="${prefix_hand}_inner_l_link" />
+      <!-- <parent link="${prefix_hand}_base_link" /> -->
       <child link="${prefix_hand}_outer_l_link" />
-      <origin xyz="0.043193 0.04015 0.0282231" rpy="0.0 0.0 0.0" />
+      <origin xyz="-0.01988747 0.025 -0.01022197" rpy="0.0 0.0 0.0" />
+      <!-- <origin xyz="0.043193 0.04015 0.0282231" rpy="0.0 0.0 0.0" /> -->
       <axis xyz="0.0 0.0 -1.0" />
       <mimic joint="${prefix_hand}_joint" multiplier="1.0" offset="0" />
@@ -115,7 +123,9 @@
       </visual>
       <collision>
-        <origin xyz="0.0 0.0 0.0" rpy="0.0 0.0 ${M_PI/2.0}" />
-        <geometry>
-          <mesh filename="package://sobit_pro_description/meshes/hand/hand_outer_l.stl" scale="0.001 0.001 0.001" />
+        <origin xyz="${0.06123+0.04281/2} 0.0 -${0.056/2}" rpy="0.0 0.0 0.0" />
+        <!-- <origin xyz="0.0 0.0 0.0" rpy="0.0 0.0 ${M_PI/2.0}" /> -->
+        <geometry>
+          <box size="0.04281 0.01 0.056" />
+          <!-- <mesh filename="package://sobit_pro_description/meshes/hand/hand_outer_l.stl" scale="0.001 0.001 0.001" /> -->
         </geometry>
       </collision>
@@ -129,7 +139,9 @@
     </link>
     <joint name="${prefix_hand}_outer_r_joint" type="revolute">
-      <parent link="${prefix_hand}_base_link" />
+      <parent link="${prefix_hand}_inner_r_link" />
+      <!-- <parent link="${prefix_hand}_base_link" /> -->
       <child link="${prefix_hand}_outer_r_link" />
-      <origin xyz="0.043193 -0.04015 0.0282231" rpy="0.0 0.0 0.0" />
+      <origin xyz="-0.01988747 -0.025 -0.01022197" rpy="0.0 0.0 0.0" />
+      <!-- <origin xyz="0.043193 -0.04015 0.0282231" rpy="0.0 0.0 0.0" /> -->
       <axis xyz="0.0 0.0 1.0" />
       <mimic joint="${prefix_hand}_joint" multiplier="1.0" offset="0" />
@@ -145,7 +157,9 @@
       </visual>
       <collision>
-        <origin xyz="0.0 0.0 0.0" rpy="0.0 0.0 ${M_PI/2.0}" />
-        <geometry>
-          <mesh filename="package://sobit_pro_description/meshes/hand/hand_outer_r.stl" scale="0.001 0.001 0.001" />
+        <origin xyz="${0.06123+0.04281/2} 0.0 -${0.056/2}" rpy="0.0 0.0 0.0" />
+        <!-- <origin xyz="0.0 0.0 0.0" rpy="0.0 0.0 ${M_PI/2.0}" /> -->
+        <geometry>
+          <box size="0.04281 0.01 0.056" />
+          <!-- <mesh filename="package://sobit_pro_description/meshes/hand/hand_outer_r.stl" scale="0.001 0.001 0.001" /> -->
         </geometry>
       </collision>
@@ -175,7 +189,9 @@
       </visual>
       <collision>
-        <origin xyz="0.0 0.0 0.0" rpy="0.0 0.0 ${M_PI/2.0}" />
-        <geometry>
-          <mesh filename="package://sobit_pro_description/meshes/hand/hand_finger_l.stl" scale="0.001 0.001 0.001" />
+        <origin xyz="${0.03+(0.08+0.00707)/2} -0.025 -${0.018/2}" rpy="0.0 0.0 0.0" />
+        <!-- <origin xyz="0.0 0.0 0.0" rpy="0.0 0.0 ${M_PI/2.0}" /> -->
+        <geometry>
+          <box size="${0.08-0.00707} 0.01137 0.044" />
+          <!-- <mesh filename="package://sobit_pro_description/meshes/hand/hand_finger_l.stl" scale="0.001 0.001 0.001" /> -->
         </geometry>
       </collision>
@@ -205,7 +221,9 @@
       </visual>
       <collision>
-        <origin xyz="0.0 0.0 0.0" rpy="0.0 0.0 ${M_PI/2.0}" />
-        <geometry>
-          <mesh filename="package://sobit_pro_description/meshes/hand/hand_finger_r.stl" scale="0.001 0.001 0.001" />
+        <origin xyz="${0.03+(0.08+0.00707)/2} 0.025 -${0.018/2}" rpy="0.0 0.0 0.0" />
+        <!-- <origin xyz="0.0 0.0 0.0" rpy="0.0 0.0 ${M_PI/2.0}" /> -->
+        <geometry>
+          <box size="${0.08-0.00707} 0.01137 0.044" />
+          <!-- <mesh filename="package://sobit_pro_description/meshes/hand/hand_finger_r.stl" scale="0.001 0.001 0.001" /> -->
         </geometry>
       </collision>

File: sobit_pro_description/urdf/head/head.urdf.xacro (robot description, xacro)
@@ -20,7 +20,9 @@
       </visual>
       <collision>
-        <origin xyz="0.0 0.0 0.0" rpy="${M_PI/2.0} 0.0 ${M_PI/2.0}" />
+        <origin xyz="${0.05125-0.15125/2} 0.0 0.0" rpy="0.0 0.0 0.0" />
+        <!-- <origin xyz="0.0 0.0 0.0" rpy="${M_PI/2.0} 0.0 ${M_PI/2.0}" /> -->
         <geometry>
-          <mesh filename="package://sobit_pro_description/meshes/head/head_camera_base.stl" scale="0.001 0.001 0.001" />
+          <box size="0.15125 0.0285 0.044"/>
+          <!-- <mesh filename="package://sobit_pro_description/meshes/head/head_camera_base.stl" scale="0.001 0.001 0.001" /> -->
         </geometry>
       </collision>
@@ -53,7 +55,9 @@
       </visual>
       <collision>
-        <origin xyz="0.0 0.0 0.0" rpy="0.0 0.0 ${M_PI/2.0}" />
+        <origin xyz="0.0 0.0 ${0.00525+0.03525/2}" rpy="0.0 0.0 0.0" />
+        <!-- <origin xyz="0.0 0.0 0.0" rpy="0.0 0.0 ${M_PI/2.0}" /> -->
         <geometry>
-          <mesh filename="package://sobit_pro_description/meshes/head/head_camera_pan.stl" scale="0.001 0.001 0.001" />
+          <box size="0.0285 0.037 0.03525"/>
+          <!-- <mesh filename="package://sobit_pro_description/meshes/head/head_camera_pan.stl" scale="0.001 0.001 0.001" /> -->
         </geometry>
       </collision>
@@ -86,7 +90,9 @@
       </visual>
       <collision>
-        <origin xyz="0.0 0.0 0.0" rpy="0.0 0.0 ${M_PI/2.0}" />
+        <origin xyz="0.0 0.0 ${0.028+0.0115/2}" rpy="0.0 0.0 0.0" />
+        <!-- <origin xyz="0.0 0.0 0.0" rpy="0.0 0.0 ${M_PI/2.0}" /> -->
         <geometry>
-          <mesh filename="package://sobit_pro_description/meshes/head/head_camera_tilt.stl" scale="0.001 0.001 0.001" />
+          <box size="0.046 0.0466 0.0115"/>
+          <!-- <mesh filename="package://sobit_pro_description/meshes/head/head_camera_tilt.stl" scale="0.001 0.001 0.001" /> -->
         </geometry>
       </collision>

File: sobit_pro_description/urdf/sensor/lidar.urdf.xacro (robot description, xacro)
@@ -16,7 +16,9 @@
       </visual>
       <collision>
-        <origin xyz="0.0 0.0 0.0" rpy="${M_PI/2} 0.0 ${M_PI}" />
+        <origin xyz="${0.092/2} 0.0 -${0.007/2}" rpy="0.0 0.0 0.0" />
+        <!-- <origin xyz="0.0 0.0 0.0" rpy="${M_PI/2} 0.0 ${M_PI}" /> -->
         <geometry>
-          <mesh filename="package://sobit_pro_description/meshes/sensor/lidar_base.stl" scale="0.001 0.001 0.001" />
+          <box size="0.092 0.184 0.007"/>
+          <!-- <mesh filename="package://sobit_pro_description/meshes/sensor/lidar_base.stl" scale="0.001 0.001 0.001" /> -->
         </geometry>
       </collision>

File: sobit_pro_description/urdf/sensor/mic.urdf.xacro (robot description, xacro)
@@ -16,7 +16,9 @@
       </visual>
       <collision>
-        <origin xyz="0.0 0.0 0.0" rpy="${M_PI/2} 0.0 ${M_PI}" />
+        <origin xyz="0.0 ${(0.02-0.1146-0.0146)/2} -${0.02/2}" rpy="0.0 0.0 0.0" />
+        <!-- <origin xyz="0.0 0.0 0.0" rpy="${M_PI/2} 0.0 ${M_PI}" /> -->
         <geometry>
-          <mesh filename="package://sobit_pro_description/meshes/sensor/mic_base.stl" scale="0.001 0.001 0.001" />
+          <box size="0.0292 ${0.1146+0.0146} 0.03"/>
+          <!-- <mesh filename="package://sobit_pro_description/meshes/sensor/mic_base.stl" scale="0.001 0.001 0.001" /> -->
         </geometry>
         <material name="black" />
@@ -44,7 +46,9 @@
       </visual>
       <collision>
-        <origin xyz="0.0 0.0 0.0" rpy="${M_PI/2} 0.0 ${M_PI}" />
+        <origin xyz="${0.0+0.04911} -${0.0112/2} ${0.035+0.0266}" rpy="0.0 ${M_PI/2-25*M_PI/180} 0.0" />
+        <!-- <origin xyz="0.0 0.0 0.0" rpy="${M_PI/2} 0.0 ${M_PI}" /> -->
         <geometry>
-          <mesh filename="package://sobit_pro_description/meshes/sensor/mic.stl" scale="0.001 0.001 0.001" />
+          <cylinder radius="${0.022/2}" length="0.281"/>
+          <!-- <mesh filename="package://sobit_pro_description/meshes/sensor/mic.stl" scale="0.001 0.001 0.001" /> -->
         </geometry>
         <material name="black" />

File: sobit_pro_description/urdf/wheel/wheel.urdf.xacro (robot description, xacro)
@@ -16,7 +16,9 @@
       </visual>
       <collision>
-        <origin xyz="0.0 0.0 0.0" rpy="${M_PI/2.0} 0.0 ${M_PI/2.0}" />
+        <origin xyz="${0.01388-0.05525/2} 0.0 -${0.005+0.034/2+0.02/2}" rpy="${M_PI/2.0} 0.0 ${M_PI/2.0}" />
+        <!-- <origin xyz="0.0 0.0 0.0" rpy="${M_PI/2.0} 0.0 ${M_PI/2.0}" /> -->
         <geometry>
-          <mesh filename="package://sobit_pro_description/meshes/wheel/wheel_base.stl" scale="0.001 0.001 0.001" />
+          <box size="0.0285 0.084 0.05525" />
+          <!-- <mesh filename="package://sobit_pro_description/meshes/wheel/wheel_base.stl" scale="0.001 0.001 0.001" /> -->
         </geometry>
       </collision>
@@ -48,7 +50,9 @@
       </visual>
       <collision>
-        <origin xyz="0.0 0.0 0.0" rpy="${M_PI/2} 0.0 ${M_PI/2}" />
+        <origin xyz="${0.0244+0.0436/2} 0.0 ${0.034/2+0.0149-0.1766/2}" rpy="${M_PI/2} 0.0 ${M_PI/2}" />
+        <!-- <origin xyz="0.0 0.0 0.0" rpy="${M_PI/2} 0.0 ${M_PI/2}" /> -->
         <geometry>
-          <mesh filename="package://sobit_pro_description/meshes/wheel/wheel_steer.stl" scale="0.001 0.001 0.001" />
+          <box size="0.0495 0.1766 0.0436" />
+          <!-- <mesh filename="package://sobit_pro_description/meshes/wheel/wheel_steer.stl" scale="0.001 0.001 0.001" /> -->
         </geometry>
       </collision>
@@ -64,5 +68,5 @@
   <xacro:macro name="stack_wheel_drive" params="parent prefix number x_loc y_loc z_loc roll=0.0 pitch=0.0 yaw=0.0">
     <joint name="wheel_${prefix}_drive_joint" type="revolute">
-      <origin xyz="${x_loc} ${y_loc} ${z_loc}" rpy="${roll} ${pitch} ${yaw}" />
+      <origin xyz="${x_loc+0.0019} ${y_loc} ${z_loc}" rpy="${roll} ${pitch} ${yaw}" />
       <parent link="${parent}" />
       <child link="wheel_${prefix}_drive_link" />
@@ -80,7 +84,9 @@
       </visual>
       <collision>
-        <origin xyz="0.0 0.0 0.0" rpy="${M_PI/2} 0.0 ${M_PI+M_PI/2.0}" />
+        <origin xyz="-${0.0055+0.029/2} 0.0 0.0" rpy="${M_PI/2} 0.0 ${M_PI+M_PI/2.0}" />
+        <!-- <origin xyz="0.0 0.0 0.0" rpy="${M_PI/2} 0.0 ${M_PI+M_PI/2.0}" /> -->
         <geometry>
-          <mesh filename="package://sobit_pro_description/meshes/wheel/wheel_drive.stl" scale="0.001 0.001 0.001" />
+          <cylinder radius="${0.144/2}" length="0.029"/>
+          <!-- <mesh filename="package://sobit_pro_description/meshes/wheel/wheel_drive.stl" scale="0.001 0.001 0.001" /> -->
         </geometry>
       </collision>
@@ -99,12 +105,12 @@
     <xacro:stack_wheel_steer_base parent="${parent}" prefix="b_r" number="3" x_loc= "-${0.210*cos(radians(45.))}" y_loc= "-${0.210*cos(radians(45.))}" z_loc="-0.019" />
     <xacro:stack_wheel_steer_base parent="${parent}" prefix="f_r" number="4" x_loc= "${0.210*cos(radians(45.))}"  y_loc= "-${0.210*cos(radians(45.))}" z_loc="-0.019" />
-    <xacro:stack_wheel_steer parent="wheel_f_l_steer_base_link" prefix="f_l" number="1" x_loc= "0.013875"  y_loc= "0.0"  z_loc="-0.032" />
-    <xacro:stack_wheel_steer parent="wheel_b_l_steer_base_link" prefix="b_l" number="2" x_loc= "0.013875" y_loc= "0.0"  z_loc="-0.032" />
+    <xacro:stack_wheel_steer parent="wheel_f_l_steer_base_link" prefix="f_l" number="1" x_loc= "0.013875" y_loc= "0.0" z_loc="-0.032" />
+    <xacro:stack_wheel_steer parent="wheel_b_l_steer_base_link" prefix="b_l" number="2" x_loc= "0.013875" y_loc= "0.0" z_loc="-0.032" />
     <xacro:stack_wheel_steer parent="wheel_b_r_steer_base_link" prefix="b_r" number="3" x_loc= "0.013875" y_loc= "0.0" z_loc="-0.032" />
-    <xacro:stack_wheel_steer parent="wheel_f_r_steer_base_link" prefix="f_r" number="4" x_loc= "0.013875"  y_loc= "0.0" z_loc="-0.032" />
-    <xacro:stack_wheel_drive parent="wheel_f_l_steer_link" prefix="f_l" number="1" x_loc= "0.02"  y_loc= "0.0"  z_loc="-0.118" />
-    <xacro:stack_wheel_drive parent="wheel_b_l_steer_link" prefix="b_l" number="2" x_loc= "0.02" y_loc= "0.0"  z_loc="-0.118" />
+    <xacro:stack_wheel_steer parent="wheel_f_r_steer_base_link" prefix="f_r" number="4" x_loc= "0.013875" y_loc= "0.0" z_loc="-0.032" />
+    <xacro:stack_wheel_drive parent="wheel_f_l_steer_link" prefix="f_l" number="1" x_loc= "0.02" y_loc= "0.0" z_loc="-0.118" />
+    <xacro:stack_wheel_drive parent="wheel_b_l_steer_link" prefix="b_l" number="2" x_loc= "0.02" y_loc= "0.0" z_loc="-0.118" />
     <xacro:stack_wheel_drive parent="wheel_b_r_steer_link" prefix="b_r" number="3" x_loc= "0.02" y_loc= "0.0" z_loc="-0.118" />
-    <xacro:stack_wheel_drive parent="wheel_f_r_steer_link" prefix="f_r" number="4" x_loc= "0.02"  y_loc= "0.0" z_loc="-0.118" />
+    <xacro:stack_wheel_drive parent="wheel_f_r_steer_link" prefix="f_r" number="4" x_loc= "0.02" y_loc= "0.0" z_loc="-0.118" />
   </xacro:macro>
 </robot>
