Commit message: [FIX] add proper inertia

File: sobit_pro_description/urdf/arm/arm.urdf.xacro (robot description, xacro)
@@ -25,9 +25,12 @@
       </collision>
       <inertial>
-        <origin xyz="0.0 0.0 0.0" rpy="${M_PI/2} 0.0 0.0" />
-        <mass value="0.08" />
-        <inertia ixx="1.0" ixy="0.0" ixz="0.0"
-                 iyy="1.0" iyz="0.0"
-                 izz="1.0" />
+        <origin xyz="${0.140/2} 0.0 ${0.043/2}" rpy="0.0 0.0 ${M_PI/2}" />
+        <mass value="0.08" />
+        <inertia ixx="${1/12*0.08*(0.140**2+0.043**2)}" ixy="0.0" ixz="0.0"
+                 iyy="${1/12*0.08*(0.156**2+0.043**2)}" iyz="0.0"
+                 izz="${1/12*0.08*(0.140**2+0.156**2)}" />
+        <!-- <inertia ixx="1.0" ixy="0.0" ixz="0.0"
+                 iyy="1.0" iyz="0.0"
+                 izz="1.0" /> -->
       </inertial>
     </link>
@@ -57,9 +60,12 @@
       </collision>
       <inertial>
-        <origin xyz="0.0 0.0 0.0" rpy="${M_PI/2} 0.0 ${M_PI/2}" />
-        <mass value="0.08" />
-        <inertia ixx="1.0" ixy="0.0" ixz="0.0"
-                 iyy="1.0" iyz="0.0"
-                 izz="1.0" />
+        <origin xyz="${0.1166/2+0.0224} 0.0 0.0" rpy="0.0 0.0 ${M_PI/2}" />
+        <mass value="0.08" />
+        <inertia ixx="${1/12*0.08*(0.1166**2+0.043**2)}" ixy="0.0" ixz="0.0"
+                 iyy="${1/12*0.08*(0.124**2 +0.043**2)}" iyz="0.0"
+                 izz="${1/12*0.08*(0.1166**2+0.124**2)}" />
+        <!-- <inertia ixx="1.0" ixy="0.0" ixz="0.0"
+                 iyy="1.0" iyz="0.0"
+                 izz="1.0" /> -->
       </inertial>
     </link>
@@ -99,9 +105,12 @@
       </collision>
       <inertial>
-        <origin xyz="0.0 0.0 0.0" rpy="${M_PI/2} 0.0 ${M_PI/2}" />
-        <mass value="0.08" />
-        <inertia ixx="1.0" ixy="0.0" ixz="0.0"
-                 iyy="1.0" iyz="0.0"
-                 izz="1.0" />
+        <origin xyz="${0.023+0.127/2} 0.0 0.0" rpy="0.0 0.0 ${M_PI/2}" />
+        <mass value="0.08" />
+        <inertia ixx="${1/12*0.08*(0.127**2+0.035**2)}" ixy="0.0" ixz="0.0"
+                 iyy="${1/12*0.08*(0.048**2+0.035**2)}" iyz="0.0"
+                 izz="${1/12*0.08*(0.127**2+0.048**2)}" />
+        <!-- <inertia ixx="1.0" ixy="0.0" ixz="0.0"
+                 iyy="1.0" iyz="0.0"
+                 izz="1.0" /> -->
       </inertial>
     </link>
@@ -133,17 +142,20 @@
       </visual>
       <collision>
-        <origin xyz="${0.03+0.120/2} 0.0 -${(0.0215-0.01825)/2}" rpy="0.0 0.0 0.0" />
-        <!-- <origin xyz="0.0 0.0 0.0" rpy="${M_PI/2} 0.0 ${M_PI/2}" /> -->
-        <geometry>
-          <box size="0.120 0.048 0.03975" />
+        <origin xyz="${0.028-0.005/2} 0.0 -${(0.0215-0.01825)/2}" rpy="0.0 0.0 0.0" />
+        <!-- <origin xyz="0.0 0.0 0.0" rpy="${M_PI/2} 0.0 ${M_PI/2}" /> -->
+        <geometry>
+          <box size="0.005 0.041 0.024" />
           <!-- <mesh filename="package://sobit_pro_description/meshes/arm/arm_elbow_lower_tilt.stl" scale="0.001 0.001 0.001" /> -->
         </geometry>
       </collision>
       <inertial>
-        <origin xyz="0.0 0.0 0.0" rpy="${M_PI/2} 0.0 ${M_PI/2}" />
-        <mass value="0.08" />
-        <inertia ixx="1.0" ixy="0.0" ixz="0.0"
-                 iyy="1.0" iyz="0.0"
-                 izz="1.0" />
+        <origin xyz="${0.028-0.005/2} 0.0 -${(0.0215-0.01825)/2}" rpy="0.0 0.0 ${M_PI/2}" />
+        <mass value="0.08" />
+        <inertia ixx="${1/12*0.08*(0.005**2+0.024**2)}" ixy="0.0" ixz="0.0"
+                 iyy="${1/12*0.08*(0.041**2+0.024**2)}" iyz="0.0"
+                 izz="${1/12*0.08*(0.005**2+0.041**2)}" />
+        <!-- <inertia ixx="1.0" ixy="0.0" ixz="0.0"
+                 iyy="1.0" iyz="0.0"
+                 izz="1.0" /> -->
       </inertial>
     </link>
@@ -164,16 +176,22 @@
         <material name="black" />
       </visual>
-      <!-- <collision>
-        <origin xyz="0.0 0.0 0.0" rpy="${M_PI/2} 0.0 ${M_PI/2}" />
-        <geometry>
-          <mesh filename="package://sobit_pro_description/meshes/arm/arm_elbow_lower_pan.stl" scale="0.001 0.001 0.001" />
-        </geometry>
-      </collision> -->
-      <inertial>
-        <origin xyz="0.0 0.0 0.0" rpy="${M_PI/2} 0.0 ${M_PI/2}" />
-        <mass value="0.08" />
-        <inertia ixx="1.0" ixy="0.0" ixz="0.0"
-                 iyy="1.0" iyz="0.0"
-                 izz="1.0" />
+      <collision>
+        <origin xyz="${0.002+0.120/2} 0.0 -${(0.0215-0.01825)/2}" rpy="0.0 0.0 0.0" />
+        <!-- <origin xyz="0.0 0.0 0.0" rpy="${M_PI/2} 0.0 ${M_PI/2}" /> -->
+        <geometry>
+          <box size="0.120 0.048 0.03975" />
+          <!-- <mesh filename="package://sobit_pro_description/meshes/arm/arm_elbow_lower_pan.stl" scale="0.001 0.001 0.001" /> -->
+        </geometry>
+      </collision>
+      <inertial>
+        <origin xyz="${0.002+0.120/2} 0.0 -${(0.0215-0.01825)/2}" rpy="0.0 0.0 ${M_PI/2}" />
+        <mass value="0.08" />
+        <!-- CHECK -->
+        <inertia ixx="${1/12*0.08*(0.120**2+0.03975**2)}" ixy="0.0" ixz="0.0"
+                 iyy="${1/12*0.08*(0.048**2+0.03975**2)}" iyz="0.0"
+                 izz="${1/12*0.08*(0.120**2+0.048**2)}" />
+        <!-- <inertia ixx="0.001" ixy="0.0" ixz="0.0"
+                 iyy="0.001" iyz="0.0"
+                 izz="0.001" /> -->
       </inertial>
     </link>

File: sobit_pro_description/urdf/back/back.urdf.xacro (robot description, xacro)
@@ -24,9 +24,12 @@
       </collision>
       <inertial>
-        <origin xyz="0.0 0.0 0.0" rpy="0.0 0.0 ${M_PI}" />
-        <mass value="1" />
-        <inertia ixx="1.0" ixy="0.0" ixz="0.0"
+        <origin xyz="0.0 0.0 ${0.517/2}" rpy="0.0 0.0 0.0" />
+        <mass value="0.5" />
+        <inertia ixx="${1/12*0.5*(0.02**2+0.517**2)}" ixy="0.0" ixz="0.0"
+                 iyy="${1/12*0.5*(0.02**2+0.517**2)}" iyz="0.0"
+                 izz="${1/12*0.5*(0.02**2+0.02**2)}" />
+        <!-- <inertia ixx="1.0" ixy="0.0" ixz="0.0"
                  iyy="1.0" iyz="0.0"
-                 izz="1.0" />
+                 izz="1.0" /> -->
       </inertial>
     </link>

File: sobit_pro_description/urdf/body/cover.urdf.xacro (robot description, xacro)
@@ -24,7 +24,12 @@
       </collision>
       <inertial>
-        <origin xyz="0.0 0.0 0.0" rpy="${M_PI/2} 0.0 ${M_PI/2}" />
-        <mass value="0.000001" />
-        <inertia ixx="0.0001" ixy="0.0" ixz="0.0" iyy="0.0001" iyz="0.0" izz="0.0001" />
+        <origin xyz="-${0.02893+0.3/2} 0.0 ${0.034-0.489/2}" rpy="0.0 0.0 0.0" />
+        <mass value="0.732" />
+        <inertia ixx="${1/12*0.732*(((0.02893+0.3/2)*2)**2+0.489**2)}"  ixy="0.0" ixz="0.0"
+                 iyy="${1/12*0.732*(0.3965**2+0.489**2)}"               iyz="0.0"
+                 izz="${1/12*0.732*(((0.02893+0.3/2)*2)**2+0.3965**2)}" />
+        <!-- <inertia ixx="0.0001" ixy="0.0" ixz="0.0"
+                 iyy="0.0001" iyz="0.0"
+                 izz="0.0001" /> -->
       </inertial>
     </link>

File: sobit_pro_description/urdf/body/plate.urdf.xacro (robot description, xacro)
@@ -24,9 +24,12 @@
       </collision>
       <inertial>
-        <origin xyz="0.0 0.0 0.0" rpy="0.0 0.0 0.0" />
+        <origin xyz="0.0 0.0 -${0.009/2}" rpy="0.0 0.0 0.0" />
         <mass value="0.08" />
-        <inertia ixx="1.0" ixy="0.0" ixz="0.0"
+        <inertia ixx="${1/12*0.08*(0.3**2+0.009**2)}" ixy="0.0" ixz="0.0"
+                 iyy="${1/12*0.08*(0.3**2+0.009**2)}" iyz="0.0"
+                 izz="${1/12*0.08*(0.3**2+0.3**2)}" />
+        <!-- <inertia ixx="1.0" ixy="0.0" ixz="0.0"
                  iyy="1.0" iyz="0.0"
-                 izz="1.0" />
+                 izz="1.0" /> -->
       </inertial>
     </link>
@@ -53,9 +56,12 @@
       </collision>
       <inertial>
-        <origin xyz="0.0 0.0 0.0" rpy="0.0 0.0 0.0" />
+        <origin xyz="0.0 0.0 -${0.009/2}" rpy="0.0 0.0 0.0" />
         <mass value="0.08" />
-        <inertia ixx="1.0" ixy="0.0" ixz="0.0"
+        <inertia ixx="${1/12*0.08*(0.3**2+0.009**2)}" ixy="0.0" ixz="0.0"
+                 iyy="${1/12*0.08*(0.3**2+0.009**2)}" iyz="0.0"
+                 izz="${1/12*0.08*(0.3**2+0.3**2)}" />
+        <!-- <inertia ixx="1.0" ixy="0.0" ixz="0.0"
                  iyy="1.0" iyz="0.0"
-                 izz="1.0" />
+                 izz="1.0" /> -->
       </inertial>
     </link>
@@ -82,9 +88,12 @@
       </collision>
       <inertial>
-        <origin xyz="0.0 0.0 0.0" rpy="0.0 0.0 ${M_PI/2}" />
+        <origin xyz="0.0 0.0 -${0.009/2}" rpy="0.0 0.0 0.0" />
         <mass value="0.08" />
-        <inertia ixx="1.0" ixy="0.0" ixz="0.0"
+        <inertia ixx="${1/12*0.08*(0.3**2+0.009**2)}" ixy="0.0" ixz="0.0"
+                 iyy="${1/12*0.08*(0.3**2+0.009**2)}" iyz="0.0"
+                 izz="${1/12*0.08*(0.3**2+0.3**2)}" />
+        <!-- <inertia ixx="1.0" ixy="0.0" ixz="0.0"
                  iyy="1.0" iyz="0.0"
-                 izz="1.0" />
+                 izz="1.0" /> -->
       </inertial>
     </link>

File: sobit_pro_description/urdf/hand/hand.urdf.xacro (robot description, xacro)
@@ -25,9 +25,12 @@
       </collision>
       <inertial>
-        <origin xyz="0.0 0.0 0.0" rpy="${M_PI/2.0} 0.0 ${M_PI/2.0}" />
-        <mass value="0.08" />
-        <inertia ixx="1.0" ixy="0.0" ixz="0.0"
-                 iyy="1.0" iyz="0.0"
-                 izz="1.0" />
+        <origin xyz="${0.0215+(0.08251-0.0215)/2} 0.0 ${(0.0415-0.033)/2}" rpy="0.0 0.0 ${M_PI/2}" />
+        <mass value="0.08" />
+        <inertia ixx="${1/12*0.08*(0.06102**2+0.0745**2)}" ixy="0.0" ixz="0.0"
+                 iyy="${1/12*0.08*(0.102**2  +0.0745**2)}" iyz="0.0"
+                 izz="${1/12*0.08*(0.06102**2+0.102**2)}" />
+        <!-- <inertia ixx="1.0" ixy="0.0" ixz="0.0"
+                 iyy="1.0" iyz="0.0"
+                 izz="1.0" /> -->
       </inertial>
     </link>
@@ -65,9 +68,12 @@
       </collision>
       <inertial>
-        <origin xyz="0.0 0.0 0.0" rpy="0.0 0.0 0.0" />
-        <mass value="0.08" />
-        <inertia ixx="1.0" ixy="0.0" ixz="0.0"
-                 iyy="1.0" iyz="0.0"
-                 izz="1.0" />
+        <origin xyz="${0.05408+(0.06006-0.00707)/2} 0.0 -${0.066/2}" rpy="0.0 0.0 ${M_PI/2}" />
+        <mass value="0.08" />
+        <inertia ixx="${1/12*0.08*((0.06006-0.0071)**2+0.066**2)}" ixy="0.0" ixz="0.0"
+                 iyy="${1/12*0.08*(0.01**2+0.066**2)}"             iyz="0.0"
+                 izz="${1/12*0.08*((0.06006-0.0071)**2+0.01**2)}" />
+        <!-- <inertia ixx="1.0" ixy="0.0" ixz="0.0"
+                 iyy="1.0" iyz="0.0"
+                 izz="1.0" /> -->
       </inertial>
     </link>
@@ -97,9 +103,12 @@
       </collision>
       <inertial>
-        <origin xyz="0.0 0.0 0.0" rpy="0.0 0.0 0.0" />
-        <mass value="0.08" />
-        <inertia ixx="1.0" ixy="0.0" ixz="0.0"
-                 iyy="1.0" iyz="0.0"
-                 izz="1.0" />
+        <origin xyz="${0.05408+(0.06006-0.00707)/2} 0.0 -${0.066/2}" rpy="0.0 0.0 ${M_PI/2}" />
+        <mass value="0.08" />
+        <inertia ixx="${1/12*0.08*((0.06006-0.0071)**2+0.066**2)}" ixy="0.0" ixz="0.0"
+                 iyy="${1/12*0.08*(0.01**2+0.066**2)}"             iyz="0.0"
+                 izz="${1/12*0.08*((0.06006-0.0071)**2+0.01**2)}" />
+        <!-- <inertia ixx="1.0" ixy="0.0" ixz="0.0"
+                 iyy="1.0" iyz="0.0"
+                 izz="1.0" /> -->
       </inertial>
     </link>
@@ -131,9 +140,12 @@
       </collision>
       <inertial>
-        <origin xyz="0.0 0.0 0.0" rpy="0.0 0.0 0.0" />
-        <mass value="0.08" />
-        <inertia ixx="1.0" ixy="0.0" ixz="0.0"
-                 iyy="1.0" iyz="0.0"
-                 izz="1.0" />
+        <origin xyz="${0.06123+0.04281/2} 0.0 -${0.056/2}" rpy="0.0 0.0 ${M_PI/2}" />
+        <mass value="0.08" />
+        <inertia ixx="${1/12*0.08*(0.04281**2+0.056**2)}" ixy="0.0" ixz="0.0"
+                 iyy="${1/12*0.08*(0.01**2   +0.056**2)}" iyz="0.0"
+                 izz="${1/12*0.08*(0.04281**2+0.01**2)}" />
+        <!-- <inertia ixx="1.0" ixy="0.0" ixz="0.0"
+                 iyy="1.0" iyz="0.0"
+                 izz="1.0" /> -->
       </inertial>
     </link>
@@ -165,9 +177,12 @@
       </collision>
       <inertial>
-        <origin xyz="0.0 0.0 0.0" rpy="0.0 0.0 0.0" />
-        <mass value="0.08" />
-        <inertia ixx="1.0" ixy="0.0" ixz="0.0"
-                 iyy="1.0" iyz="0.0"
-                 izz="1.0" />
+        <origin xyz="${0.06123+0.04281/2} 0.0 -${0.056/2}" rpy="0.0 0.0 ${M_PI/2}" />
+        <mass value="0.08" />
+        <inertia ixx="${1/12*0.08*(0.04281**2+0.056**2)}" ixy="0.0" ixz="0.0"
+                 iyy="${1/12*0.08*(0.01**2   +0.056**2)}" iyz="0.0"
+                 izz="${1/12*0.08*(0.04281**2+0.01**2)}" />
+        <!-- <inertia ixx="1.0" ixy="0.0" ixz="0.0"
+                 iyy="1.0" iyz="0.0"
+                 izz="1.0" /> -->
       </inertial>
     </link>
@@ -197,9 +212,12 @@
       </collision>
       <inertial>
-        <origin xyz="0.0 0.0 0.0" rpy="0.0 0.0 0.0" />
-        <mass value="0.08" />
-        <inertia ixx="1.0" ixy="0.0" ixz="0.0"
-                 iyy="1.0" iyz="0.0"
-                 izz="1.0" />
+        <origin xyz="${0.007071+(0.012042+0.061128)/2} 0.0 -${0.018/2}" rpy="0.0 0.0 ${M_PI/2}" />
+        <mass value="0.08" />
+        <inertia ixx="${1/12*0.08*((0.012042+0.061128)**2+0.044**2)}" ixy="0.0" ixz="0.0"
+                 iyy="${1/12*0.08*(0.01137**2+0.044**2)}"             iyz="0.0"
+                 izz="${1/12*0.08*((0.012042+0.061128)**2+0.01137**2)}" />
+        <!-- <inertia ixx="1.0" ixy="0.0" ixz="0.0"
+                 iyy="1.0" iyz="0.0"
+                 izz="1.0" /> -->
       </inertial>
     </link>
@@ -229,9 +247,12 @@
       </collision>
       <inertial>
-        <origin xyz="0.0 0.0 0.0" rpy="0.0 0.0 0.0" />
-        <mass value="0.08" />
-        <inertia ixx="1.0" ixy="0.0" ixz="0.0"
-                 iyy="1.0" iyz="0.0"
-                 izz="1.0" />
+        <origin xyz="${0.007071+(0.012042+0.061128)/2} 0.0 -${0.018/2}" rpy="0.0 0.0 ${M_PI/2}" />
+        <mass value="0.08" />
+        <inertia ixx="${1/12*0.08*((0.012042+0.061128)**2+0.044**2)}"   ixy="0.0" ixz="0.0"
+                 iyy="${1/12*0.08*(0.01137**2+0.044**2)}"               iyz="0.0"
+                 izz="${1/12*0.08*((0.012042+0.061128)**2+0.01137**2)}" />
+        <!-- <inertia ixx="1.0" ixy="0.0" ixz="0.0"
+                 iyy="1.0" iyz="0.0"
+                 izz="1.0" /> -->
       </inertial>
     </link>

File: sobit_pro_description/urdf/head/head.urdf.xacro (robot description, xacro)
@@ -28,9 +28,12 @@
       </collision>
       <inertial>
-        <origin xyz="0.0 0.0 0.0" rpy="${M_PI/2.0} 0.0 ${M_PI/2.0}" />
+        <origin xyz="${0.05125-0.15125/2} 0.0 0.0" rpy="0.0 0.0 0.0" />
         <mass value="0.08" />
-        <inertia ixx="1.0" ixy="0.0" ixz="0.0"
+        <inertia ixx="${1/12*0.08*(0.15125**2+0.044**2)}" ixy="0.0" ixz="0.0"
+                 iyy="${1/12*0.08*(0.0285**2 +0.044**2)}" iyz="0.0"
+                 izz="${1/12*0.08*(0.15125**2+0.0285**2)}" />
+        <!-- <inertia ixx="1.0" ixy="0.0" ixz="0.0"
                  iyy="1.0" iyz="0.0"
-                 izz="1.0" />
+                 izz="1.0" /> -->
       </inertial>
     </link>
@@ -63,9 +66,12 @@
       </collision>
       <inertial>
-        <origin xyz="0.0 0.0 0.0" rpy="0.0 0.0 ${M_PI/2.0}" />
+        <origin xyz="0.0 0.0 ${0.00525+0.03525/2}" rpy="0.0 0.0 ${M_PI/2}" />
         <mass value="0.08" />
-        <inertia ixx="1.0" ixy="0.0" ixz="0.0"
+        <inertia ixx="${1/12*0.08*(0.0285**2+0.03525**2)}" ixy="0.0" ixz="0.0"
+                 iyy="${1/12*0.08*(0.037**2 +0.03525**2)}" iyz="0.0"
+                 izz="${1/12*0.08*(0.0285**2+0.037**2)}" />
+        <!-- <inertia ixx="1.0" ixy="0.0" ixz="0.0"
                  iyy="1.0" iyz="0.0"
-                 izz="1.0" />
+                 izz="1.0" /> -->
       </inertial>
     </link>
@@ -98,9 +104,12 @@
       </collision>
       <inertial>
-        <origin xyz="0.0 0.0 0.0" rpy="0.0 0.0 ${M_PI/2.0}" />
+        <origin xyz="0.0 0.0 ${0.028+0.0115/2}" rpy="0.0 0.0 0.0" />
         <mass value="0.08" />
-        <inertia ixx="1.0" ixy="0.0" ixz="0.0"
+        <inertia ixx="${1/12*0.08*(0.046**2 +0.0115**2)}" ixy="0.0" ixz="0.0"
+                 iyy="${1/12*0.08*(0.0466**2+0.0115**2)}" iyz="0.0"
+                 izz="${1/12*0.08*(0.046**2 +0.0466**2)}" />
+        <!-- <inertia ixx="1.0" ixy="0.0" ixz="0.0"
                  iyy="1.0" iyz="0.0"
-                 izz="1.0" />
+                 izz="1.0" /> -->
       </inertial>
     </link>

File: sobit_pro_description/urdf/sensor/lidar.urdf.xacro (robot description, xacro)
@@ -24,9 +24,12 @@
       </collision>
       <inertial>
-        <origin xyz="0.0 0.0 0.0" rpy="${M_PI/2} 0.0 ${M_PI}" />
+        <origin xyz="${0.092/2} 0.0 -${0.007/2}" rpy="0.0 0.0 0.0" />
         <mass value="0.08" />
-        <inertia ixx="1.0" ixy="0.0" ixz="0.0"
+        <inertia ixx="${1/12*0.08*(0.092**2+0.007**2)}" ixy="0.0" ixz="0.0"
+                 iyy="${1/12*0.08*(0.184**2+0.007**2)}" iyz="0.0"
+                 izz="${1/12*0.08*(0.092**2+0.184**2)}" />
+        <!-- <inertia ixx="1.0" ixy="0.0" ixz="0.0"
                  iyy="1.0" iyz="0.0"
-                 izz="1.0" />
+                 izz="1.0" /> -->
       </inertial>
     </link>

File: sobit_pro_description/urdf/sensor/mic.urdf.xacro (robot description, xacro)
@@ -25,9 +25,13 @@
       </collision>
       <inertial>
-        <origin xyz="0.0 0.0 0.0" rpy="${M_PI/2} 0.0 ${M_PI}" />
-        <mass value="1" />
-        <inertia ixx="1.0" ixy="0.0" ixz="0.0"
+        <origin xyz="0.0 ${(0.02-0.1146-0.0146)/2} -${0.02/2}" rpy="0.0 0.0 0.0" />
+        <!-- APPROX -->
+        <mass value="0.15" />
+        <inertia ixx="${1/12*0.15*(0.0292**2+0.03**2)}"            ixy="0.0" ixz="0.0"
+                 iyy="${1/12*0.15*((0.1146+0.0146)**2+0.03**2)}"   iyz="0.0"
+                 izz="${1/12*0.15*(0.0292**2+(0.1146+0.0146)**2)}" />
+        <!-- <inertia ixx="1.0" ixy="0.0" ixz="0.0"
                  iyy="1.0" iyz="0.0"
-                 izz="1.0" />
+                 izz="1.0" /> -->
       </inertial>
     </link>
@@ -55,9 +59,9 @@
       </collision>
       <inertial>
-        <origin xyz="0.0 0.0 0.0" rpy="${M_PI/2} 0.0 ${M_PI}" />
-        <mass value="1" />
-        <inertia ixx="1.0" ixy="0.0" ixz="0.0"
-                 iyy="1.0" iyz="0.0"
-                 izz="1.0" />
+        <origin xyz="${0.0+0.04911} -${0.0112/2} ${0.035+0.0266}" rpy="0.0 ${M_PI/2-25*M_PI/180} 0.0" />
+        <mass value="0.235" />
+        <inertia ixx="${1/2 *0.235*(0.022/2)**2}"              ixy="0.0" ixz="0.0"
+                 iyy="${1/12*0.235*(3*(0.022/2)**2+0.281**2)}" iyz="0.0"
+                 izz="${1/12*0.235*(3*(0.022/2)**2+0.281**2)}" />
       </inertial>
     </link>
