Commit message: [FIX] add proper inertia

File: sobit_pro_description/urdf/wheel/wheel.urdf.xacro (robot description, xacro)
@@ -16,17 +16,21 @@
       </visual>
       <collision>
-        <origin xyz="${0.01388-0.05525/2} 0.0 -${0.005+0.034/2+0.02/2}" rpy="${M_PI/2.0} 0.0 ${M_PI/2.0}" />
+        <origin xyz="${0.01388-0.05525/2} 0.0 -${0.005+0.034/2+0.02/2}" rpy="0.0 0.0 0.0" />
         <!-- <origin xyz="0.0 0.0 0.0" rpy="${M_PI/2.0} 0.0 ${M_PI/2.0}" /> -->
         <geometry>
-          <box size="0.0285 0.084 0.05525" />
+          <box size="0.05525 0.0285 0.084" />
           <!-- <mesh filename="package://sobit_pro_description/meshes/wheel/wheel_base.stl" scale="0.001 0.001 0.001" /> -->
         </geometry>
       </collision>
       <inertial>
-        <origin xyz="0.0 0.0 0.0" rpy="${M_PI/2.0} 0.0 ${M_PI/2.0}" />
+        <origin xyz="${0.01388-0.05525/2} 0.0 -${0.005+0.034/2+0.02/2}" rpy="0.0 0.0 0.0" />
+        <!-- <origin xyz="0.0 0.0 0.0" rpy="${M_PI/2.0} 0.0 ${M_PI/2.0}" /> -->
         <mass value="1" />
-        <inertia ixx="1.0" ixy="0.0" ixz="0.0"
+        <inertia ixx="${1/12*1*(0.05525**2+0.084**2)}" ixy="0.0" ixz="0.0"
+                 iyy="${1/12*1*(0.0285**2 +0.084**2)}" iyz="0.0"
+                 izz="${1/12*1*(0.05525**2+0.0285**2)}" />
+        <!-- <inertia ixx="1.0" ixy="0.0" ixz="0.0"
                  iyy="1.0" iyz="0.0"
-                 izz="1.0" />
+                 izz="1.0" /> -->
       </inertial>
     </link>
@@ -50,17 +54,21 @@
       </visual>
       <collision>
-        <origin xyz="${0.0244+0.0436/2} 0.0 ${0.034/2+0.0149-0.1766/2}" rpy="${M_PI/2} 0.0 ${M_PI/2}" />
+        <origin xyz="${0.0244+0.0436/2} 0.0 ${0.034/2+0.0149-0.1766/2}" rpy="0.0 0.0 0.0" />
         <!-- <origin xyz="0.0 0.0 0.0" rpy="${M_PI/2} 0.0 ${M_PI/2}" /> -->
         <geometry>
-          <box size="0.0495 0.1766 0.0436" />
+          <!-- <box size="0.0495 0.1766 0.0436" /> -->
+          <box size="0.0436 0.0495 0.1766" />
           <!-- <mesh filename="package://sobit_pro_description/meshes/wheel/wheel_steer.stl" scale="0.001 0.001 0.001" /> -->
         </geometry>
       </collision>
       <inertial>
-        <origin xyz="0.0 0.0 0.0" rpy="${M_PI/2} 0.0 ${M_PI/2}" />
+        <origin xyz="${0.0244+0.0436/2} 0.0 ${0.034/2+0.0149-0.1766/2}" rpy="0.0 0.0 0.0" />
         <mass value="1" />
-        <inertia ixx="1.0" ixy="0.0" ixz="0.0"
+        <inertia ixx="${1/12*1*(0.0436**2+0.1766**2)}" ixy="0.0" ixz="0.0"
+                 iyy="${1/12*1*(0.0495**2+0.1766**2)}" iyz="0.0"
+                 izz="${1/12*1*(0.0436**2+0.0495**2)}" />
+        <!-- <inertia ixx="1.0" ixy="0.0" ixz="0.0"
                  iyy="1.0" iyz="0.0"
-                 izz="1.0" />
+                 izz="1.0" /> -->
       </inertial>
     </link>
@@ -91,17 +99,20 @@
       </collision>
       <inertial>
-        <origin xyz="0.0 0.0 0.0" rpy="${M_PI/2} 0.0 ${M_PI+M_PI/2.0}" />
+        <origin xyz="-${0.0055+0.029/2} 0.0 0.0" rpy="0.0 0.0 0.0" />
         <mass value="1" />
-        <inertia ixx="1.0" ixy="0.0" ixz="0.0"
+        <inertia ixx="${1/2 *1*(0.144/2)**2}"              ixy="0.0" ixz="0.0"
+                 iyy="${1/12*1*(3*(0.144/2)**2+0.029**2)}" iyz="0.0"
+                 izz="${1/12*1*(3*(0.144/2)**2+0.029**2)}" />
+        <!-- <inertia ixx="1.0" ixy="0.0" ixz="0.0"
                  iyy="1.0" iyz="0.0"
-                 izz="1.0" />
+                 izz="1.0" /> -->
       </inertial>
     </link>
   </xacro:macro>
   <xacro:macro name="wheel" params="parent prefix">
-    <xacro:stack_wheel_steer_base parent="${parent}" prefix="f_l" number="1" x_loc= "${0.210*cos(radians(45.))}"  y_loc= "${0.210*cos(radians(45.))}"  z_loc="-0.019" />
-    <xacro:stack_wheel_steer_base parent="${parent}" prefix="b_l" number="2" x_loc= "-${0.210*cos(radians(45.))}" y_loc= "${0.210*cos(radians(45.))}"  z_loc="-0.019" />
+    <xacro:stack_wheel_steer_base parent="${parent}" prefix="f_l" number="1" x_loc= " ${0.210*cos(radians(45.))}" y_loc= " ${0.210*cos(radians(45.))}" z_loc="-0.019" />
+    <xacro:stack_wheel_steer_base parent="${parent}" prefix="b_l" number="2" x_loc= "-${0.210*cos(radians(45.))}" y_loc= " ${0.210*cos(radians(45.))}" z_loc="-0.019" />
     <xacro:stack_wheel_steer_base parent="${parent}" prefix="b_r" number="3" x_loc= "-${0.210*cos(radians(45.))}" y_loc= "-${0.210*cos(radians(45.))}" z_loc="-0.019" />
-    <xacro:stack_wheel_steer_base parent="${parent}" prefix="f_r" number="4" x_loc= "${0.210*cos(radians(45.))}"  y_loc= "-${0.210*cos(radians(45.))}" z_loc="-0.019" />
+    <xacro:stack_wheel_steer_base parent="${parent}" prefix="f_r" number="4" x_loc= " ${0.210*cos(radians(45.))}" y_loc= "-${0.210*cos(radians(45.))}" z_loc="-0.019" />
     <xacro:stack_wheel_steer parent="wheel_f_l_steer_base_link" prefix="f_l" number="1" x_loc= "0.013875" y_loc= "0.0" z_loc="-0.032" />
     <xacro:stack_wheel_steer parent="wheel_b_l_steer_base_link" prefix="b_l" number="2" x_loc= "0.013875" y_loc= "0.0" z_loc="-0.032" />

Commit message: [UNDO] keep the virtual links

File: sobit_pro_description/urdf/arm/arm.urdf.xacro (robot description, xacro)
@@ -70,5 +70,5 @@
       </inertial>
     </link>
-    <!-- <joint name="${prefix}_shoulder_2_tilt_joint" type="revolute" >
+    <joint name="${prefix}_shoulder_2_tilt_joint" type="revolute" >
       <parent link="${prefix}_base_link" />
       <child link="${prefix}_shoulder_2_tilt_link" />
@@ -79,5 +79,5 @@
       <dynamics damping="0.2" friction="0" />
     </joint>
-    <link name="${prefix}_shoulder_2_tilt_link" /> -->
+    <link name="${prefix}_shoulder_2_tilt_link" />
     <joint name="${prefix}_elbow_upper_1_tilt_joint" type="revolute" >
       <parent link="${prefix}_shoulder_1_tilt_link" />
@@ -115,5 +115,5 @@
       </inertial>
     </link>
-    <!-- <joint name="${prefix}_elbow_upper_2_tilt_joint" type="revolute" >
+    <joint name="${prefix}_elbow_upper_2_tilt_joint" type="revolute" >
       <parent link="${prefix}_shoulder_1_tilt_link" />
       <child link="${prefix}_elbow_upper_2_tilt_link" />
@@ -124,5 +124,5 @@
       <dynamics damping="0.2" friction="0" />
     </joint>
-    <link name="${prefix}_elbow_upper_2_tilt_link" /> -->
+    <link name="${prefix}_elbow_upper_2_tilt_link" />
     <joint name="${prefix}_elbow_lower_tilt_joint" type="revolute" >
       <parent link="${prefix}_elbow_upper_1_tilt_link" />

File: sobit_pro_description/urdf/hand/hand.urdf.xacro (robot description, xacro)
@@ -192,5 +192,5 @@
       <origin xyz="0.114316 0.0 -0.027729" rpy="0.0 0.0 0.0" />
       <axis xyz="0.0 0.0 1.0" />
-      <mimic joint="${prefix_hand}_inner_l_joint" multiplier="-1.0" offset="0" />
+      <mimic joint="${prefix_hand}_joint" multiplier="1.0" offset="0" />
       <limit lower="${-M_PI/2.0}" upper="0" effort="1" velocity="1" />
     </joint>
@@ -227,5 +227,5 @@
       <origin xyz="0.114316 0.0 -0.027729" rpy="0.0 0.0 0.0" />
       <axis xyz="0.0 0.0 1.0" />
-      <mimic joint="${prefix_hand}_inner_r_joint" multiplier="-1.0" offset="0" />
+      <mimic joint="${prefix_hand}_joint" multiplier="-1.0" offset="0" />
       <limit lower="${-M_PI/2.0}" upper="0" effort="1" velocity="1" />
     </joint>

Commit message: [FIX] rotation direction was inversed: arm_elbow_lower_pan_joint

File: sobit_pro_description/urdf/arm/arm.urdf.xacro (robot description, xacro)
@@ -164,5 +164,5 @@
       <child link="${prefix}_elbow_lower_pan_link" />
       <origin xyz="0.028 0.0 0.0" rpy="0.0 0.0 0.0" />
-      <axis xyz="-1.0 0.0 0.0 " />
+      <axis xyz="1.0 0.0 0.0 " />
       <limit lower="${-M_PI / 2}" upper="${M_PI/2}" effort="10" velocity="10" />
       <!-- <dynamics damping="0.2" friction="0" /> -->
