Commit message: add arm2_1_joint and arm2_2_joint

File: sobit_pro_description/urdf/arm/arm.transmission.xacro (robot description, xacro)
@@ -4,5 +4,6 @@
     <position_joint_transmission joint="${prefix}1_1_joint" reduction="1" />
     <position_joint_transmission joint="${prefix}1_2_joint" reduction="1" />
-    <position_joint_transmission joint="${prefix}2_joint" reduction="1" />
+    <position_joint_transmission joint="${prefix}2_1_joint" reduction="1" />
+    <position_joint_transmission joint="${prefix}2_2_joint" reduction="1" />
     <position_joint_transmission joint="${prefix}3_joint" reduction="1" />
     <position_joint_transmission joint="${prefix}4_joint" reduction="1" />

File: sobit_pro_description/urdf/arm/arm.urdf.xacro (robot description, xacro)
@@ -40,5 +40,5 @@
     </link>
     <joint name="${prefix}1_2_joint" type="revolute">
-      <parent link="${prefix}1_1_link" />
+      <parent link="${prefix}_base_link" />
       <child link="${prefix}1_2_link" />
       <origin xyz="0 0 0" rpy="${M_PI / 2} 0 0" />
@@ -50,7 +50,7 @@
       <origin xyz="0 0 0" rpy="1.570796327 0 0" />
     </link>
-    <joint name="${prefix}2_joint" type="revolute">
+    <joint name="${prefix}2_1_joint" type="revolute">
       <parent link="${prefix}1_1_link" />
-      <child link="${prefix}2_link" />
+      <child link="${prefix}2_1_link" />
       <origin xyz="0 0 0.15" rpy="-1.137 0 0" />
       <axis xyz="-1 0 0" />
@@ -58,5 +58,5 @@
       <dynamics damping="0.2" friction="0"/>
     </joint>
-    <link name="${prefix}2_link">
+    <link name="${prefix}2_1_link">
       <visual>
         <origin xyz="0 0 -0.15" rpy="1.570796327 0 0" />
@@ -66,6 +66,17 @@
       </visual>
     </link>
+    <joint name="${prefix}2_2_joint" type="revolute">
+      <parent link="${prefix}1_1_link" />
+      <child link="${prefix}2_2_link" />
+      <origin xyz="0 0 0.15" rpy="-1.137 0 0" />
+      <axis xyz="-1 0 0" />
+      <limit lower="${-M_PI / 2}" upper="${M_PI / 2}" effort="10" velocity="10"/>
+      <dynamics damping="0.2" friction="0"/>
+    </joint>
+    <link name="${prefix}2_2_link">
+      <origin xyz="0 0 -0.15" rpy="1.570796327 0 0" />
+    </link>
     <joint name="${prefix}3_joint" type="revolute">
-      <parent link="${prefix}2_link" />
+      <parent link="${prefix}2_1_link" />
       <child link="${prefix}3_link" />
       <origin xyz="0 -0.13594617 0.06339274" rpy="-1.30 0 0" />

Commit message: update urdf transmission and style

File: sobit_pro_description/urdf/arm/arm.transmission.xacro (robot description, xacro)
@@ -2,10 +2,10 @@
 <robot xmlns:xacro="http://ros.org/wiki/xacro">
   <xacro:macro name="arm_transmission" params="prefix">
-    <position_joint_transmission joint="${prefix}1_1_joint" reduction="1" />
-    <position_joint_transmission joint="${prefix}1_2_joint" reduction="1" />
-    <position_joint_transmission joint="${prefix}2_1_joint" reduction="1" />
-    <position_joint_transmission joint="${prefix}2_2_joint" reduction="1" />
-    <position_joint_transmission joint="${prefix}3_joint" reduction="1" />
-    <position_joint_transmission joint="${prefix}4_joint" reduction="1" />
+    <position_joint_transmission joint="${prefix}_shoulder_1_tilt_joint" reduction="1" />
+    <position_joint_transmission joint="${prefix}_shoulder_2_tilt_joint" reduction="1" />
+    <position_joint_transmission joint="${prefix}_elbow_upper_1_tilt_joint" reduction="1" />
+    <position_joint_transmission joint="${prefix}_elbow_upper_2_tilt_joint" reduction="1" />
+    <position_joint_transmission joint="${prefix}_elbow_lower_tilt_link" reduction="1" />
+    <position_joint_transmission joint="${prefix}_wrist_tilt_joint" reduction="1" />
   </xacro:macro>
 </robot>

File: sobit_pro_description/urdf/arm/arm.urdf.xacro (robot description, xacro)
@@ -1,5 +1,5 @@
 <?xml version="1.0" encoding="UTF-8" ?>
 <robot name="arm" xmlns:xacro="http://ros.org/wiki/xacro" >
-  <!-- <xacro:include filename="$(find sobit_pro_description)/urdf/arm/arm.transmission.xacro" /> -->
+  <xacro:include filename="$(find sobit_pro_description)/urdf/arm/arm.transmission.xacro" />
   <xacro:macro name="arm" params="prefix parent" >
     <joint name="${prefix}_base_joint" type="fixed" >
@@ -149,5 +149,5 @@
     </joint>
     <link name="${prefix}_wrist_tilt_link" />
-    <!-- <xacro:arm_transmission prefix="${prefix}" /> -->
+    <xacro:arm_transmission prefix="${prefix}" />
   </xacro:macro>
 </robot>

File: sobit_pro_description/urdf/hand/hand.urdf.xacro (robot description, xacro)
@@ -1,7 +1,6 @@
 <?xml version="1.0" encoding="UTF-8" ?>
 <robot name="hand" xmlns:xacro="http://ros.org/wiki/xacro">
-  <!-- <xacro:include filename="$(find sobit_pro_description)/urdf/hand/hand.transmission.xacro" /> -->
+  <xacro:include filename="$(find sobit_pro_description)/urdf/hand/hand.transmission.xacro" />
   <xacro:macro name="hand" params="prefix_hand prefix_finger parent">
-    <!-- <xacro:hand_transmission prefix_hand="${prefix_hand}" prefix_finger="${prefix_finger}" /> -->
     <joint name="${prefix_hand}_base_joint" type="fixed">
       <parent link="${parent}" />
@@ -219,4 +218,5 @@
       </inertial>
     </link>
+    <xacro:hand_transmission prefix_hand="${prefix_hand}" prefix_finger="${prefix_finger}" />
   </xacro:macro>
 </robot>

File: sobit_pro_description/urdf/head/head.transmission.xacro (robot description, xacro)
@@ -2,6 +2,6 @@
 <robot xmlns:xacro="http://ros.org/wiki/xacro">
   <xacro:macro name="head_transmission" params="prefix">
-    <position_joint_transmission joint="${prefix}_pan_joint" reduction="1" />
-    <position_joint_transmission joint="${prefix}_tilt_joint" reduction="1" />
+    <position_joint_transmission joint="${prefix}_camera_pan_joint" reduction="1" />
+    <position_joint_transmission joint="${prefix}_camera_tilt_joint" reduction="1" />
   </xacro:macro>
 </robot>

File: sobit_pro_description/urdf/head/head.urdf.xacro (robot description, xacro)
@@ -1,5 +1,5 @@
 <?xml version="1.0" encoding="UTF-8" ?>
 <robot name="head" xmlns:xacro="http://ros.org/wiki/xacro">
-  <!-- <xacro:include filename="$(find sobit_pro_description)/urdf/head/head.transmission.xacro" /> -->
+  <xacro:include filename="$(find sobit_pro_description)/urdf/head/head.transmission.xacro" />
   <xacro:macro name="head" params="prefix parent">
     <joint name="${prefix}_camera_base_joint" type="fixed">
@@ -88,5 +88,5 @@
       </inertial>
     </link>
-    <!-- <xacro:head_transmission prefix="${prefix}" /> -->
+    <xacro:head_transmission prefix="${prefix}" />
   </xacro:macro>
 </robot>

File: sobit_pro_description/urdf/materials.urdf.xacro (robot description, xacro)
@@ -25,9 +25,3 @@
     <color rgba="0.175 0.175 0.175 1.0" />
   </material>
-  <!-- <material name="aluminum">
-    <color rgba="0.5 0.5 0.5 1"/>
-  </material> -->
-  <!-- <material name="plastic">
-    <color rgba="0.1 0.1 0.1 1"/>
-  </material> -->
 </robot>

File: sobit_pro_description/urdf/sensor/matrix.urdf.xacro (robot description, xacro)
@@ -1,6 +1,5 @@
 <?xml version="1.0" encoding="UTF-8" ?>
 <!-- Reference: https://matrix-io.github.io/matrix-documentation/matrix-creator/resources/microphone/ -->
-<robot name="matrix"
-  xmlns:xacro="http://ros.org/wiki/xacro">
+<robot name="matrix" xmlns:xacro="http://ros.org/wiki/xacro">
   <xacro:macro name="matrix" params="prefix parent">
     <joint name="${prefix}_board_joint" type="fixed">

File: sobit_pro_description/urdf/sensor/realsense_l515.urdf.xacro (robot description, xacro)
@@ -1,9 +1,3 @@
 <?xml version="1.0"?>
-<!--
-License: Apache 2.0. See LICENSE file in root directory.
-Copyright(c) 2017 Intel Corporation. All Rights Reserved
-This is the URDF model for the Intel RealSense L515 camera, in its
-aluminum peripherial evaluation case.
--->
 <robot name="realsense_l515" xmlns:xacro="http://ros.org/wiki/xacro">
   <xacro:macro name="realsense_l515" params="prefix parent">

Commit message: update urdf for 5dof

File: sobit_pro_description/urdf/arm/arm.transmission.xacro (robot description, xacro)
@@ -7,4 +7,5 @@
     <position_joint_transmission joint="${prefix}_elbow_upper_2_tilt_joint" reduction="1" />
     <position_joint_transmission joint="${prefix}_elbow_lower_tilt_link"    reduction="1" />
+    <position_joint_transmission joint="${prefix}_elbow_lower_pan_link"    reduction="1" />
     <position_joint_transmission joint="${prefix}_wrist_tilt_joint"         reduction="1" />
   </xacro:macro>

File: sobit_pro_description/urdf/arm/arm.urdf.xacro (robot description, xacro)
@@ -122,5 +122,5 @@
         <origin xyz="0.0 0.0 0.0" rpy="${M_PI/2} 0.0 ${M_PI/2}" />
         <geometry>
-          <mesh filename="package://sobit_pro_description/meshes/arm/arm_lower.stl" scale="0.001 0.001 0.001" />
+          <mesh filename="package://sobit_pro_description/meshes/arm/arm_elbow_lower_tilt.stl" scale="0.001 0.001 0.001" />
         </geometry>
         <material name="black" />
@@ -129,5 +129,35 @@
         <origin xyz="0.0 0.0 0.0" rpy="${M_PI/2} 0.0 ${M_PI/2}" />
         <geometry>
-          <mesh filename="package://sobit_pro_description/meshes/arm/arm_lower.stl" scale="0.001 0.001 0.001" />
+          <mesh filename="package://sobit_pro_description/meshes/arm/arm_elbow_lower_tilt.stl" scale="0.001 0.001 0.001" />
+        </geometry>
+      </collision>
+      <inertial>
+        <origin xyz="0.0 0.0 0.0" rpy="${M_PI/2} 0.0 ${M_PI/2}" />
+        <mass value="0.08" />
+        <inertia ixx="1.0" ixy="0.0" ixz="0.0"
+                 iyy="1.0" iyz="0.0"
+                 izz="1.0" />
+      </inertial>
+    </link>
+    <joint name="${prefix}_elbow_lower_pan_joint" type="revolute" >
+      <parent link="${prefix}_elbow_lower_tilt_link" />
+      <child link="${prefix}_elbow_lower_pan_link" />
+      <origin xyz="0.028 0.0 0.0" rpy="0.0 0.0 0.0" />
+      <axis xyz="-1.0 0.0 0.0 " />
+      <limit lower="${-M_PI / 2}" upper="${M_PI/2}" effort="10" velocity="10" />
+      <!-- <dynamics damping="0.2" friction="0" /> -->
+    </joint>
+    <link name="${prefix}_elbow_lower_pan_link" >
+      <visual>
+        <origin xyz="0.0 0.0 0.0" rpy="${M_PI/2} 0.0 ${M_PI/2}" />
+        <geometry>
+          <mesh filename="package://sobit_pro_description/meshes/arm/arm_elbow_lower_pan.stl" scale="0.001 0.001 0.001" />
+        </geometry>
+        <material name="black" />
+      </visual>
+      <collision>
+        <origin xyz="0.0 0.0 0.0" rpy="${M_PI/2} 0.0 ${M_PI/2}" />
+        <geometry>
+          <mesh filename="package://sobit_pro_description/meshes/arm/arm_elbow_lower_pan.stl" scale="0.001 0.001 0.001" />
         </geometry>
       </collision>
@@ -141,7 +171,7 @@
     </link>
     <joint name="${prefix}_wrist_tilt_joint" type="revolute" >
-      <parent link="${prefix}_elbow_lower_tilt_link" />
+      <parent link="${prefix}_elbow_lower_pan_link" />
       <child link="${prefix}_wrist_tilt_link" />
-      <origin xyz="0.1500 0.0 0.0" rpy="0.0 0.0 0.0" />
+      <origin xyz="0.122009 0.0 0.0" rpy="0.0 0.0 0.0" />
       <axis xyz="0.0 -1.0 0.0" />
       <limit lower="${-M_PI / 2}" upper="${M_PI/2}" effort="10" velocity="10" />

Commit message: [FIX] controllers, transmissions, values, gazebo

File: sobit_pro_description/urdf/arm/arm.transmission.xacro (robot description, xacro)
@@ -3,11 +3,11 @@
        xmlns:xacro="http://ros.org/wiki/xacro">
   <xacro:macro name="arm_transmission" params="prefix">
-    <xacro:position_joint_transmission joint="${prefix}_shoulder_1_tilt_joint"    reduction="1" />
-    <xacro:position_joint_transmission joint="${prefix}_shoulder_2_tilt_joint"    reduction="1" />
-    <xacro:position_joint_transmission joint="${prefix}_elbow_upper_1_tilt_joint" reduction="1" />
-    <xacro:position_joint_transmission joint="${prefix}_elbow_upper_2_tilt_joint" reduction="1" />
-    <xacro:position_joint_transmission joint="${prefix}_elbow_lower_tilt_joint"   reduction="1" />
-    <xacro:position_joint_transmission joint="${prefix}_elbow_lower_pan_joint"    reduction="1" />
-    <xacro:position_joint_transmission joint="${prefix}_wrist_tilt_joint"         reduction="1" />
+    <xacro:SimpleTransmissionPosition joint="${prefix}_shoulder_1_tilt_joint"    reduction="1" />
+    <xacro:SimpleTransmissionPosition joint="${prefix}_shoulder_2_tilt_joint"    reduction="1" />
+    <xacro:SimpleTransmissionPosition joint="${prefix}_elbow_upper_1_tilt_joint" reduction="1" />
+    <xacro:SimpleTransmissionPosition joint="${prefix}_elbow_upper_2_tilt_joint" reduction="1" />
+    <xacro:SimpleTransmissionPosition joint="${prefix}_elbow_lower_tilt_joint"   reduction="1" />
+    <xacro:SimpleTransmissionPosition joint="${prefix}_elbow_lower_pan_joint"    reduction="1" />
+    <xacro:SimpleTransmissionPosition joint="${prefix}_wrist_tilt_joint"         reduction="1" />
   </xacro:macro>
 </robot>

File: sobit_pro_description/urdf/arm/arm.urdf.xacro (robot description, xacro)
@@ -66,9 +66,17 @@
       <origin xyz="0.1560 0.0 0.0215" rpy="0.0 0.0 ${M_PI}" />
       <axis xyz="0.0 1.0 0.0 " />
-      <mimic joint="${prefix}_shoulder_1_tilt_joint" multiplier="1" offset="0" />
+      <!-- <mimic joint="${prefix}_shoulder_1_tilt_joint" multiplier="1" offset="0" /> -->
       <limit lower="${-M_PI/2}" upper="${M_PI/2}" effort="${10.6*2}" velocity="11.031179004" />
       <dynamics damping="0.2" friction="0" />
     </joint>
-    <link name="${prefix}_shoulder_2_tilt_link" />
+    <link name="${prefix}_shoulder_2_tilt_link" >
+      <inertial>
+        <origin xyz="${0.1166/2+0.0224} 0.0 0.0" rpy="0.0 0.0 ${M_PI/2}" />
+        <mass value="0.08" />
+        <inertia ixx="${1/12*0.08*(0.1166**2+0.043**2)}" ixy="0.0" ixz="0.0"
+                 iyy="${1/12*0.08*(0.124**2 +0.043**2)}" iyz="0.0"
+                 izz="${1/12*0.08*(0.1166**2+0.124**2)}" />
+      </inertial>
+    </link>
     <joint name="${prefix}_elbow_upper_1_tilt_joint" type="revolute" >
       <parent link="${prefix}_shoulder_1_tilt_link" />
@@ -106,9 +114,17 @@
       <origin xyz="0.1500 0.0 0.0" rpy="0.0 0.0 ${M_PI}" />
       <axis xyz="0.0 1.0 0.0 " />
-      <mimic joint="${prefix}_elbow_upper_1_tilt_joint" multiplier="1" offset="0" />
+      <!-- <mimic joint="${prefix}_elbow_upper_1_tilt_joint" multiplier="1" offset="0" /> -->
       <limit lower="${-M_PI/2}" upper="${M_PI/2}" effort="${4.1*2}" velocity="9.59233" />
       <dynamics damping="0.2" friction="0" />
     </joint>
-    <link name="${prefix}_elbow_upper_2_tilt_link" />
+    <link name="${prefix}_elbow_upper_2_tilt_link" >
+      <inertial>
+        <origin xyz="${0.023+0.127/2} 0.0 0.0" rpy="0.0 0.0 ${M_PI/2}" />
+        <mass value="0.08" />
+        <inertia ixx="${1/12*0.08*(0.127**2+0.035**2)}" ixy="0.0" ixz="0.0"
+                 iyy="${1/12*0.08*(0.048**2+0.035**2)}" iyz="0.0"
+                 izz="${1/12*0.08*(0.127**2+0.048**2)}" />
+      </inertial>
+    </link>
     <joint name="${prefix}_elbow_lower_tilt_joint" type="revolute" >
       <parent link="${prefix}_elbow_upper_1_tilt_link" />

File: sobit_pro_description/urdf/hand/hand.transmission.xacro (robot description, xacro)
@@ -3,11 +3,11 @@
        xmlns:xacro="http://ros.org/wiki/xacro">
   <xacro:macro name="hand_transmission" params="prefix_hand prefix_finger">
-    <xacro:position_joint_transmission joint="${prefix_hand}_joint"         reduction="1" />
-    <!-- <xacro:position_joint_transmission joint="${prefix_hand}_inner_l_joint" reduction="1" /> -->
-    <!-- <xacro:position_joint_transmission joint="${prefix_hand}_inner_r_joint" reduction="1" /> -->
-    <!-- <xacro:position_joint_transmission joint="${prefix_hand}_outer_l_joint" reduction="1" /> -->
-    <!-- <xacro:position_joint_transmission joint="${prefix_hand}_outer_r_joint" reduction="1" /> -->
-    <!-- <xacro:position_joint_transmission joint="${prefix_hand}_${prefix_finger}_l_joint" reduction="1" /> -->
-    <!-- <xacro:position_joint_transmission joint="${prefix_hand}_${prefix_finger}_r_joint" reduction="1" /> -->
+    <xacro:SimpleTransmissionPosition joint="${prefix_hand}_joint"         reduction="1" />
+    <!-- <xacro:SimpleTransmissionPosition joint="${prefix_hand}_inner_l_joint" reduction="1" /> -->
+    <!-- <xacro:SimpleTransmissionPosition joint="${prefix_hand}_inner_r_joint" reduction="1" /> -->
+    <!-- <xacro:SimpleTransmissionPosition joint="${prefix_hand}_outer_l_joint" reduction="1" /> -->
+    <!-- <xacro:SimpleTransmissionPosition joint="${prefix_hand}_outer_r_joint" reduction="1" /> -->
+    <!-- <xacro:SimpleTransmissionPosition joint="${prefix_hand}_${prefix_finger}_l_joint" reduction="1" /> -->
+    <!-- <xacro:SimpleTransmissionPosition joint="${prefix_hand}_${prefix_finger}_r_joint" reduction="1" /> -->
   </xacro:macro>
 </robot>

File: sobit_pro_description/urdf/head/head.transmission.xacro (robot description, xacro)
@@ -3,6 +3,6 @@
        xmlns:xacro="http://ros.org/wiki/xacro">
   <xacro:macro name="head_transmission" params="prefix">
-    <xacro:position_joint_transmission joint="${prefix}_pan_joint"  reduction="1" />
-    <xacro:position_joint_transmission joint="${prefix}_tilt_joint" reduction="1" />
+    <xacro:SimpleTransmissionPosition joint="${prefix}_pan_joint"  reduction="1" />
+    <xacro:SimpleTransmissionPosition joint="${prefix}_tilt_joint" reduction="1" />
   </xacro:macro>
 </robot>

File: sobit_pro_description/urdf/transmission.urdf.xacro (robot description, xacro)
@@ -1,6 +1,6 @@
 <?xml version="1.0" encoding="UTF-8" ?>
-<!-- SOBIT MINI (transmission) -->
-<robot name="sobit_mini_transmission" xmlns:xacro="http://ros.org/wiki/xacro">
-  <!-- Transmission macro: Position -->
+<!-- SOBIT PRO (transmission) -->
+<robot name="sobit_pro_transmission" xmlns:xacro="http://ros.org/wiki/xacro">
+  <!-- Transmission macro - Position -->
   <xacro:macro name="SimpleTransmissionPosition" params="joint reduction">
     <transmission name="${joint}_transmission">
@@ -14,5 +14,5 @@
     </transmission>
   </xacro:macro>
-  <!-- Transmission macro: Effort -->
+  <!-- Transmission macro - Effort -->
   <xacro:macro name="SimpleTransmissionEffort" params="joint reduction">
     <transmission name="${joint}_transmission">
@@ -26,5 +26,5 @@
     </transmission>
   </xacro:macro>
-  <!-- Transmission macro: Velocity -->
+  <!-- Transmission macro - Velocity -->
   <xacro:macro name="SimpleTransmissionVelocity" params="joint reduction">
     <transmission name="${joint}_transmission">

File: sobit_pro_description/urdf/wheel/wheel.transmission.xacro (robot description, xacro)
@@ -3,12 +3,12 @@
        xmlns:xacro="http://ros.org/wiki/xacro">
   <xacro:macro name="wheel_transmission" params="prefix">
-    <xacro:position_joint_transmission joint="${prefix}_f_l_steer_joint" reduction="1" />
-    <xacro:position_joint_transmission joint="${prefix}_f_r_steer_joint" reduction="1" />
-    <xacro:position_joint_transmission joint="${prefix}_b_l_steer_joint" reduction="1" />
-    <xacro:position_joint_transmission joint="${prefix}_b_r_steer_joint" reduction="1" />
-    <xacro:velocity_joint_transmission joint="${prefix}_f_l_drive_joint" reduction="1" />
-    <xacro:velocity_joint_transmission joint="${prefix}_f_r_drive_joint" reduction="1" />
-    <xacro:velocity_joint_transmission joint="${prefix}_b_l_drive_joint" reduction="1" />
-    <xacro:velocity_joint_transmission joint="${prefix}_b_r_drive_joint" reduction="1" />
+    <xacro:SimpleTransmissionPosition joint="${prefix}_f_l_steer_joint" reduction="1" />
+    <xacro:SimpleTransmissionPosition joint="${prefix}_f_r_steer_joint" reduction="1" />
+    <xacro:SimpleTransmissionPosition joint="${prefix}_b_l_steer_joint" reduction="1" />
+    <xacro:SimpleTransmissionPosition joint="${prefix}_b_r_steer_joint" reduction="1" />
+    <xacro:SimpleTransmissionVelocity joint="${prefix}_f_l_drive_joint" reduction="1" />
+    <xacro:SimpleTransmissionVelocity joint="${prefix}_f_r_drive_joint" reduction="1" />
+    <xacro:SimpleTransmissionVelocity joint="${prefix}_b_l_drive_joint" reduction="1" />
+    <xacro:SimpleTransmissionVelocity joint="${prefix}_b_r_drive_joint" reduction="1" />
   </xacro:macro>
 </robot>

File: sobit_pro_description/urdf/wheel/wheel.urdf.xacro (robot description, xacro)
@@ -17,10 +17,10 @@
         <material name="black" />
       </visual>
-      <collision>
+      <!-- <collision>
         <origin xyz="${0.01388-0.05525/2} 0.0 -${0.005+0.034/2+0.02/2}" rpy="0.0 0.0 0.0" />
         <geometry>
           <box size="0.05525 0.0285 0.084" />
         </geometry>
-      </collision>
+      </collision> -->
       <inertial>
         <origin xyz="${0.01388-0.05525/2} 0.0 -${0.005+0.034/2+0.02/2}" rpy="0.0 0.0 0.0" />
@@ -49,10 +49,10 @@
         <material name="black" />
       </visual>
-      <collision>
+      <!-- <collision>
         <origin xyz="${0.0244+0.0436/2} 0.0 ${0.034/2+0.0149-0.1766/2}" rpy="0.0 0.0 0.0" />
         <geometry>
           <box size="0.0436 0.0495 0.1766" />
         </geometry>
-      </collision>
+      </collision> -->
       <inertial>
         <origin xyz="${0.0244+0.0436/2} 0.0 ${0.034/2+0.0149-0.1766/2}" rpy="0.0 0.0 0.0" />
@@ -70,5 +70,5 @@
       <child link="wheel_${prefix}_drive_link" />
       <axis xyz="-1.0 0.0 0.0 " />
-      <limit effort="3.0" velocity="7.913672" />
+      <limit effort="10.0" velocity="7.913672" />
     </joint>
     <link name="wheel_${prefix}_drive_link">
