Commit message: [FIX] correct link to hand

File: sobit_pro_description/urdf/hand/hand.urdf.xacro (robot description, xacro)
@@ -44,6 +44,6 @@
       <child link="${prefix_hand}_inner_l_link" />
       <origin xyz="0.0631932 0.0151495 0.0372231" rpy="0.0 0.0 0.0" />
-      <axis xyz="0.0 0.0 -1.0" />
-      <mimic joint="${prefix_hand}_joint" multiplier="1.0" offset="0" />
+      <axis xyz="0.0 0.0 1.0" />
+      <mimic joint="${prefix_hand}_joint" multiplier="-1.0" offset="0" />
       <limit lower="${-M_PI/2.0}" upper="0" effort="1" velocity="1" />
     </joint>
@@ -105,11 +105,11 @@
     </link>
     <joint name="${prefix_hand}_outer_l_joint" type="revolute">
-      <parent link="${prefix_hand}_inner_l_link" />
-      <!-- <parent link="${prefix_hand}_base_link" /> -->
+      <!-- <parent link="${prefix_hand}_inner_l_link" /> -->
+      <parent link="${prefix_hand}_base_link" />
       <child link="${prefix_hand}_outer_l_link" />
-      <origin xyz="-0.01988747 0.025 -0.01022197" rpy="0.0 0.0 0.0" />
-      <!-- <origin xyz="0.043193 0.04015 0.0282231" rpy="0.0 0.0 0.0" /> -->
-      <axis xyz="0.0 0.0 -1.0" />
-      <mimic joint="${prefix_hand}_joint" multiplier="1.0" offset="0" />
+      <!-- <origin xyz="-0.01988747 0.025 -0.01022197" rpy="0.0 0.0 0.0" /> -->
+      <origin xyz="0.043193 0.04015 0.0282231" rpy="0.0 0.0 0.0" />
+      <axis xyz="0.0 0.0 1.0" />
+      <mimic joint="${prefix_hand}_inner_l_joint" multiplier="1.0" offset="0" />
       <limit lower="${-M_PI/2.0}" upper="0" effort="1" velocity="1" />
     </joint>
@@ -139,9 +139,9 @@
     </link>
     <joint name="${prefix_hand}_outer_r_joint" type="revolute">
-      <parent link="${prefix_hand}_inner_r_link" />
-      <!-- <parent link="${prefix_hand}_base_link" /> -->
+      <!-- <parent link="${prefix_hand}_inner_r_link" /> -->
+      <parent link="${prefix_hand}_base_link" />
       <child link="${prefix_hand}_outer_r_link" />
-      <origin xyz="-0.01988747 -0.025 -0.01022197" rpy="0.0 0.0 0.0" />
-      <!-- <origin xyz="0.043193 -0.04015 0.0282231" rpy="0.0 0.0 0.0" /> -->
+      <!-- <origin xyz="-0.01988747 -0.025 -0.01022197" rpy="0.0 0.0 0.0" /> -->
+      <origin xyz="0.043193 -0.04015 0.0282231" rpy="0.0 0.0 0.0" />
       <axis xyz="0.0 0.0 1.0" />
       <mimic joint="${prefix_hand}_joint" multiplier="1.0" offset="0" />
@@ -173,14 +173,14 @@
     </link>
     <joint name="${prefix_hand}_${prefix_finger}_l_joint" type="revolute">
-      <parent link="${prefix_hand}_outer_l_link" />
+      <parent link="${prefix_hand}_inner_l_link" />
       <child link="${prefix_hand}_${prefix_finger}_l_link" />
-      <origin xyz="0.1040 0.0 -0.0190" rpy="0.0 0.0 0.0" />
-      <axis xyz="0.0 0.0 1.0" />
-      <mimic joint="${prefix_hand}_joint" multiplier="1.0" offset="0" />
+      <origin xyz="0.114316 0.0 -0.027729" rpy="0.0 0.0 0.0" />
+      <axis xyz="0.0 0.0 1.0" />
+      <mimic joint="${prefix_hand}_inner_l_joint" multiplier="-1.0" offset="0" />
       <limit lower="${-M_PI/2.0}" upper="0" effort="1" velocity="1" />
     </joint>
     <link name="${prefix_hand}_${prefix_finger}_l_link">
       <visual>
-        <origin xyz="0.0 0.0 0.0" rpy="0.0 0.0 ${M_PI/2.0}" />
+        <origin xyz="-0.029998 0.025 0.0" rpy="0.0 0.0 ${M_PI/2.0}" />
         <geometry>
           <mesh filename="package://sobit_pro_description/meshes/hand/hand_finger_l.stl" scale="0.001 0.001 0.001" />
@@ -189,8 +189,8 @@
       </visual>
       <collision>
-        <origin xyz="${0.03+(0.08+0.00707)/2} -0.025 -${0.018/2}" rpy="0.0 0.0 0.0" />
-        <!-- <origin xyz="0.0 0.0 0.0" rpy="0.0 0.0 ${M_PI/2.0}" /> -->
-        <geometry>
-          <box size="${0.08-0.00707} 0.01137 0.044" />
+        <origin xyz="${0.007071+(0.012042+0.061128)/2} 0.0 -${0.018/2}" rpy="0.0 0.0 0.0" />
+        <!-- <origin xyz="0.0 0.0 0.0" rpy="0.0 0.0 ${M_PI/2.0}" /> -->
+        <geometry>
+          <box size="${0.012042+0.061128} 0.01137 0.044" />
           <!-- <mesh filename="package://sobit_pro_description/meshes/hand/hand_finger_l.stl" scale="0.001 0.001 0.001" /> -->
         </geometry>
@@ -205,14 +205,14 @@
     </link>
     <joint name="${prefix_hand}_${prefix_finger}_r_joint" type="revolute">
-      <parent link="${prefix_hand}_outer_r_link" />
+      <parent link="${prefix_hand}_inner_r_link" />
       <child link="${prefix_hand}_${prefix_finger}_r_link" />
-      <origin xyz="0.1040 0.0 -0.0190" rpy="0.0 0.0 0.0" />
-      <axis xyz="0.0 0.0 -1.0" />
-      <mimic joint="${prefix_hand}_joint" multiplier="1.0" offset="0" />
+      <origin xyz="0.114316 0.0 -0.027729" rpy="0.0 0.0 0.0" />
+      <axis xyz="0.0 0.0 1.0" />
+      <mimic joint="${prefix_hand}_inner_r_joint" multiplier="-1.0" offset="0" />
       <limit lower="${-M_PI/2.0}" upper="0" effort="1" velocity="1" />
     </joint>
     <link name="${prefix_hand}_${prefix_finger}_r_link">
       <visual>
-        <origin xyz="0.0 0.0 0.0" rpy="0.0 0.0 ${M_PI/2.0}" />
+        <origin xyz="-0.029998 -0.025 0.0" rpy="0.0 0.0 ${M_PI/2.0}" />
         <geometry>
           <mesh filename="package://sobit_pro_description/meshes/hand/hand_finger_r.stl" scale="0.001 0.001 0.001" />
@@ -221,8 +221,8 @@
       </visual>
       <collision>
-        <origin xyz="${0.03+(0.08+0.00707)/2} 0.025 -${0.018/2}" rpy="0.0 0.0 0.0" />
-        <!-- <origin xyz="0.0 0.0 0.0" rpy="0.0 0.0 ${M_PI/2.0}" /> -->
-        <geometry>
-          <box size="${0.08-0.00707} 0.01137 0.044" />
+        <origin xyz="${0.007071+(0.012042+0.061128)/2} 0.0 -${0.018/2}" rpy="0.0 0.0 0.0" />
+        <!-- <origin xyz="0.0 0.0 0.0" rpy="0.0 0.0 ${M_PI/2.0}" /> -->
+        <geometry>
+          <box size="${0.012042+0.061128} 0.01137 0.044" />
           <!-- <mesh filename="package://sobit_pro_description/meshes/hand/hand_finger_r.stl" scale="0.001 0.001 0.001" /> -->
         </geometry>

Commit message: [UPD] Velocities and effort for hand in gazebo

File: sobit_pro_description/urdf/hand/hand.urdf.xacro (robot description, xacro)
@@ -42,5 +42,5 @@
       <origin xyz="0.0631932 0.0151495 0.0372231" rpy="0.0 0.0 0.0" />
       <axis xyz="0.0 0.0 1.0" />
-      <limit lower="0" upper="${M_PI/2.0}" effort="1.0" velocity="2.0"/>
+      <limit lower="0" upper="${M_PI/2.0}" effort="1.0" velocity="4.796165"/>
       <mimic joint="${prefix_hand}_joint" multiplier="1" offset="0" />
       <!-- <dynamics damping="50.0" friction="5.0"/> -->
@@ -74,5 +74,5 @@
       <origin xyz="0.0631932 -0.0151495 0.0372231" rpy="0.0 0.0 0.0" />
       <axis xyz="0.0 0.0 1.0" />
-      <limit lower="${-M_PI/2.0}" upper="0" effort="1.0" velocity="2.0" />
+      <limit lower="${-M_PI/2.0}" upper="0" effort="1.0" velocity="4.796165" />
     </joint>
     <link name="${prefix_hand}_link">
@@ -105,5 +105,5 @@
       <axis xyz="0.0 0.0 1.0" />
       <!-- <mimic joint="{prefix_hand}_joint" multiplier="1.0" offset="0" /> -->
-      <limit lower="0" upper="${M_PI/2.0}" effort="1.0" velocity="2.0"/>
+      <limit lower="0" upper="${M_PI/2.0}" effort="1.0" velocity="4.796165"/>
     </joint>
     <link name="${prefix_hand}_outer_l_link">
@@ -136,5 +136,5 @@
       <origin xyz="0.043193 -0.04015 0.0282231" rpy="0.0 0.0 0.0" />
       <axis xyz="0.0 0.0 1.0" />
-      <limit lower="${-M_PI/2.0}" upper="0" effort="1.0" velocity="2.0"/>
+      <limit lower="${-M_PI/2.0}" upper="0" effort="1.0" velocity="4.796165"/>
       <mimic joint="${prefix_hand}_joint" multiplier="1.0" offset="0" />
     </joint>
@@ -169,5 +169,5 @@
       <axis xyz="0.0 0.0 1.0" />
       <mimic joint="${prefix_hand}_joint" multiplier="1.0" offset="0" />
-      <limit lower="${-M_PI/2.0}" upper="0" effort="4.1" velocity="4" />
+      <limit lower="${-M_PI/2.0}" upper="0" effort="4.1" velocity="4.796165" />
       <!-- <dynamics damping="0.05" friction="0.0"/> -->
     </joint>
@@ -200,5 +200,5 @@
       <axis xyz="0.0 0.0 1.0" />
       <mimic joint="${prefix_hand}_joint" multiplier="-1.0" offset="0" />
-      <limit lower="0" upper="${M_PI/2.0}" effort="4.1" velocity="1" />
+      <limit lower="0" upper="${M_PI/2.0}" effort="4.1" velocity="4.796165" />
       <!-- <dynamics damping="50.0" friction="5.0"/> -->
     </joint>

Commit message: [fix]behavior of the joint_hand  when started display.launch.py

File: sobit_pro_description/urdf/hand/hand.urdf.xacro (robot description, xacro)
@@ -43,5 +43,5 @@
       <axis xyz="0.0 0.0 1.0" />
       <limit lower="0" upper="${M_PI/2.0}" effort="1.0" velocity="4.796165"/>
-      <mimic joint="${prefix_hand}_joint" multiplier="1" offset="0" />
+      <mimic joint="${prefix_hand}_joint" multiplier="-1.0" offset="0" />
       <!-- <dynamics damping="50.0" friction="5.0"/> -->
     </joint>
@@ -99,10 +99,10 @@
     </link>
 <xacro:if value="${enable_outer_l}">
-    <joint name="${prefix_hand}_outer_l_joint" type="continuous">
+    <joint name="${prefix_hand}_outer_l_joint" type="revolute">
       <parent link="${prefix_hand}_base_link" />
       <child link="${prefix_hand}_outer_l_link" />
       <origin xyz="0.043193 0.04015 0.0282231" rpy="0.0 0.0 0.0" />
       <axis xyz="0.0 0.0 1.0" />
-      <!-- <mimic joint="{prefix_hand}_joint" multiplier="1.0" offset="0" /> -->
+      <mimic joint="${prefix_hand}_joint" multiplier="-1.0" offset="0" />
       <limit lower="0" upper="${M_PI/2.0}" effort="1.0" velocity="4.796165"/>
     </joint>
